File: Input Hardware/PCB/Input Board/Rx.kicad_sch (KiCad schematic)
At the start: 32 parts

Commit message: Revert "Merge branch 'main' of https://github.com/seanryder264/HAYES"
This reverts commit bd795aa78e7b7049f2eb147f65c5fdd388d288f7, reversing
changes made to 52c69ad61d85eaec29fd6b5b9781512ece56f4ea.
Connections:
- net Rx Preamp 1/RXIN1: no longer names the net of L201.2
- net Rx Preamp 1/RXIN2: no longer names the net of L202.2
- net Rx Preamp 1/RXIN3: no longer names the net of L203.2
- net Rx Preamp 1/RXIN4: no longer names the net of L204.2
- net Rx Preamp 1/RXIN5: no longer names the net of L205.2
- net Rx Preamp 1/RXIN6: no longer names the net of L206.2
- net Rx Preamp 1/RXIN7: no longer names the net of L207.2
- net Rx Preamp 1/RXIN8: no longer names the net of L208.2
Other:
- sheet Rx Row Amplifier 1 renamed Rx Preamp 1
- sheet Rx Row Amplifier 2 renamed Rx Preamp 2
- sheet Rx Row Amplifier 3 renamed Rx Preamp 3
- sheet Rx Row Amplifier 4 renamed Rx Preamp 4
- sheet Rx Preamp 1 ports: added none; removed RXIN1, RXIN2, RXIN3, RXIN4, RXIN5, RXIN6, RXIN7, RXIN8, RXOUT1, RXOUT2, RXOUT3, RXOUT4, RXOUT5, RXOUT6, RXOUT7, RXOUT8
- moved on the sheet: L201, L202, L203, L204, L205, L206, L207, L208, L209, L210, L211, L212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
