File: Input Hardware/PCB/Input Board/Input Board.kicad_sch (KiCad schematic)
At the start: 4 parts

Commit message: Progress
Other:
- sheet Multiplexing, Gain & Filtering renamed Multiplex, Gain & Filter 1
- added sheet Measurement & Control (ctrl.kicad_sch)
- added sheet Multiplex, Gain & Filter 2 (mux.kicad_sch)
- added sheet Multiplex, Gain & Filter 3 (mux.kicad_sch)
- added sheet Multiplex, Gain & Filter 4 (mux.kicad_sch)
- sheet Multiplex, Gain & Filter 1 ports: added In1, In2, In3, In4, In5, In6, In7, In8, Mux A, Mux B, Mux C, Mux Inhibit, Out; removed Rx1, Rx10, Rx11, Rx12, Rx13, Rx14, Rx15, Rx16, Rx17, Rx18, Rx19, Rx2, Rx20, Rx21, Rx22, Rx23, Rx24, Rx25, Rx26, Rx27, Rx28, Rx29, Rx3, Rx30, Rx31, Rx32, Rx4, Rx5, Rx6, Rx7, Rx8, Rx9

Commit message: Fix Name
Other:
- sheet Measurement & Control ports: added Rx1, Rx2, Rx3, Rx4; removed none
Changed lines of the file:
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@@
+	(wire
+		(pts
+			(xy 88.9 71.12) (xy 88.9 48.26)
+		)
+		(stroke
+			(width 0)
+			(type default)
+		)
+	)
 	(wire
 		(pts
@@
 	(wire
 		(pts
+			(xy 76.2 121.92) (xy 93.98 121.92)
+		)
+		(stroke
+			(width 0)
+			(type default)
+		)
+	)
+	(wire
+		(pts
 			(xy 76.2 78.74) (xy 78.74 78.74)
 		)
@@
 	(wire
 		(pts
-			(xy 86.36 35.56) (xy 95.25 35.56)
-		)
-		(stroke
-			(width 0)
-			(type default)
-		)
-	)
-	(wire
-		(pts
-			(xy 78.74 27.94) (xy 95.25 27.94)
+			(xy 86.36 35.56) (xy 96.52 35.56)
+		)
+		(stroke
+			(width 0)
+			(type default)
+		)
+	)
+	(wire
+		(pts
+			(xy 78.74 27.94) (xy 96.52 27.94)
 		)
 		(stroke
@@
 	(wire
 		(pts
-			(xy 83.82 33.02) (xy 95.25 33.02)
+			(xy 83.82 33.02) (xy 96.52 33.02)
 		)
 		(stroke
@@
 	(wire
 		(pts
+			(xy 76.2 96.52) (xy 91.44 96.52)
+		)
+		(stroke
+			(width 0)
+			(type default)
+		)
+	)
+	(wire
+		(pts
 			(xy 38.1 119.38) (xy 50.8 119.38)
 		)
@@
 	(wire
 		(pts
+			(xy 91.44 50.8) (xy 96.52 50.8)
+		)
+		(stroke
+			(width 0)
+			(type default)
+		)
+	)
+	(wire
+		(pts
 			(xy 76.2 35.56) (xy 86.36 35.56)
 		)
@@
 	(wire
 		(pts
+			(xy 88.9 48.26) (xy 96.52 48.26)
+		)
+		(stroke
+			(width 0)
+			(type default)
+		)
+	)
+	(wire
+		(pts
 			(xy 38.1 60.96) (xy 50.8 60.96)
 		)
@@
 	(wire
 		(pts
-			(xy 81.28 30.48) (xy 95.25 30.48)
+			(xy 93.98 121.92) (xy 93.98 53.34)
+		)
+		(stroke
+			(width 0)
+			(type default)
+		)
+	)
+	(wire
+		(pts
+			(xy 81.28 30.48) (xy 96.52 30.48)
 		)
 		(stroke
@@
 	(wire
 		(pts
+			(xy 91.44 96.52) (xy 91.44 50.8)
+		)
+		(stroke
+			(width 0)
+			(type default)
+		)
+	)
+	(wire
+		(pts
+			(xy 76.2 45.72) (xy 96.52 45.72)
+		)
+		(stroke
+			(width 0)
+			(type default)
+		)
+	)
+	(wire
+		(pts
 			(xy 76.2 81.28) (xy 81.28 81.28)
 		)
@@
 	(wire
 		(pts
+			(xy 76.2 71.12) (xy 88.9 71.12)
+		)
+		(stroke
+			(width 0)
+			(type default)
+		)
+	)
+	(wire
+		(pts
 			(xy 76.2 58.42) (xy 83.82 58.42)
 		)
@@
 		(pts
 			(xy 38.1 38.1) (xy 50.8 38.1)
+		)
+		(stroke
+			(width 0)
+			(type default)
+		)
+	)
+	(wire
+		(pts
+			(xy 93.98 53.34) (xy 96.52 53.34)
 		)
 		(stroke
@@
 	)
 	(sheet
-		(at 95.25 25.4)
-		(size 25.4 38.1)
+		(at 96.52 25.4)
+		(size 30.48 38.1)
 		(exclude_from_sim no)
 		(in_bom yes)
@@
 		)
 		(property "Sheetname" "Measurement & Control"
-			(at 95.25 24.6884 0)
+			(at 96.52 24.6884 0)
 			(effects
 				(font
@@
 		)
 		(property "Sheetfile" "ctrl.kicad_sch"
-			(at 95.25 64.0846 0)
+			(at 96.52 64.0846 0)
 			(effects
 				(font
@@
 		)
 		(pin "Mux A" output
-			(at 95.25 27.94 180)
+			(at 96.52 27.94 180)
 			(effects
 				(font
@@
 		)
 		(pin "Mux B" output
-			(at 95.25 30.48 180)
+			(at 96.52 30.48 180)
 			(effects
 				(font
@@
 		)
 		(pin "Mux C" output
-			(at 95.25 33.02 180)
+			(at 96.52 33.02 180)
 			(effects
 				(font
@@
 		)
 		(pin "Mux Inhibit" output
-			(at 95.25 35.56 180)
-			(effects
-				(font
+			(at 96.52 35.56 180)
+			(effects
+				(font
+					(size 1.27 1.27)
+				)
+				(justify left)
+			)
+		)
+		(pin "Rx1" input
+			(at 96.52 45.72 180)
+			(effects
+				(font
+					(size 1.27 1.27)
+				)
+				(justify left)
+			)
+		)
+		(pin "Rx2" input
+			(at 96.52 48.26 180)
+			(effects
+				(font
+					(size 1.27 1.27)
+				)
+				(justify left)
+			)
+		)
+		(pin "Rx3" input
+			(at 96.52 50.8 180)
+			(effects
+				(font
+					(size 1.27 1.27)
+				)
+				(justify left)
+			)
+		)
+		(pin "Rx4" input
+			(at 96.52 53.34 180)
+			(effects
+				(font

Commit message: Progress
Other:
- added sheet Transmit Coils (Tx.kicad_sch)
- added sheet User Input (Input.kicad_sch)
- sheet Measurement & Control ports: added RCLK, SDO, SRCLK, ~{OE}, ~{SRCLR}; removed none
- note added: "Check Supplies and 2.5V reference voltages"

Commit message: WEEEE
Changed lines of the file:
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@@
-	)
-	(junction
-		(at 88.9 177.8)
-		(diameter 0)
-		(color 0 0 0 0)
 	)
 	(junction
@@
 	)
 	(symbol
-		(lib_id "power:GNDPWR")
-		(at 88.9 177.8 90)
-		(unit 1)
-		(exclude_from_sim no)
-		(in_bom yes)
-		(on_board yes)
-		(dnp no)
-		(fields_autoplaced yes)
-		(property "Reference" "#PWR059"
-			(at 93.98 177.8 0)
-			(effects
-				(font
-					(size 1.27 1.27)
-				)
-				(hide yes)
-			)
-		)
-		(property "Value" "GNDPWR"
-			(at 92.71 177.9269 90)
-			(effects
-				(font
-					(size 1.27 1.27)
-				)
-				(justify right)
-			)
-		)
-		(property "Footprint" ""
-			(at 90.17 177.8 0)
-			(effects
-				(font
-					(size 1.27 1.27)
-				)
-				(hide yes)
-			)
-		)
-		(property "Datasheet" ""
-			(at 90.17 177.8 0)
-			(effects
-				(font
-					(size 1.27 1.27)
-				)
-				(hide yes)
-			)
-		)
-		(property "Description" "Power symbol creates a global label with name \"GNDPWR\" , global ground"
-			(at 88.9 177.8 0)
-			(effects
-				(font
-					(size 1.27 1.27)
-				)
-				(hide yes)
-			)
-		)
-		(pin "1"
-		)
-		(instances
-			(project ""
-				(path "/198ad8d1-66e3-4deb-889c-1af2b81e67c3"
-					(reference "#PWR059")
-					(unit 1)
-				)
-			)
-		)
-	)
-	(symbol
 		(lib_id "Mechanical:MountingHole")
 		(at 25.4 171.45 0)
@@
 	(symbol
 		(lib_id "power:GND")
-		(at 88.9 177.8 0)
+		(at 88.9 177.8 90)
 		(unit 1)
 		(exclude_from_sim no)
@@
 		(fields_autoplaced yes)
 		(property "Reference" "#PWR058"
-			(at 88.9 184.15 0)
+			(at 95.25 177.8 0)
 			(effects
 				(font
@@
 		)
 		(property "Value" "GND"
-			(at 88.9 182.88 0)
-			(effects
-				(font
-					(size 1.27 1.27)
-				)
-			)
-		)
+			(at 92.71 177.7999 90)
+			(effects
+				(font
+					(size 1.27 1.27)
+				)
+				(justify right)
+			)
+		)

Commit message: Power Board, Row amplifier setup etc
Other:
- added sheet Power (power.kicad_sch)
Changed lines of the file:
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@@
+	)
+	(sheet
+		(at 135.89 153.67)
+		(size 27.94 24.13)
+		(exclude_from_sim no)
+		(in_bom yes)
+		(on_board yes)
+		(dnp no)
+		(fields_autoplaced yes)
+		(stroke
+			(width 0.1524)
+			(type solid)
+		)
+		(fill
+			(color 0 0 0 0.0000)
+		)
+		(property "Sheetname" "Power"
+			(at 135.89 152.9584 0)
+			(effects
+				(font
+					(size 1.27 1.27)
+				)
+				(justify left bottom)
+			)
+		)
+		(property "Sheetfile" "power.kicad_sch"
+			(at 135.89 178.3846 0)
+			(effects
+				(font
+					(size 1.27 1.27)
+				)
+				(justify left top)
+			)
+		)
+		(instances
+			(project "Input Board"
+				(path "/198ad8d1-66e3-4deb-889c-1af2b81e67c3"
+					(page "14")
+				)
+			)
+		)
 	)
 	(sheet

Commit message: integrate
Other:
- note removed: "Check Supplies and 2.5V reference voltages"
Changed lines of the file:
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@@
 	(generator_version "9.0")
 	(paper "A4")
-	(text "Check Supplies and 2.5V reference voltages"
-		(exclude_from_sim no)
-		(at 88.9 175.26 0)
-		(effects
-			(font
-				(size 1.27 1.27)
-			)
-		)
-	)
 	(junction
 		(at 83.82 58.42)
@@
 	)
 	(symbol
-		(lib_id "power:GNDA")
-		(at 88.9 177.8 270)
-		(unit 1)
-		(exclude_from_sim no)
-		(in_bom yes)
-		(on_board yes)
-		(dnp no)
-		(fields_autoplaced yes)
-		(property "Reference" "#PWR057"
-			(at 82.55 177.8 0)
-			(effects
-				(font
-					(size 1.27 1.27)
-				)
-				(hide yes)
-			)
-		)
-		(property "Value" "GNDA"
-			(at 85.09 177.7999 90)
-			(effects
-				(font
-					(size 1.27 1.27)
-				)
-				(justify right)
-			)
-		)
-		(property "Footprint" ""
-			(at 88.9 177.8 0)
-			(effects
-				(font
-					(size 1.27 1.27)
-				)
-				(hide yes)
-			)
-		)
-		(property "Datasheet" ""
-			(at 88.9 177.8 0)
-			(effects
-				(font
-					(size 1.27 1.27)
-				)
-				(hide yes)
-			)
-		)
-		(property "Description" "Power symbol creates a global label with name \"GNDA\" , analog ground"
-			(at 88.9 177.8 0)
-			(effects
-				(font
-					(size 1.27 1.27)
-				)
-				(hide yes)
-			)
-		)
-		(pin "1"
-		)
-		(instances
-			(project ""
-				(path "/198ad8d1-66e3-4deb-889c-1af2b81e67c3"
-					(reference "#PWR057")
-					(unit 1)
-				)
-			)
-		)
-	)
-	(symbol
 		(lib_id "Mechanical:MountingHole")
 		(at 25.4 171.45 0)
@@
 					(unit 1)
 				)
-			)
-		)
-	)
-	(symbol
-		(lib_id "power:GND")
-		(at 88.9 177.8 90)
-		(unit 1)
-		(exclude_from_sim no)
-		(in_bom yes)
-		(on_board yes)
-		(dnp no)
-		(fields_autoplaced yes)
-		(property "Reference" "#PWR058"
-			(at 95.25 177.8 0)
-			(effects
-				(font
-					(size 1.27 1.27)
-				)
-				(hide yes)
-			)
-		)
-		(property "Value" "GND"
-			(at 92.71 177.7999 90)
-			(effects
-				(font
-					(size 1.27 1.27)
-				)
-				(justify right)
-			)
-		)
-		(property "Footprint" ""
-			(at 88.9 177.8 0)
-			(effects
-				(font
-					(size 1.27 1.27)
-				)
-				(hide yes)
-			)
-		)
-		(property "Datasheet" ""
-			(at 88.9 177.8 0)
-			(effects
-				(font
-					(size 1.27 1.27)
-				)
-				(hide yes)
-			)
-		)
-		(property "Description" "Power symbol creates a global label with name \"GND\" , ground"
-			(at 88.9 177.8 0)
-			(effects
-				(font
-					(size 1.27 1.27)
-				)
-				(hide yes)
-			)
-		)
-		(pin "1"
-		)
-		(instances
-			(project ""
-				(path "/198ad8d1-66e3-4deb-889c-1af2b81e67c3"
-					(reference "#PWR058")
-					(unit 1)
-				)

Commit message: test commit and minor updates
Parts:
- removed H101, H102, H103, H104: MountingHole, MountingHole:MountingHole_3.2mm_M3, symbol Mechanical:MountingHole
- added H1, H2, H3, H4, H5, H6: MountingHole, MountingHole:MountingHole_3.2mm_M3, symbol Mechanical:MountingHole

Commit message: explosion 💥
Other:
- sheet Multiplex, Gain & Filter 1 renamed Demux & Amplifier 4
- sheet Multiplex, Gain & Filter 2 renamed Demux & Amplifier 2
- sheet Multiplex, Gain & Filter 3 renamed Demux & Amplifier 1
- sheet Multiplex, Gain & Filter 4 renamed Demux & Amplifier 3
- sheet Receive Coils renamed Receiver Stage
Changed lines of the file:
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@@
 			(color 0 0 0 0.0000)
 		)
-		(property "Sheetname" "Multiplex, Gain & Filter 1"
+		(property "Sheetname" "Demux & Amplifier 4"
 			(at 50.8 25.9584 0)
 			(effects
@@
 			(color 0 0 0 0.0000)
 		)
-		(property "Sheetname" "Multiplex, Gain & Filter 4"
+		(property "Sheetname" "Demux & Amplifier 3"
 			(at 50.8 102.1584 0)
 			(effects
@@
 			(color 0 0 0 0.0000)
 		)
-		(property "Sheetname" "Multiplex, Gain & Filter 3"
+		(property "Sheetname" "Demux & Amplifier 1"
 			(at 50.8 76.7584 0)
 			(effects
@@
 			(color 0 0 0 0.0000)
 		)
-		(property "Sheetname" "Multiplex, Gain & Filter 2"
+		(property "Sheetname" "Demux & Amplifier 2"
 			(at 50.8 51.3584 0)
 			(effects
@@
 			(color 0 0 0 0.0000)
 		)
-		(property "Sheetname" "Receive Coils"
+		(property "Sheetname" "Receiver Stage"
 			(at 25.4 24.6884 0)
 			(effects
