File: Input Hardware/PCB/Input Board/Input Board.kicad_sch (KiCad schematic)
At the start: 4 parts

Commit message: sims and other crap
Other:
- sheet Transmit Coils ports: added DRIVER_RCLK, DRIVER_SER, DRIVER_SRCLK, DRIVER_~{SLEEP}; removed RCLK, SDI, SRCLK, ~{OE}

Commit message: Schematic Cleanup
Other:
- sheet Measurement & Control ports: added none; removed ~{OE}
- sheet Transmit Coils ports: added none; removed DRIVER_~{SLEEP}

Commit message: Layout Progress
Other:
- sheet Measurement & Control ports: added Push_1, Push_2, Push_3; removed TSC_1, TSC_2, TSC_3
- sheet User Input ports: added Push_1, Push_2, Push_3; removed TSC_1, TSC_2, TSC_3
Changed lines of the file:
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@@
-			)
-		)
-		(pin "TSC_1" output
-			(at 139.7 99.06 180)
-			(effects
-				(font
-					(size 1.27 1.27)
-				)
-				(justify left)
-			)
-		)
-		(pin "TSC_2" output
-			(at 139.7 101.6 180)
-			(effects
-				(font
-					(size 1.27 1.27)
-				)
-				(justify left)
-			)
-		)
-		(pin "TSC_3" output
-			(at 139.7 104.14 180)
-			(effects
-				(font
-					(size 1.27 1.27)
-				)
-				(justify left)
 			)
 		)
@@
 		(pin "UI_SRCLK" output
 			(at 139.7 111.76 180)
+			(effects
+				(font
+					(size 1.27 1.27)
+				)
+				(justify left)
+			)
+		)
+		(pin "Push_1" input
+			(at 139.7 99.06 180)
+			(effects
+				(font
+					(size 1.27 1.27)
+				)
+				(justify left)
+			)
+		)
+		(pin "Push_2" input
+			(at 139.7 101.6 180)
+			(effects
+				(font
+					(size 1.27 1.27)
+				)
+				(justify left)
+			)
+		)
+		(pin "Push_3" input
+			(at 139.7 104.14 180)
 			(effects
 				(font
@@
 			)
 		)
-		(pin "TSC_1" input
-			(at 127 99.06 0)
-			(effects
-				(font
-					(size 1.27 1.27)
-				)
-				(justify right)
-			)
-		)
-		(pin "TSC_2" input
-			(at 127 101.6 0)
-			(effects
-				(font
-					(size 1.27 1.27)
-				)
-				(justify right)
-			)
-		)
-		(pin "TSC_3" input
-			(at 127 104.14 0)
-			(effects
-				(font
-					(size 1.27 1.27)
-				)
-				(justify right)
-			)
-		)
 		(pin "UI_RCLK" input
 			(at 127 114.3 0)
@@
 			(effects
 				(font
+					(size 1.27 1.27)
+				)
+				(justify right)
+			)
+		)
+		(pin "Push_1" output
+			(at 127 99.06 0)
+			(effects
+				(font
+					(size 1.27 1.27)
+				)
+				(justify right)
+			)
+		)
+		(pin "Push_2" output
+			(at 127 101.6 0)
+			(effects
+				(font
+					(size 1.27 1.27)
+				)
+				(justify right)
+			)
+		)
+		(pin "Push_3" output
+			(at 127 104.14 0)
+			(effects
+				(font

Commit message: sleep pin rewire
Other:
- sheet Measurement & Control ports: added SLEEP; removed none
- sheet Transmit Coils ports: added SLEEP; removed none
Changed lines of the file:
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@@
+	(wire
+		(pts
+			(xy 165.1 35.56) (xy 180.34 35.56)
+		)
+		(stroke
+			(width 0)
+			(type default)
+		)
+	)
 	(wire
 		(pts
@@
 			)
 		)
+		(pin "SLEEP" input
+			(at 165.1 35.56 0)
+			(effects
+				(font
+					(size 1.27 1.27)
+				)
+				(justify right)
+			)
+		)
 		(instances
 			(project "Input Board"
@@
 			(effects
 				(font
+					(size 1.27 1.27)
+				)
+				(justify left)
+			)
+		)
+		(pin "SLEEP" input
+			(at 180.34 35.56 180)
+			(effects
+				(font

Commit message: minor cosmetic
Other:
- note removed: "Broken Stuff/Fixes/Recs: > Input Offset Wiring > Rotary Encoder Wiring > No names on buttons if possible to allow for maximum flexibility (potentially ontop instead?) > OSC_OUT conflict with Cube"
- moved on the sheet: H101, H102, H103, H104
Changed lines of the file:
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@@
 	(generator_version "9.0")
 	(paper "A4")
-	(rectangle
-		(start 186.69 109.22)
-		(end 246.38 153.67)
-		(stroke
-			(width 0)
-			(type default)
-		)
-		(fill
-			(type none)
-		)
-	)
-	(text "Broken Stuff/Fixes/Recs:\n\n> Input Offset Wiring\n> Rotary Encoder Wiring\n> No names on buttons if possible to allow for maximum \nflexibility (potentially ontop instead?)\n> OSC_OUT conflict with Cube"
-		(exclude_from_sim no)
-		(at 187.96 118.11 0)
-		(effects
-			(font
-				(size 1.27 1.27)
-			)
-			(justify left)
-		)
-	)
 	(junction
 		(at 83.82 58.42)
@@
 	(symbol
 		(lib_id "Mechanical:MountingHole")
-		(at 46.99 181.61 0)
+		(at 19.05 191.77 0)
 		(unit 1)
 		(exclude_from_sim no)
@@
 		(fields_autoplaced yes)
 		(property "Reference" "H104"
-			(at 49.53 180.3399 0)
+			(at 21.59 190.4999 0)
 			(effects
 				(font
@@
 		)
 		(property "Value" "MountingHole"
-			(at 49.53 182.8799 0)
+			(at 21.59 193.0399 0)
 			(effects
 				(font
@@
 		)
 		(property "Footprint" "MountingHole:MountingHole_3.2mm_M3"
-			(at 46.99 181.61 0)
+			(at 19.05 191.77 0)
 			(effects
 				(font
@@
 		)
 		(property "Datasheet" "~"
-			(at 46.99 181.61 0)
+			(at 19.05 191.77 0)
 			(effects
 				(font
@@
 		)
 		(property "Description" "Mounting Hole without connection"
-			(at 46.99 181.61 0)
+			(at 19.05 191.77 0)
 			(effects
 				(font
@@
 	(symbol
 		(lib_id "Mechanical:MountingHole")
-		(at 46.99 166.37 0)
+		(at 19.05 176.53 0)
 		(unit 1)
 		(exclude_from_sim no)
@@
 		(fields_autoplaced yes)
 		(property "Reference" "H101"
-			(at 49.53 165.0999 0)
+			(at 21.59 175.2599 0)
 			(effects
 				(font
@@
 		)
 		(property "Value" "MountingHole"
-			(at 49.53 167.6399 0)
+			(at 21.59 177.7999 0)
 			(effects
 				(font
@@
 		)
 		(property "Footprint" "MountingHole:MountingHole_3.2mm_M3"
-			(at 46.99 166.37 0)
+			(at 19.05 176.53 0)
 			(effects
 				(font
@@
 		)
 		(property "Datasheet" "~"
-			(at 46.99 166.37 0)
+			(at 19.05 176.53 0)
 			(effects
 				(font
@@
 		)
 		(property "Description" "Mounting Hole without connection"
-			(at 46.99 166.37 0)
+			(at 19.05 176.53 0)
 			(effects
 				(font
@@
 	(symbol
 		(lib_id "Mechanical:MountingHole")
-		(at 46.99 176.53 0)
+		(at 19.05 186.69 0)
 		(unit 1)
 		(exclude_from_sim no)
@@
 		(fields_autoplaced yes)
 		(property "Reference" "H103"
-			(at 49.53 175.2599 0)
+			(at 21.59 185.4199 0)
 			(effects
 				(font
@@
 		)
 		(property "Value" "MountingHole"
-			(at 49.53 177.7999 0)
+			(at 21.59 187.9599 0)
 			(effects
 				(font
@@
 		)
 		(property "Footprint" "MountingHole:MountingHole_3.2mm_M3"
-			(at 46.99 176.53 0)
+			(at 19.05 186.69 0)
 			(effects
 				(font
@@
 		)
 		(property "Datasheet" "~"
-			(at 46.99 176.53 0)
+			(at 19.05 186.69 0)
 			(effects
 				(font
@@
 		)
 		(property "Description" "Mounting Hole without connection"
-			(at 46.99 176.53 0)
+			(at 19.05 186.69 0)
 			(effects
 				(font
@@
 	(symbol
 		(lib_id "Mechanical:MountingHole")
-		(at 46.99 171.45 0)
+		(at 19.05 181.61 0)
 		(unit 1)
 		(exclude_from_sim no)
@@
 		(fields_autoplaced yes)
 		(property "Reference" "H102"
-			(at 49.53 170.1799 0)
+			(at 21.59 180.3399 0)
 			(effects
 				(font
@@
 		)
 		(property "Value" "MountingHole"
-			(at 49.53 172.7199 0)
+			(at 21.59 182.8799 0)
 			(effects
 				(font
@@
 		)
 		(property "Footprint" "MountingHole:MountingHole_3.2mm_M3"
-			(at 46.99 171.45 0)
+			(at 19.05 181.61 0)
 			(effects
 				(font
@@
 		)
 		(property "Datasheet" "~"
-			(at 46.99 171.45 0)
+			(at 19.05 181.61 0)
 			(effects
 				(font
@@
 		)
 		(property "Description" "Mounting Hole without connection"
-			(at 46.99 171.45 0)
+			(at 19.05 181.61 0)
 			(effects
 				(font
@@
 	)
 	(sheet
-		(at 139.7 135.89)
-		(size 12.7 7.62)
+		(at 180.34 80.01)
+		(size 12.7 11.43)
 		(exclude_from_sim no)
 		(in_bom yes)
@@
 		)
 		(property "Sheetname" "Power"
-			(at 139.7 135.1784 0)
+			(at 180.34 79.2984 0)
 			(effects
 				(font
@@
 		)
 		(property "Sheetfile" "power.kicad_sch"
-			(at 139.7 144.0946 0)
-			(effects
-				(font
+			(at 180.34 92.0246 0)
+			(effects
+				(font
