File: Input Hardware/PCB/Input Board/power.kicad_sch (KiCad schematic)
At the start: 10 parts, among them U1 LM317_TO-252, U3 LM317_TO-252

Commit message: integrate
Parts:
- R3: value 1k -> 768
Connections:
- net 1.8V renamed 1.65V
- net VUSB renamed +5V
Changed lines of the file:
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@@
+	)
+	(junction
+		(at 44.45 50.8)
+		(diameter 0)
+		(color 0 0 0 0)
 	)
 	(junction
@@
 	(wire
 		(pts
-			(xy 41.91 62.23) (xy 58.42 62.23)
-		)
-		(stroke
-			(width 0)
-			(type default)
-		)
-	)
-	(wire
-		(pts
 			(xy 71.12 107.95) (xy 58.42 107.95)
 		)
@@
 	(wire
 		(pts
-			(xy 135.89 107.95) (xy 135.89 106.68)
-		)
-		(stroke
-			(width 0)
-			(type default)
-		)
-	)
-	(wire
-		(pts
 			(xy 58.42 62.23) (xy 71.12 62.23)
 		)
@@
 	(wire
 		(pts
-			(xy 41.91 62.23) (xy 41.91 60.96)
-		)
-		(stroke
-			(width 0)
-			(type default)
-		)
-	)
-	(wire
-		(pts
 			(xy 71.12 72.39) (xy 71.12 87.63)
 		)
@@
 	(wire
 		(pts
+			(xy 44.45 62.23) (xy 58.42 62.23)
+		)
+		(stroke
+			(width 0)
+			(type default)
+		)
+	)
+	(wire
+		(pts
 			(xy 71.12 87.63) (xy 90.17 87.63)
 		)
@@
 	(wire
 		(pts
+			(xy 38.1 50.8) (xy 44.45 50.8)
+		)
+		(stroke
+			(width 0)
+			(type default)
+		)
+	)
+	(wire
+		(pts
 			(xy 102.87 62.23) (xy 115.57 62.23)
 		)
@@
 	(wire
 		(pts
+			(xy 44.45 50.8) (xy 44.45 62.23)
+		)
+		(stroke
+			(width 0)
+			(type default)
+		)
+	)
+	(wire
+		(pts
 			(xy 58.42 107.95) (xy 58.42 62.23)
 		)
@@
 	(wire
 		(pts
+			(xy 44.45 50.8) (xy 50.8 50.8)
+		)
+		(stroke
+			(width 0)
+			(type default)
+		)
+	)
+	(wire
+		(pts
 			(xy 71.12 64.77) (xy 71.12 62.23)
 		)
@@
 	)
 	(image
-		(at 240.03 83.82)
+		(at 260.35 81.28)
 		(data "iVBORw0KGgoAAAANSUhEUgAAArgAAAGkCAYAAADaPFZSAAAAAXNSR0IArs4c6QAAAARnQU1BAACx"
 			"jwv8YQUAAAAJcEhZcwAADsMAAA7DAcdvqGQAAKTbSURBVHhe7N0HfBNlHwfwX5Kmu3RAN3vvvaEF"
@@
 		)
 	)
+	(global_label "1.65V"
+		(shape input)
+		(at 135.89 107.95 0)
+		(fields_autoplaced yes)
+		(effects
+			(font
+				(size 1.27 1.27)
+			)
+			(justify left)
+		)
+		(property "Intersheetrefs" "${INTERSHEET_REFS}"
+			(at 144.1971 107.95 0)
+			(effects
+				(font
+					(size 1.27 1.27)
+				)
+				(justify left)
+				(hide yes)
+			)
+		)
+	)
+	(symbol
+		(lib_id "power:VBUS")
+		(at 38.1 50.8 90)
+		(unit 1)
+		(exclude_from_sim no)
+		(in_bom yes)
+		(on_board yes)
+		(dnp no)
+		(fields_autoplaced yes)
+		(property "Reference" "#PWR0130"
+			(at 41.91 50.8 0)
+			(effects
+				(font
+					(size 1.27 1.27)
+				)
+				(hide yes)
+			)
+		)
+		(property "Value" "VBUS"
+			(at 34.29 50.7999 90)
+			(effects
+				(font
+					(size 1.27 1.27)
+				)
+				(justify left)
+			)
+		)
+		(property "Footprint" ""
+			(at 38.1 50.8 0)
+			(effects
+				(font
+					(size 1.27 1.27)
+				)
+				(hide yes)
+			)
+		)
+		(property "Datasheet" ""
+			(at 38.1 50.8 0)
+			(effects
+				(font
+					(size 1.27 1.27)
+				)
+				(hide yes)
+			)
+		)
+		(property "Description" "Power symbol creates a global label with name \"VBUS\""
+			(at 38.1 50.8 0)
+			(effects
+				(font
+					(size 1.27 1.27)
+				)
+				(hide yes)
+			)
+		)
+		(pin "1"
+		)
+		(instances
+			(project ""
+				(path "/198ad8d1-66e3-4deb-889c-1af2b81e67c3/11f39170-493e-4ecf-a6ba-aee1374b2ff1"
+					(reference "#PWR0130")
+					(unit 1)
+				)
+			)
+		)
+	)
+	(symbol
+		(lib_id "power:+5V")
+		(at 50.8 50.8 270)
+		(unit 1)
+		(exclude_from_sim no)
+		(in_bom yes)
+		(on_board yes)
+		(dnp no)
+		(fields_autoplaced yes)
+		(property "Reference" "#PWR0131"
+			(at 46.99 50.8 0)
+			(effects
+				(font
+					(size 1.27 1.27)
+				)
+				(hide yes)
+			)
+		)
+		(property "Value" "+5V"
+			(at 54.61 50.7999 90)
+			(effects
+				(font
+					(size 1.27 1.27)
+				)
+				(justify left)
+			)
+		)
+		(property "Footprint" ""
+			(at 50.8 50.8 0)
+			(effects
+				(font
+					(size 1.27 1.27)
+				)
+				(hide yes)
+			)
+		)
+		(property "Datasheet" ""
+			(at 50.8 50.8 0)
+			(effects
+				(font
+					(size 1.27 1.27)
+				)
+				(hide yes)
+			)
+		)
+		(property "Description" "Power symbol creates a global label with name \"+5V\""
+			(at 50.8 50.8 0)
+			(effects
+				(font
+					(size 1.27 1.27)
+				)
+				(hide yes)
+			)
+		)
+		(pin "1"
+		)
+		(instances
+			(project ""
+				(path "/198ad8d1-66e3-4deb-889c-1af2b81e67c3/11f39170-493e-4ecf-a6ba-aee1374b2ff1"
+					(reference "#PWR0131")
+					(unit 1)
+				)
+			)
+		)
+	)
 	(symbol
 		(lib_id "Device:R")
@@
 	)
 	(symbol
-		(lib_id "power:+3.3V")
-		(at 41.91 60.96 0)
-		(unit 1)
-		(exclude_from_sim no)
-		(in_bom yes)
-		(on_board yes)
-		(dnp no)
-		(fields_autoplaced yes)
-		(property "Reference" "#PWR0123"
-			(at 41.91 64.77 0)
-			(effects
-				(font
-					(size 1.27 1.27)
-				)
-				(hide yes)
-			)
-		)
-		(property "Value" "VUSB"
-			(at 41.91 55.88 0)
-			(effects
-				(font
-					(size 1.27 1.27)
-				)
-			)
-		)
-		(property "Footprint" ""
-			(at 41.91 60.96 0)
-			(effects
-				(font
-					(size 1.27 1.27)
-				)
-				(hide yes)
-			)
-		)
-		(property "Datasheet" ""
-			(at 41.91 60.96 0)
-			(effects
-				(font
-					(size 1.27 1.27)
-				)
-				(hide yes)
-			)
-		)
-		(property "Description" "Power symbol creates a global label with name \"+3.3V\""
-			(at 41.91 60.96 0)
-			(effects
-				(font
-					(size 1.27 1.27)
-				)
-				(hide yes)
-			)
-		)
-		(pin "1"
-		)
-		(instances
-			(project "Input Board"
-				(path "/198ad8d1-66e3-4deb-889c-1af2b81e67c3/11f39170-493e-4ecf-a6ba-aee1374b2ff1"
-					(reference "#PWR0123")
-					(unit 1)
-				)
-			)
-		)
-	)
-	(symbol
 		(lib_id "Device:C")
 		(at 71.12 68.58 0)
@@
 	)
 	(symbol
-		(lib_id "power:+3.3V")
-		(at 135.89 106.68 0)
-		(unit 1)
-		(exclude_from_sim no)
-		(in_bom yes)
-		(on_board yes)
-		(dnp no)
-		(fields_autoplaced yes)
-		(property "Reference" "#PWR0121"
-			(at 135.89 110.49 0)
-			(effects
-				(font
-					(size 1.27 1.27)
-				)
-				(hide yes)
-			)
-		)
-		(property "Value" "1.8V"
-			(at 135.89 101.6 0)
-			(effects
-				(font
-					(size 1.27 1.27)
-				)
-			)
-		)
-		(property "Footprint" ""
-			(at 135.89 106.68 0)
-			(effects
-				(font
-					(size 1.27 1.27)
-				)
-				(hide yes)
-			)
-		)
-		(property "Datasheet" ""
-			(at 135.89 106.68 0)
-			(effects
-				(font
-					(size 1.27 1.27)
-				)
-				(hide yes)
-			)
-		)
-		(property "Description" "Power symbol creates a global label with name \"+3.3V\""
-			(at 135.89 106.68 0)
-			(effects
-				(font
-					(size 1.27 1.27)
-				)
-				(hide yes)
-			)
-		)
-		(pin "1"
-		)
-		(instances
-			(project "Input Board"
-				(path "/198ad8d1-66e3-4deb-889c-1af2b81e67c3/11f39170-493e-4ecf-a6ba-aee1374b2ff1"
-					(reference "#PWR0121")
-					(unit 1)
-				)
-			)
-		)
-	)
-	(symbol
 		(lib_id "Device:R")
 		(at 90.17 81.28 0)
@@
 			)
 		)
-		(property "Value" "1k"
+		(property "Value" "768"
 			(at 92.71 128.2699 0)
 			(effects

Commit message: test commit and minor updates
Parts:
- R3: value 768 -> 750
Other:
- note added: "1.65V"
- note removed: "1.8V"
Changed lines of the file:
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@@
 	(generator_version "9.0")
 	(paper "A4")
-	(text "1.8V\n"
+	(text "1.65V\n"
 		(exclude_from_sim no)
 		(at 90.17 97.79 0)
@@
 			)
 		)
-		(property "Value" "768"
+		(property "Value" "750"
 			(at 92.71 128.2699 0)
 			(effects

Commit message: explosion 💥
Parts:
- added C? (x2): 100n, Capacitor_SMD:C_0402_1005Metric, symbol Device:C
- added C? (x2): 1u, Capacitor_SMD:C_0805_2012Metric, symbol Device:C
- added FB2: 120, SamacSys_Parts:BLM31KN102BH1L, symbol Device:FerriteBead
- renumbered C2 to C?, C1 to C?, C3 to C?, C4 to C?, R5 to R?, R2 to R?, R3 to R?, R1 to R?
Connections:
- net 1.65V: now also C?.1, C?.1, FB2.1; no longer C?.1, R?.1, U3.2 (VO)
- net 3.3V: now also FB2.2
- net GND: now reaches C?.2, C?.2, R?.2
- net GND: now also C?.2, C?.2, R?.2, C?.2, C?.2, C?.2, C?.2
- new net: C?.1, FB2.2, R?.1, U3.2 (VO)
- new net VDDA: C?.1, C?.1, FB2.1

Commit message: Modify preamp
Parts:
- added FB2: 120, SamacSys_Parts:BLM31KN102BH1L, symbol Device:FerriteBead
- renumbered FB2 to FB1
Connections:
- net 1.65V: now also FB2.1; no longer FB1.1
- net at C?.1, R?.1, U3.2 (VO): now also FB2.2; no longer FB1.2

Commit message: more fixes
Parts:
- removed FB2: 120, SamacSys_Parts:BLM31KN102BH1L, symbol Device:FerriteBead
- renumbered FB1 to FB2
Connections:
- net 1.65V: now also FB2.1
- net at C?.1, R?.1, U3.2 (VO): now also FB2.2
