File: Input Hardware/PCB/Input Board/power.kicad_sch (KiCad schematic)
At the start: 21 parts, among them U1 LM317_TO-252, U3 LM317_TO-252

Commit message: Fix files idc
Parts:
- C1201, C1202, C1203, C1204: renamed from C?; footprint (none) -> Capacitor_SMD:C_0603_1608Metric
- C1205, C1206: renamed from C?; footprint Capacitor_SMD:C_0402_1005Metric -> Capacitor_SMD:C_0603_1608Metric
- C1207, C1208: renamed from C?; footprint Capacitor_SMD:C_0805_2012Metric -> Capacitor_SMD:C_0603_1608Metric
- FB1201: renamed from FB1; footprint SamacSys_Parts:BLM31KN102BH1L -> Inductor_SMD:L_1206_3216Metric
- FB1202: renamed from FB2; footprint SamacSys_Parts:BLM31KN102BH1L -> Inductor_SMD:L_1206_3216Metric
- R1201, R1202, R1203, R1204: renamed from R?; footprint (none) -> Resistor_SMD:R_0603_1608Metric
- gave numbers to parts that had none: 5
- renumbered U1 to U1201, U3 to U1202

Commit message: sims and other crap
Parts:
- added C?: 100u, Capacitor_SMD:C_Elec_4x5.8, symbol Device:C
Connections:
- net +5V: now also C?.1
- net GND: now also C?.2
Changed lines of the file:
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@@
 	)
 	(junction
+		(at 46.99 62.23)
+		(diameter 0)
+		(color 0 0 0 0)
+	)
+	(junction
 		(at 90.17 120.65)
 		(diameter 0)
@@
 	(wire
 		(pts
+			(xy 46.99 76.2) (xy 46.99 73.66)
+		)
+		(stroke
+			(width 0)
+			(type default)
+		)
+	)
+	(wire
+		(pts
 			(xy 167.64 105.41) (xy 167.64 107.95)
 		)
@@
 	(wire
 		(pts
+			(xy 46.99 62.23) (xy 58.42 62.23)
+		)
+		(stroke
+			(width 0)
+			(type default)
+		)
+	)
+	(wire
+		(pts
+			(xy 46.99 66.04) (xy 46.99 62.23)
+		)
+		(stroke
+			(width 0)
+			(type default)
+		)
+	)
+	(wire
+		(pts
 			(xy 158.75 60.96) (xy 158.75 62.23)
 		)
@@
 	(wire
 		(pts
-			(xy 44.45 62.23) (xy 58.42 62.23)
+			(xy 44.45 62.23) (xy 46.99 62.23)
 		)
 		(stroke
@@
 	)
 	(symbol
+		(lib_name "GND_1")
+		(lib_id "power:GND")
+		(at 46.99 76.2 0)
+		(mirror y)
+		(unit 1)
+		(exclude_from_sim no)
+		(in_bom yes)
+		(on_board yes)
+		(dnp no)
+		(fields_autoplaced yes)
+		(property "Reference" "#PWR089"
+			(at 46.99 82.55 0)
+			(effects
+				(font
+					(size 1.27 1.27)
+				)
+				(hide yes)
+			)
+		)
+		(property "Value" "GND"
+			(at 46.99 81.28 0)
+			(effects
+				(font
+					(size 1.27 1.27)
+				)
+			)
+		)
+		(property "Footprint" ""
+			(at 46.99 76.2 0)
+			(effects
+				(font
+					(size 1.27 1.27)
+				)
+				(hide yes)
+			)
+		)
+		(property "Datasheet" ""
+			(at 46.99 76.2 0)
+			(effects
+				(font
+					(size 1.27 1.27)
+				)
+				(hide yes)
+			)
+		)
+		(property "Description" "Power symbol creates a global label with name \"GND\" , ground"
+			(at 46.99 76.2 0)
+			(effects
+				(font
+					(size 1.27 1.27)
+				)
+				(hide yes)
+			)
+		)
+		(pin "1"
+		)
+		(instances
+			(project "Input Board"
+				(path "/198ad8d1-66e3-4deb-889c-1af2b81e67c3/11f39170-493e-4ecf-a6ba-aee1374b2ff1"
+					(reference "#PWR089")
+					(unit 1)
+				)
+			)
+		)
+	)
+	(symbol
 		(lib_id "power:+3.3V")
 		(at 134.62 60.96 0)
@@
 					(unit 1)
 				)
+			)
+		)
+	)
+	(symbol
+		(lib_id "Device:C")
+		(at 46.99 69.85 0)
+		(unit 1)
+		(exclude_from_sim no)
+		(in_bom yes)
+		(on_board yes)
+		(dnp no)
+		(fields_autoplaced yes)
+		(property "Reference" "C?"
+			(at 50.8 68.5799 0)
+			(effects
+				(font
+					(size 1.27 1.27)
+				)
+				(justify left)
+			)
+		)
+		(property "Value" "100u"
+			(at 50.8 71.1199 0)
+			(effects
+				(font
+					(size 1.27 1.27)
+				)
+				(justify left)
+			)
+		)
+		(property "Footprint" "Capacitor_SMD:C_Elec_4x5.8"
+			(at 47.9552 73.66 0)
+			(effects
+				(font
+					(size 1.27 1.27)
+				)
+				(hide yes)
+			)
+		)
+		(property "Datasheet" "~"
+			(at 46.99 69.85 0)
+			(effects
+				(font
+					(size 1.27 1.27)
+				)
+				(hide yes)
+			)
+		)
+		(property "Description" "Unpolarized capacitor"
+			(at 46.99 69.85 0)
+			(effects
+				(font
+					(size 1.27 1.27)
+				)
+				(hide yes)
+			)
+		)
+		(pin "2"
+		)
+		(pin "1"
+		)
+		(instances
+			(project "Input Board"
+				(path "/198ad8d1-66e3-4deb-889c-1af2b81e67c3/11f39170-493e-4ecf-a6ba-aee1374b2ff1"
+					(reference "C?")
+					(unit 1)
+				)

Commit message: package type change
Parts:
- gave numbers to parts that had none: 1
Changed lines of the file:
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@@
 		(dnp no)
 		(fields_autoplaced yes)
-		(property "Reference" "#PWR089"
+		(property "Reference" "#PWR0137"
 			(at 46.99 82.55 0)
 			(effects
@@
 			(project "Input Board"
 				(path "/198ad8d1-66e3-4deb-889c-1af2b81e67c3/11f39170-493e-4ecf-a6ba-aee1374b2ff1"
-					(reference "#PWR089")
+					(reference "#PWR0137")
 					(unit 1)
 				)
@@
 		(dnp no)
 		(fields_autoplaced yes)
-		(property "Reference" "C?"
+		(property "Reference" "C1"
 			(at 50.8 68.5799 0)
 			(effects
@@
 			(project "Input Board"
 				(path "/198ad8d1-66e3-4deb-889c-1af2b81e67c3/11f39170-493e-4ecf-a6ba-aee1374b2ff1"
-					(reference "C?")
-					(unit 1)
-				)
+					(reference "C1")
+					(unit 1)
+				)

Commit message: Schematic Cleanup
Parts:
- renumbered C1 to C?
Changed lines of the file:
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@@
 		(dnp no)
 		(fields_autoplaced yes)
-		(property "Reference" "#PWR0137"
+		(property "Reference" "#PWR089"
 			(at 46.99 82.55 0)
 			(effects
@@
 			(project "Input Board"
 				(path "/198ad8d1-66e3-4deb-889c-1af2b81e67c3/11f39170-493e-4ecf-a6ba-aee1374b2ff1"
-					(reference "#PWR0137")
+					(reference "#PWR089")
 					(unit 1)
 				)
@@
 		(dnp no)
 		(fields_autoplaced yes)
-		(property "Reference" "C1"
+		(property "Reference" "C?"
 			(at 50.8 68.5799 0)
 			(effects
@@
 			(project "Input Board"
 				(path "/198ad8d1-66e3-4deb-889c-1af2b81e67c3/11f39170-493e-4ecf-a6ba-aee1374b2ff1"
-					(reference "C1")
-					(unit 1)
-				)
+					(reference "C?")
+					(unit 1)
+				)

Commit message: Layout Progress
Parts:
- gave numbers to parts that had none: 1
- renumbered C1201 to C1702, C1202 to C1703, C1203 to C1704, C1204 to C1705, C1205 to C1706, C1206 to C1707, C1207 to C1708, C1208 to C1709, FB1201 to FB1701, FB1202 to FB1702, R1201 to R1701, R1202 to R1702, R1203 to R1703, R1204 to R1704, TP1201 to TP1701, TP1202 to TP1702, TP1203 to TP1703, TP1204 to TP1704, TP1205 to TP1705, U1201 to U1701, U1202 to U1702

Commit message: minor schematic changes and value assignment
Parts:
- added C?: 1u, Capacitor_SMD:C_Elec_4x5.8, symbol Device:C
- added D?: ~, LED_SMD:LED_0603_1608Metric, symbol Device:LED
- added R?: 220, Resistor_SMD:R_0603_1608Metric, symbol Device:R
Connections:
- net +5V: now also C?.1, R?.1
- net GND: now also C?.2, D?.1 (K)
- new net: D?.2 (A), R?.2
Other:
- moved on the sheet: TP1701

Commit message: updates
Parts:
- R?: value 220 -> 180
Changed lines of the file:
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@@
 			)
 		)
-		(property "Value" "220"
+		(property "Value" "180"
 			(at 30.48 97.7899 0)
 			(effects

Commit message: changes
Parts:
- gave numbers to parts that had none: 3
Changed lines of the file:
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@@
 		(dnp no)
 		(fields_autoplaced yes)
-		(property "Reference" "R?"
+		(property "Reference" "R4"
 			(at 30.48 95.2499 0)
 			(effects
@@
 			(project "Input Board"
 				(path "/198ad8d1-66e3-4deb-889c-1af2b81e67c3/11f39170-493e-4ecf-a6ba-aee1374b2ff1"
-					(reference "R?")
+					(reference "R4")
 					(unit 1)
 				)
@@
 		(dnp no)
 		(fields_autoplaced yes)
-		(property "Reference" "D?"
+		(property "Reference" "D1"
 			(at 30.48 105.7274 90)
 			(effects
@@
 			(project "Input Board"
 				(path "/198ad8d1-66e3-4deb-889c-1af2b81e67c3/11f39170-493e-4ecf-a6ba-aee1374b2ff1"
-					(reference "D?")
+					(reference "D1")
 					(unit 1)
 				)
@@
 		(dnp no)
 		(fields_autoplaced yes)
-		(property "Reference" "C?"
+		(property "Reference" "C4"
 			(at 39.37 68.5799 0)
 			(effects
@@
 			(project "Input Board"
 				(path "/198ad8d1-66e3-4deb-889c-1af2b81e67c3/11f39170-493e-4ecf-a6ba-aee1374b2ff1"
-					(reference "C?")
-					(unit 1)
-				)
+					(reference "C4")
+					(unit 1)
+				)
