File: Input Hardware/PCB/Input Board/mux.kicad_sch (KiCad schematic)
At the start: 2 parts

Commit message: Progress
Parts:
- added C?: 100n, Capacitor_SMD:C_0603_1608Metric, symbol Device:C
- added U (x5): MCP6499, Package_SO:SOIC-14_3.9x8.7mm_P1.27mm, symbol Device:Opamp_Quad
Connections:
- net +5V: now also C?.1
- new net GNDA: C?.2

Commit message: said hello
Parts:
- renumbered U to U?
Changed lines of the file:
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@@
 		(dnp no)
 		(fields_autoplaced yes)
-		(property "Reference" "U"
+		(property "Reference" "U?"
 			(at 114.3 53.34 0)
 			(effects
@@
 			(project ""
 				(path "/198ad8d1-66e3-4deb-889c-1af2b81e67c3/0fc095cc-6ee6-4117-a537-6519c9828b80"
+					(reference "U?")
+					(unit 1)
+				)
+				(path "/198ad8d1-66e3-4deb-889c-1af2b81e67c3/908995ee-e872-4b00-89ed-692dff603043"
+					(reference "U?")
+					(unit 1)
+				)
+				(path "/198ad8d1-66e3-4deb-889c-1af2b81e67c3/be7b6b67-fb63-4121-a158-51987fefa9a9"
+					(reference "U?")
+					(unit 1)
+				)
+				(path "/198ad8d1-66e3-4deb-889c-1af2b81e67c3/bf2971a4-4e8b-460e-806a-6c5050f52bee"
 					(reference "U?")
 					(unit 1)
@@
 		(dnp no)
 		(fields_autoplaced yes)
-		(property "Reference" "U"
+		(property "Reference" "U?"
 			(at 166.37 53.34 0)
 			(effects
@@
 					(reference "U?")
 					(unit 3)
+				)
+				(path "/198ad8d1-66e3-4deb-889c-1af2b81e67c3/908995ee-e872-4b00-89ed-692dff603043"
+					(reference "U?")
+					(unit 1)
+				)
+				(path "/198ad8d1-66e3-4deb-889c-1af2b81e67c3/be7b6b67-fb63-4121-a158-51987fefa9a9"
+					(reference "U?")
+					(unit 1)
+				)
+				(path "/198ad8d1-66e3-4deb-889c-1af2b81e67c3/bf2971a4-4e8b-460e-806a-6c5050f52bee"
+					(reference "U?")
+					(unit 1)
 				)
 			)
@@
 		(dnp no)
 		(fields_autoplaced yes)
-		(property "Reference" "U"
+		(property "Reference" "U?"
 			(at 184.15 53.34 0)
 			(effects
@@
 					(reference "U?")
 					(unit 4)
+				)
+				(path "/198ad8d1-66e3-4deb-889c-1af2b81e67c3/908995ee-e872-4b00-89ed-692dff603043"
+					(reference "U?")
+					(unit 1)
+				)
+				(path "/198ad8d1-66e3-4deb-889c-1af2b81e67c3/be7b6b67-fb63-4121-a158-51987fefa9a9"
+					(reference "U?")
+					(unit 1)
+				)
+				(path "/198ad8d1-66e3-4deb-889c-1af2b81e67c3/bf2971a4-4e8b-460e-806a-6c5050f52bee"
+					(reference "U?")
+					(unit 1)
 				)
 			)
@@
 		(dnp no)
 		(fields_autoplaced yes)
-		(property "Reference" "U"
+		(property "Reference" "U?"
 			(at 39.37 170.1799 0)
 			(effects
@@
 					(reference "U?")
 					(unit 5)
+				)
+				(path "/198ad8d1-66e3-4deb-889c-1af2b81e67c3/908995ee-e872-4b00-89ed-692dff603043"
+					(reference "U?")
+					(unit 1)
+				)
+				(path "/198ad8d1-66e3-4deb-889c-1af2b81e67c3/be7b6b67-fb63-4121-a158-51987fefa9a9"
+					(reference "U?")
+					(unit 1)
+				)
+				(path "/198ad8d1-66e3-4deb-889c-1af2b81e67c3/bf2971a4-4e8b-460e-806a-6c5050f52bee"
+					(reference "U?")
+					(unit 1)
 				)
 			)
@@
 		(dnp no)
 		(fields_autoplaced yes)
-		(property "Reference" "U"
+		(property "Reference" "U?"
 			(at 139.7 53.34 0)
 			(effects
@@
 					(unit 2)
 				)
-			)
+				(path "/198ad8d1-66e3-4deb-889c-1af2b81e67c3/908995ee-e872-4b00-89ed-692dff603043"
+					(reference "U?")
+					(unit 1)
+				)
+				(path "/198ad8d1-66e3-4deb-889c-1af2b81e67c3/be7b6b67-fb63-4121-a158-51987fefa9a9"
+					(reference "U?")
+					(unit 1)
+				)
+				(path "/198ad8d1-66e3-4deb-889c-1af2b81e67c3/bf2971a4-4e8b-460e-806a-6c5050f52bee"
+					(reference "U?")
+					(unit 1)
+				)
+			)

Commit message: Reminder
Other:
- note added: "include pulldown"
Changed lines of the file:
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@@
 	(generator_version "9.0")
 	(paper "A4")
+	(text "include pulldown"
+		(exclude_from_sim no)
+		(at 80.01 53.34 0)
+		(effects
+			(font
+				(size 1.27 1.27)
+			)
+			(justify left bottom)
+		)
+	)
 	(junction
 		(at 44.45 179.07)

Commit message: integrate
Connections:
- net +5V renamed +3.3V
Changed lines of the file:
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@@
 	)
 	(junction
-		(at 38.1 163.83)
+		(at 44.45 163.83)
 		(diameter 0)
 		(color 0 0 0 0)
@@
 	(wire
 		(pts
-			(xy 44.45 179.07) (xy 50.8 179.07)
+			(xy 25.4 165.1) (xy 25.4 167.64)
 		)
 		(stroke
@@
 	(wire
 		(pts
-			(xy 25.4 165.1) (xy 25.4 167.64)
+			(xy 44.45 179.07) (xy 50.8 179.07)
 		)
 		(stroke
@@
 	(wire
 		(pts
-			(xy 50.8 163.83) (xy 38.1 163.83)
+			(xy 38.1 163.83) (xy 44.45 163.83)
+		)
+		(stroke
+			(width 0)
+			(type default)
+		)
+	)
+	(wire
+		(pts
+			(xy 44.45 163.83) (xy 50.8 163.83)
 		)
 		(stroke
@@
 			)
 			(justify right)
-		)
-	)
-	(symbol
-		(lib_id "power:+5V")
-		(at 45.72 45.72 0)
-		(unit 1)
-		(exclude_from_sim no)
-		(in_bom yes)
-		(on_board yes)
-		(dnp no)
-		(property "Reference" "#PWR037"
-			(at 45.72 49.53 0)
-			(effects
-				(font
-					(size 1.27 1.27)
-				)
-				(hide yes)
-			)
-		)
-		(property "Value" "+5V"
-			(at 45.72 41.91 0)
-			(effects
-				(font
-					(size 1.27 1.27)
-				)
-			)
-		)
-		(property "Footprint" ""
-			(at 45.72 45.72 0)
-			(effects
-				(font
-					(size 1.27 1.27)
-				)
-				(hide yes)
-			)
-		)
-		(property "Datasheet" ""
-			(at 45.72 45.72 0)
-			(effects
-				(font
-					(size 1.27 1.27)
-				)
-				(hide yes)
-			)
-		)
-		(property "Description" "Power symbol creates a global label with name \"+5V\""
-			(at 45.72 45.72 0)
-			(effects
-				(font
-					(size 1.27 1.27)
-				)
-				(hide yes)
-			)
-		)
-		(pin "1"
-		)
-		(instances
-			(project "Input Board"
-				(path "/198ad8d1-66e3-4deb-889c-1af2b81e67c3/0fc095cc-6ee6-4117-a537-6519c9828b80"
-					(reference "#PWR043")
-					(unit 1)
-				)
-				(path "/198ad8d1-66e3-4deb-889c-1af2b81e67c3/908995ee-e872-4b00-89ed-692dff603043"
-					(reference "#PWR047")
-					(unit 1)
-				)
-				(path "/198ad8d1-66e3-4deb-889c-1af2b81e67c3/be7b6b67-fb63-4121-a158-51987fefa9a9"
-					(reference "#PWR037")
-					(unit 1)
-				)
-				(path "/198ad8d1-66e3-4deb-889c-1af2b81e67c3/bf2971a4-4e8b-460e-806a-6c5050f52bee"
-					(reference "#PWR041")
-					(unit 1)
-				)
-			)
 		)
 	)
@@
 				(path "/198ad8d1-66e3-4deb-889c-1af2b81e67c3/bf2971a4-4e8b-460e-806a-6c5050f52bee"
 					(reference "U?")
-					(unit 1)
+					(unit 3)
 				)
 			)
@@
 				(path "/198ad8d1-66e3-4deb-889c-1af2b81e67c3/bf2971a4-4e8b-460e-806a-6c5050f52bee"
 					(reference "U?")
-					(unit 1)
+					(unit 4)
 				)
 			)
@@
 				(path "/198ad8d1-66e3-4deb-889c-1af2b81e67c3/bf2971a4-4e8b-460e-806a-6c5050f52bee"
 					(reference "U?")
-					(unit 1)
+					(unit 5)
 				)
 			)
@@
 	)
 	(symbol
-		(lib_id "power:+5V")
+		(lib_id "power:+3.3V")
+		(at 45.72 45.72 0)
+		(unit 1)
+		(exclude_from_sim no)
+		(in_bom yes)
+		(on_board yes)
+		(dnp no)
+		(fields_autoplaced yes)
+		(property "Reference" "#PWR037"
+			(at 45.72 49.53 0)
+			(effects
+				(font
+					(size 1.27 1.27)
+				)
+				(hide yes)
+			)
+		)
+		(property "Value" "+3.3V"
+			(at 45.72 40.64 0)
+			(effects
+				(font
+					(size 1.27 1.27)
+				)
+			)
+		)
+		(property "Footprint" ""
+			(at 45.72 45.72 0)
+			(effects
+				(font
+					(size 1.27 1.27)
+				)
+				(hide yes)
+			)
+		)
+		(property "Datasheet" ""
+			(at 45.72 45.72 0)
+			(effects
+				(font
+					(size 1.27 1.27)
+				)
+				(hide yes)
+			)
+		)
+		(property "Description" "Power symbol creates a global label with name \"+3.3V\""
+			(at 45.72 45.72 0)
+			(effects
+				(font
+					(size 1.27 1.27)
+				)
+				(hide yes)
+			)
+		)
+		(pin "1"
+		)
+		(instances
+			(project ""
+				(path "/198ad8d1-66e3-4deb-889c-1af2b81e67c3/0fc095cc-6ee6-4117-a537-6519c9828b80"
+					(reference "#PWR047")
+					(unit 1)
+				)
+				(path "/198ad8d1-66e3-4deb-889c-1af2b81e67c3/908995ee-e872-4b00-89ed-692dff603043"
+					(reference "#PWR043")
+					(unit 1)
+				)
+				(path "/198ad8d1-66e3-4deb-889c-1af2b81e67c3/be7b6b67-fb63-4121-a158-51987fefa9a9"
+					(reference "#PWR037")
+					(unit 1)
+				)
+				(path "/198ad8d1-66e3-4deb-889c-1af2b81e67c3/bf2971a4-4e8b-460e-806a-6c5050f52bee"
+					(reference "#PWR041")
+					(unit 1)
+				)
+			)
+		)
+	)
+	(symbol
+		(lib_id "power:+3.3V")
 		(at 25.4 165.1 0)
 		(unit 1)
@@
 			)
 		)
-		(property "Value" "+5V"
+		(property "Value" "+3.3V"
 			(at 25.4 160.02 0)
 			(effects
@@
 			)
 		)
-		(property "Description" "Power symbol creates a global label with name \"+5V\""
+		(property "Description" "Power symbol creates a global label with name \"+3.3V\""
 			(at 25.4 165.1 0)
 			(effects
@@
 			(project "Input Board"
 				(path "/198ad8d1-66e3-4deb-889c-1af2b81e67c3/0fc095cc-6ee6-4117-a537-6519c9828b80"
-					(reference "#PWR035")
+					(reference "#PWR045")
 					(unit 1)
 				)
 				(path "/198ad8d1-66e3-4deb-889c-1af2b81e67c3/908995ee-e872-4b00-89ed-692dff603043"
-					(reference "#PWR045")
+					(reference "#PWR039")
 					(unit 1)
 				)
@@
 				)
 				(path "/198ad8d1-66e3-4deb-889c-1af2b81e67c3/bf2971a4-4e8b-460e-806a-6c5050f52bee"
-					(reference "#PWR039")
+					(reference "#PWR035")
 					(unit 1)
 				)
@@
 				(path "/198ad8d1-66e3-4deb-889c-1af2b81e67c3/bf2971a4-4e8b-460e-806a-6c5050f52bee"
 					(reference "U?")
-					(unit 1)
+					(unit 2)
 				)
 			)
@@
 	)
 	(symbol
-		(lib_id "power:+5V")
-		(at 38.1 163.83 0)
+		(lib_id "power:+3.3V")
+		(at 44.45 163.83 0)
 		(unit 1)
 		(exclude_from_sim no)
@@
 		(fields_autoplaced yes)
 		(property "Reference" "#PWR053"
-			(at 38.1 167.64 0)
-			(effects
-				(font
-					(size 1.27 1.27)
-				)
-				(hide yes)
-			)
-		)
-		(property "Value" "+5V"
-			(at 38.1 158.75 0)
+			(at 44.45 167.64 0)
+			(effects
+				(font
+					(size 1.27 1.27)
+				)
+				(hide yes)
+			)
+		)
+		(property "Value" "+3.3V"
+			(at 44.45 158.75 0)
 			(effects
 				(font
@@
 		)
 		(property "Footprint" ""
-			(at 38.1 163.83 0)
+			(at 44.45 163.83 0)
 			(effects
 				(font
@@
 		)
 		(property "Datasheet" ""
-			(at 38.1 163.83 0)
-			(effects
-				(font
-					(size 1.27 1.27)
-				)
-				(hide yes)
-			)
-		)
-		(property "Description" "Power symbol creates a global label with name \"+5V\""
-			(at 38.1 163.83 0)
-			(effects
-				(font
+			(at 44.45 163.83 0)
+			(effects
+				(font
+					(size 1.27 1.27)
+				)
+				(hide yes)
+			)
+		)
+		(property "Description" "Power symbol creates a global label with name \"+3.3V\""
+			(at 44.45 163.83 0)
+			(effects
+				(font

Commit message: explosion 💥
Parts:
- removed U? (x5): MCP6499, Package_SO:SOIC-14_3.9x8.7mm_P1.27mm, symbol Device:Opamp_Quad
- added IC?: TLV3544IDR, SOIC127P600X175-14N, symbol TLV3544IDR:TLV3544IDR
Other:
- note added: "pulldown for what? X?"

Commit message: fodda
Other:
- moved on the sheet: IC?
Changed lines of the file:
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@@
 	(symbol
 		(lib_id "TLV3544IDR:TLV3544IDR")
-		(at 104.14 57.15 0)
+		(at 104.14 54.61 0)
 		(unit 1)
 		(exclude_from_sim no)
@@
 		(fields_autoplaced yes)
 		(property "Reference" "IC?"
+			(at 119.38 46.99 0)
+			(effects
+				(font
+					(size 1.27 1.27)
+				)
+			)
+		)
+		(property "Value" "TLV3544IDR"
 			(at 119.38 49.53 0)
 			(effects
@@
 			)
 		)
-		(property "Value" "TLV3544IDR"
-			(at 119.38 52.07 0)
-			(effects
-				(font
-					(size 1.27 1.27)
-				)
-			)
-		)
 		(property "Footprint" "SOIC127P600X175-14N"
-			(at 130.81 152.07 0)
+			(at 130.81 149.53 0)
 			(effects
 				(font
@@
 		)
 		(property "Datasheet" "http://www.ti.com/lit/gpn/tlv3544"
-			(at 130.81 252.07 0)
+			(at 130.81 249.53 0)
 			(effects
 				(font
@@
 		)
 		(property "Description" "TLV354x 200MHz, RRIO, CMOS Operational Amplifier"
-			(at 104.14 57.15 0)
+			(at 104.14 54.61 0)
 			(effects
 				(font
@@
 		)
 		(property "Height" "1.75"
-			(at 130.81 452.07 0)
+			(at 130.81 449.53 0)
 			(effects
 				(font
@@
 		)
 		(property "Mouser Part Number" "595-TLV3544IDR"
-			(at 130.81 552.07 0)
+			(at 130.81 549.53 0)
 			(effects
 				(font
@@
 		)
 		(property "Mouser Price/Stock" "https://www.mouser.co.uk/ProductDetail/Texas-Instruments/TLV3544IDR/?qs=9lcNTSmDlCpphxOg9cZfNA%3D%3D"
-			(at 130.81 652.07 0)
+			(at 130.81 649.53 0)
 			(effects
 				(font
@@
 		)
 		(property "Manufacturer_Name" "Texas Instruments"
-			(at 130.81 752.07 0)
+			(at 130.81 749.53 0)
 			(effects
 				(font
@@
 		)
 		(property "Manufacturer_Part_Number" "TLV3544IDR"
-			(at 130.81 852.07 0)
+			(at 130.81 849.53 0)
 			(effects
 				(font
@@
 		)
 		(instances
-			(project ""
+			(project "Input Board"
+				(path "/198ad8d1-66e3-4deb-889c-1af2b81e67c3/0fc095cc-6ee6-4117-a537-6519c9828b80"
+					(reference "IC?")
+					(unit 1)
+				)
+				(path "/198ad8d1-66e3-4deb-889c-1af2b81e67c3/908995ee-e872-4b00-89ed-692dff603043"
+					(reference "IC?")
+					(unit 1)
+				)
 				(path "/198ad8d1-66e3-4deb-889c-1af2b81e67c3/be7b6b67-fb63-4121-a158-51987fefa9a9"
 					(reference "IC?")
 					(unit 1)
+				)
+				(path "/198ad8d1-66e3-4deb-889c-1af2b81e67c3/bf2971a4-4e8b-460e-806a-6c5050f52bee"
+					(reference "IC?")
+					(unit 1)
