File: Input Hardware/PCB/Input Board/display.kicad_sch (KiCad schematic)
At the start: 10 parts

Commit message: adc bandpass amp and rootpage update
Parts:
- removed C? (x4): 1u, Capacitor_SMD:C_0603_1608Metric, symbol Device:C
- removed C? (x2): 2.2u, Capacitor_SMD:C_0603_1608Metric, symbol Device:C
- removed J?: 1.71" SSD1312 OLED, symbol Connector_Generic:Conn_01x16
- removed R? (x2): 10k, Resistor_SMD:R_0603_1608Metric, symbol Device:R
- removed R?: 550k, Resistor_SMD:R_0603_1608Metric, symbol Device:R
Other:
- note removed: "A0 (ADDRESS SELECITON)"
- note removed: "C1N"
- note removed: "C1P"
- note removed: "C2N"
- note removed: "C2P"
- note removed: "CS"
- note removed: "IM1 (BS[1])"
- note removed: "IREF"
- note removed: "SCL"
- note removed: "SI"
- note removed: "VCOMH"
- note removed: "VDD1"
- note removed: "VDD2"
- note removed: "VPP (VCC?)"
- note removed: "VSS"
- note removed: "check IM1 definition"
- note removed: "check VPP definition"
- note removed: "~{RES}"

Commit message: Display first attempt
Parts:
- added C? (x4): 1u, Capacitor_SMD:C_0603_1608Metric, symbol Device:C
- added C? (x2): 2.2u, Capacitor_SMD:C_0603_1608Metric, symbol Device:C
- added J?: 1.71" SSD1312 OLED, symbol Connector_Generic:Conn_01x16
- added R? (x2): 10k, Resistor_SMD:R_0603_1608Metric, symbol Device:R
- added R?: 550k, Resistor_SMD:R_0603_1608Metric, symbol Device:R
Connections:
- new net: C?.1, J?.4 (Pin_4)
- new net: C?.2, J?.3 (Pin_3)
- new net: C?.1, J?.6 (Pin_6)
- new net: C?.1, J?.7 (Pin_7)
- new net: C?.2, J?.1 (Pin_1)
- new net: C?.1, J?.2 (Pin_2)
- new net: J?.8 (Pin_8), R?.2
- new net +3.3V: C?.1, C?.1, J?.10 (Pin_10), J?.13 (Pin_13), J?.14 (Pin_14), J?.5 (Pin_5), R?.1, R?.1
- new net GND: C?.2, C?.2, C?.2, C?.2, J?.11 (Pin_11), J?.12 (Pin_12), J?.9 (Pin_9), R?.1
- new net OLED_SCL: J?.15 (Pin_15), R?.2
- new net OLED_SDA: J?.16 (Pin_16), R?.2
Other:
- note added: "A0 (ADDRESS SELECITON)"
- note added: "C1N"
- note added: "C1P"
- note added: "C2N"
- note added: "C2P"
- note added: "CS"
- note added: "IM1 (BS[1])"
- note added: "IREF"
- note added: "SCL"
- note added: "SI"
- note added: "VCOMH"
- note added: "VDD1"
- note added: "VDD2"
- note added: "VPP (VCC?)"
- note added: "VSS"
- note added: "check IM1 definition"
- note added: "check VPP definition"
- note added: "~{RES}"
