File: Input Hardware/PCB/Input Board/display.kicad_sch (KiCad schematic)
At the start: 10 parts, among them J1301 1.71" SSD1312 OLED

Commit message: Layout Progress
Parts:
- renumbered C1301 to C1601, C1302 to C1602, C1303 to C1603, C1304 to C1604, C1305 to C1605, C1306 to C1606, J1301 to J1601, R1301 to R1601, R1302 to R1602, R1303 to R1603
Changed lines of the file:
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@@
 		(dnp no)
 		(fields_autoplaced yes)
-		(property "Reference" "C1301"
+		(property "Reference" "C1601"
 			(at 67.31 113.0299 0)
 			(effects
@@
 			(project ""
 				(path "/198ad8d1-66e3-4deb-889c-1af2b81e67c3/c7ca0110-3f74-4b47-9986-2317814e0c37"
-					(reference "C1301")
+					(reference "C1601")
 					(unit 1)
 				)
@@
 		(dnp no)
 		(fields_autoplaced yes)
-		(property "Reference" "#PWR01302"
+		(property "Reference" "#PWR01602"
 			(at 127 127 0)
 			(effects
@@
 			(project "Input Board"
 				(path "/198ad8d1-66e3-4deb-889c-1af2b81e67c3/c7ca0110-3f74-4b47-9986-2317814e0c37"
-					(reference "#PWR01302")
+					(reference "#PWR01602")
 					(unit 1)
 				)
@@
 		(dnp no)
 		(fields_autoplaced yes)
-		(property "Reference" "R1301"
+		(property "Reference" "R1601"
 			(at 97.79 68.5799 0)
 			(effects
@@
 			(project "Input Board"
 				(path "/198ad8d1-66e3-4deb-889c-1af2b81e67c3/c7ca0110-3f74-4b47-9986-2317814e0c37"
-					(reference "R1301")
+					(reference "R1601")
 					(unit 1)
 				)
@@
 		(on_board yes)
 		(dnp no)
-		(property "Reference" "C1305"
+		(property "Reference" "C1605"
 			(at 146.05 54.61 90)
 			(effects
@@
 			(project "Input Board"
 				(path "/198ad8d1-66e3-4deb-889c-1af2b81e67c3/c7ca0110-3f74-4b47-9986-2317814e0c37"
-					(reference "C1305")
+					(reference "C1605")
 					(unit 1)
 				)
@@
 		(dnp no)
 		(fields_autoplaced yes)
-		(property "Reference" "C1302"
+		(property "Reference" "C1602"
 			(at 80.01 113.0299 0)
 			(effects
@@
 			(project "Input Board"
 				(path "/198ad8d1-66e3-4deb-889c-1af2b81e67c3/c7ca0110-3f74-4b47-9986-2317814e0c37"
-					(reference "C1302")
+					(reference "C1602")
 					(unit 1)
 				)
@@
 		(dnp no)
 		(fields_autoplaced yes)
-		(property "Reference" "R1303"
+		(property "Reference" "R1603"
 			(at 110.49 68.5799 0)
 			(effects
@@
 			(project ""
 				(path "/198ad8d1-66e3-4deb-889c-1af2b81e67c3/c7ca0110-3f74-4b47-9986-2317814e0c37"
-					(reference "R1303")
+					(reference "R1603")
 					(unit 1)
 				)
@@
 		(dnp no)
 		(fields_autoplaced yes)
-		(property "Reference" "C1303"
+		(property "Reference" "C1603"
 			(at 92.71 113.0299 0)
 			(effects
@@
 			(project "Input Board"
 				(path "/198ad8d1-66e3-4deb-889c-1af2b81e67c3/c7ca0110-3f74-4b47-9986-2317814e0c37"
-					(reference "C1303")
+					(reference "C1603")
 					(unit 1)
 				)
@@
 		(dnp no)
 		(fields_autoplaced yes)
-		(property "Reference" "#PWR01301"
+		(property "Reference" "#PWR01601"
 			(at 127 54.61 0)
 			(effects
@@
 			(project ""
 				(path "/198ad8d1-66e3-4deb-889c-1af2b81e67c3/c7ca0110-3f74-4b47-9986-2317814e0c37"
-					(reference "#PWR01301")
+					(reference "#PWR01601")
 					(unit 1)
 				)
@@
 		(dnp no)
 		(fields_autoplaced yes)
-		(property "Reference" "J1301"
+		(property "Reference" "J1601"
 			(at 180.34 88.8999 0)
 			(effects
@@
 			(project ""
 				(path "/198ad8d1-66e3-4deb-889c-1af2b81e67c3/c7ca0110-3f74-4b47-9986-2317814e0c37"
-					(reference "J1301")
+					(reference "J1601")
 					(unit 1)
 				)
@@
 		(on_board yes)
 		(dnp no)
-		(property "Reference" "C1306"
+		(property "Reference" "C1606"
 			(at 158.75 54.6099 90)
 			(effects
@@
 			(project "Input Board"
 				(path "/198ad8d1-66e3-4deb-889c-1af2b81e67c3/c7ca0110-3f74-4b47-9986-2317814e0c37"
-					(reference "C1306")
+					(reference "C1606")
 					(unit 1)
 				)
@@
 		(dnp no)
 		(fields_autoplaced yes)
-		(property "Reference" "C1304"
+		(property "Reference" "C1604"
 			(at 130.81 113.0299 0)
 			(effects
@@
 			(project "Input Board"
 				(path "/198ad8d1-66e3-4deb-889c-1af2b81e67c3/c7ca0110-3f74-4b47-9986-2317814e0c37"
-					(reference "C1304")
+					(reference "C1604")
 					(unit 1)
 				)
@@
 		(on_board yes)
 		(dnp no)
-		(property "Reference" "R1302"
+		(property "Reference" "R1602"
 			(at 104.14 113.03 0)
 			(effects
@@
 			(project ""
 				(path "/198ad8d1-66e3-4deb-889c-1af2b81e67c3/c7ca0110-3f74-4b47-9986-2317814e0c37"
-					(reference "R1302")
-					(unit 1)
-				)
+					(reference "R1602")
+					(unit 1)
+				)

Commit message: minor cosmetic
Other:
- note removed: "A0 (ADDRESS SELECITON)"
- note removed: "C1N"
- note removed: "C1P"
- note removed: "C2N"
- note removed: "C2P"
- note removed: "CS"
- note removed: "IM1 (BS[1])"
- note removed: "IREF"
- note removed: "SCL"
- note removed: "SI"
- note removed: "VCOMH"
- note removed: "VDD1"
- note removed: "VDD2"
- note removed: "VPP (VCC?)"
- note removed: "VSS"
- note removed: "check IM1 definition"
- note removed: "check VPP definition"
- note removed: "https://www.aliexpress.com/item/1005006387603619.html"
- note removed: "~{RES}"
Changed lines of the file:
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@@
 	(generator_version "9.0")
 	(paper "A4")
-	(text "~{RES}"
-		(exclude_from_sim no)
-		(at 171.45 101.6 0)
-		(effects
-			(font
-				(size 1.27 1.27)
-			)
-			(justify right bottom)
-		)
-	)
-	(text "C1P"
-		(exclude_from_sim no)
-		(at 171.45 73.66 0)
-		(effects
-			(font
-				(size 1.27 1.27)
-			)
-			(justify right bottom)
-		)
-	)
-	(text "C2P"
-		(exclude_from_sim no)
-		(at 171.45 76.2 0)
-		(effects
-			(font
-				(size 1.27 1.27)
-			)
-			(justify right bottom)
-		)
-	)
-	(text "check VPP definition\n"
-		(exclude_from_sim no)
-		(at 144.78 83.82 0)
-		(effects
-			(font
-				(size 1.27 1.27)
-			)
-			(justify bottom)
-		)
-	)
-	(text "VPP (VCC?)"
-		(exclude_from_sim no)
-		(at 171.45 83.82 0)
-		(effects
-			(font
-				(size 1.27 1.27)
-			)
-			(justify right bottom)
-		)
-	)
-	(text "CS"
-		(exclude_from_sim no)
-		(at 171.45 96.52 0)
-		(effects
-			(font
-				(size 1.27 1.27)
-			)
-			(justify right bottom)
-		)
-	)
-	(text "https://www.aliexpress.com/item/1005006387603619.html\n"
-		(exclude_from_sim no)
-		(at 176.53 135.89 0)
-		(effects
-			(font
-				(size 1.27 1.27)
-			)
-		)
-	)
-	(text "check IM1 definition\n"
-		(exclude_from_sim no)
-		(at 143.3743 93.98 0)
-		(effects
-			(font
-				(size 1.27 1.27)
-			)
-			(justify bottom)
-		)
-	)
-	(text "C1N"
-		(exclude_from_sim no)
-		(at 171.45 71.12 0)
-		(effects
-			(font
-				(size 1.27 1.27)
-			)
-			(justify right bottom)
-		)
-	)
-	(text "IREF"
-		(exclude_from_sim no)
-		(at 171.45 88.9 0)
-		(effects
-			(font
-				(size 1.27 1.27)
-			)
-			(justify right bottom)
-		)
-	)
-	(text "VSS"
-		(exclude_from_sim no)
-		(at 171.45 91.44 0)
-		(effects
-			(font
-				(size 1.27 1.27)
-			)
-			(justify right bottom)
-		)
-	)
-	(text "SCL"
-		(exclude_from_sim no)
-		(at 171.45 106.68 0)
-		(effects
-			(font
-				(size 1.27 1.27)
-			)
-			(justify right bottom)
-		)
-	)
-	(text "VDD1"
-		(exclude_from_sim no)
-		(at 171.45 104.14 0)
-		(effects
-			(font
-				(size 1.27 1.27)
-			)
-			(justify right bottom)
-		)
-	)
-	(text "VDD2"
-		(exclude_from_sim no)
-		(at 171.45 81.28 0)
-		(effects
-			(font
-				(size 1.27 1.27)
-			)
-			(justify right bottom)
-		)
-	)
-	(text "A0 (ADDRESS SELECITON)"
-		(exclude_from_sim no)
-		(at 171.45 99.06 0)
-		(effects
-			(font
-				(size 1.27 1.27)
-			)
-			(justify right bottom)
-		)
-	)
-	(text "IM1 (BS[1])"
-		(exclude_from_sim no)
-		(at 171.45 93.98 0)
-		(effects
-			(font
-				(size 1.27 1.27)
-			)
-			(justify right bottom)
-		)
-	)
-	(text "VCOMH"
-		(exclude_from_sim no)
-		(at 171.45 86.36 0)
-		(effects
-			(font
-				(size 1.27 1.27)
-			)
-			(justify right bottom)
-		)
-	)
-	(text "SI"
-		(exclude_from_sim no)
-		(at 171.45 109.22 0)
-		(effects
-			(font
-				(size 1.27 1.27)
-			)
-			(justify right bottom)
-		)
-	)
-	(text "C2N"
-		(exclude_from_sim no)
-		(at 171.45 78.74 0)
-		(effects
-			(font
-				(size 1.27 1.27)
-			)
-			(justify right bottom)
-		)
-	)
 	(junction
 		(at 95.25 109.22)
@@
 	(wire
 		(pts
-			(xy 172.72 73.66) (xy 154.94 73.66)
+			(xy 172.72 73.66) (xy 153.67 73.66)
 		)
 		(stroke
@@
 	(wire
 		(pts
+			(xy 163.83 63.5) (xy 162.56 63.5)
+		)
+		(stroke
+			(width 0)
+			(type default)
+		)
+	)
+	(wire
+		(pts
 			(xy 127 110.49) (xy 127 104.14)
 		)
@@
 	(wire
 		(pts
+			(xy 151.13 63.5) (xy 149.86 63.5)
+		)
+		(stroke
+			(width 0)
+			(type default)
+		)
+	)
+	(wire
+		(pts
 			(xy 57.15 106.68) (xy 107.95 106.68)
 		)
@@
 	(wire
 		(pts
-			(xy 162.56 71.12) (xy 172.72 71.12)
+			(xy 163.83 71.12) (xy 172.72 71.12)
+		)
+		(stroke
+			(width 0)
+			(type default)
+		)
+	)
+	(wire
+		(pts
+			(xy 153.67 63.5) (xy 154.94 63.5)
 		)
 		(stroke
@@
 	(wire
 		(pts
-			(xy 142.24 78.74) (xy 142.24 63.5)
-		)
-		(stroke
-			(width 0)
-			(type default)
-		)
-	)
-	(wire
-		(pts
-			(xy 149.86 76.2) (xy 172.72 76.2)
+			(xy 140.97 78.74) (xy 140.97 63.5)
+		)
+		(stroke
+			(width 0)
+			(type default)
+		)
+	)
+	(wire
+		(pts
+			(xy 151.13 76.2) (xy 172.72 76.2)
 		)
 		(stroke
@@
 	(wire
 		(pts
-			(xy 172.72 78.74) (xy 142.24 78.74)
+			(xy 172.72 78.74) (xy 140.97 78.74)
 		)
 		(stroke
@@
 	(wire
 		(pts
-			(xy 149.86 63.5) (xy 149.86 76.2)
-		)
-		(stroke
-			(width 0)
-			(type default)
-		)
-	)
-	(wire
-		(pts
-			(xy 154.94 73.66) (xy 154.94 63.5)
+			(xy 151.13 63.5) (xy 151.13 76.2)
+		)
+		(stroke
+			(width 0)
+			(type default)
+		)
+	)
+	(wire
+		(pts
+			(xy 153.67 73.66) (xy 153.67 63.5)
 		)
 		(stroke
@@
 	(wire
 		(pts
-			(xy 162.56 63.5) (xy 162.56 71.12)
+			(xy 140.97 63.5) (xy 142.24 63.5)
+		)
+		(stroke
+			(width 0)
+			(type default)
+		)
+	)
+	(wire
+		(pts
+			(xy 163.83 63.5) (xy 163.83 71.12)
 		)
 		(stroke
@@
 		(dnp no)
 		(property "Reference" "C1605"
-			(at 146.05 54.61 90)
+			(at 146.05 57.1501 90)
 			(effects
 				(font
@@
 		)
 		(property "Value" "1u"
-			(at 146.05 57.15 90)
+			(at 146.05 59.6901 90)
 			(effects
 				(font
@@
 					(size 1.27 1.27)
 				)
+				(hide yes)
 			)
 		)
@@
 		(dnp no)
 		(property "Reference" "C1606"
-			(at 158.75 54.6099 90)
+			(at 158.75 57.15 90)
 			(effects
 				(font
@@
 		)
 		(property "Value" "1u"
-			(at 158.75 57.1499 90)
+			(at 158.75 59.69 90)
 			(effects
 				(font
@@
 					(size 1.27 1.27)
 				)
-			)
-		)
+				(hide yes)
+			)
+		)
