File: Input Hardware/PCB/Input Board/Tx.kicad_sch (KiCad schematic)
At the start: 40 parts

Commit message: images and pcb stuff
Connections:
- net +5V: no longer U?.8 (~{SRCLR}), U?.8 (~{SRCLR}), U?.8 (~{SRCLR}), U?.8 (~{SRCLR})
- new net ~{SRCLR}: U?.8 (~{SRCLR}), U?.8 (~{SRCLR}), U?.8 (~{SRCLR}), U?.8 (~{SRCLR})

Commit message: Revert "images and pcb stuff"
This reverts commit 6978c7447e140ee759e19aaebffdac22097ec1b9.
Connections:
- net ~{SRCLR} is gone; now on net +5V: U?.8 (~{SRCLR}), U?.8 (~{SRCLR}), U?.8 (~{SRCLR}), U?.8 (~{SRCLR})

Commit message: More footprints
Parts:
- added C? (x4): 10u, Capacitor_SMD:C_0603_1608Metric, symbol Device:C
Connections:
- net +5V: now also C?.1, C?.1, C?.1, C?.1
- net GND: now also C?.2, C?.2, C?.2, C?.2
Other:
- moved on the sheet: C?
