File: Input Hardware/PCB/Input Board/Input Board.kicad_pcb (KiCad board)
At the start: 2 copper layers, 255 x 180 mm, 36 parts

Commit message: Fix files idc
Parts:
- added C1001: 100n, Capacitor_SMD:C_0603_1608Metric, F.Cu at (-170.3, -30.5)
- added C1002: 100n, Capacitor_SMD:C_0603_1608Metric, F.Cu at (-170.3, -28.0)
- added C1003: 100n, Capacitor_SMD:C_0603_1608Metric, F.Cu at (-170.3, -25.5)
- added C1004: 100n, Capacitor_SMD:C_0603_1608Metric, F.Cu at (-170.3, -23.0)
- added C1101: 100n, Capacitor_SMD:C_0603_1608Metric, F.Cu at (14.8, -15.9)
- added C1201: 100n, Capacitor_SMD:C_0603_1608Metric, F.Cu at (-159.9, -14.1)
- added C1202: 100n, Capacitor_SMD:C_0603_1608Metric, F.Cu at (-159.9, -11.5)
- added C1203: 1u, Capacitor_SMD:C_0603_1608Metric, F.Cu at (-159.9, -9.04)
- added C1204: 1u, Capacitor_SMD:C_0603_1608Metric, F.Cu at (-159.9, -6.53)
- added C1205: 100n, Capacitor_SMD:C_0603_1608Metric, F.Cu at (-155.9, -14.1)
- added C1206: 100n, Capacitor_SMD:C_0603_1608Metric, F.Cu at (-155.9, -11.5)
- added C1207: 1u, Capacitor_SMD:C_0603_1608Metric, F.Cu at (-155.9, -9.04)
- added C1208: 1u, Capacitor_SMD:C_0603_1608Metric, F.Cu at (-155.9, -6.53)
- added C1301: 1u, Capacitor_SMD:C_0603_1608Metric, F.Cu at (-57.5, -11.4)
- added C1302: 2.2u, Capacitor_SMD:C_0603_1608Metric, F.Cu at (-57.5, -8.93)
- added C1303: 2.2u, Capacitor_SMD:C_0603_1608Metric, F.Cu at (-57.5, -6.42)
- added C1304: 1u, Capacitor_SMD:C_0603_1608Metric, F.Cu at (-57.5, -3.90)
- added C1305: 1u, Capacitor_SMD:C_0603_1608Metric, F.Cu at (-57.5, -1.40)
- added C1306: 1u, Capacitor_SMD:C_0603_1608Metric, F.Cu at (-57.5, 1.11)
- added C301: 1.8n, Capacitor_SMD:C_0603_1608Metric, F.Cu at (-79.7, -14.1)
- added C302: 1.8n, Capacitor_SMD:C_0603_1608Metric, F.Cu at (-79.7, -11.5)
- added C303: 1.8n, Capacitor_SMD:C_0603_1608Metric, F.Cu at (-79.7, -9.04)
- added C304: 1.8n, Capacitor_SMD:C_0603_1608Metric, F.Cu at (-79.7, -6.53)
- added C305: 100n, Capacitor_SMD:C_0603_1608Metric, F.Cu at (-79.7, -4.01)
- added C306: 1.8n, Capacitor_SMD:C_0603_1608Metric, F.Cu at (-79.7, -1.50)
- added C307: 1.8n, Capacitor_SMD:C_0603_1608Metric, F.Cu at (-79.7, 1.00)
- added C308: 100n, Capacitor_SMD:C_0603_1608Metric, F.Cu at (-79.7, 3.52)
- added C309: 1.8n, Capacitor_SMD:C_0603_1608Metric, F.Cu at (-79.7, 6.03)
- added C310: 1.8n, Capacitor_SMD:C_0603_1608Metric, F.Cu at (-75.7, -14.1)
- added C311: 1.8n, Capacitor_SMD:C_0603_1608Metric, F.Cu at (-75.7, -11.5)
- added C312: 1.8n, Capacitor_SMD:C_0603_1608Metric, F.Cu at (-75.7, -9.04)
- added C313: 1.8n, Capacitor_SMD:C_0603_1608Metric, F.Cu at (-75.7, -6.53)
- added C314: 1.8n, Capacitor_SMD:C_0603_1608Metric, F.Cu at (-75.7, -4.01)
- added C315: 1.8n, Capacitor_SMD:C_0603_1608Metric, F.Cu at (-75.7, -1.50)
- added C316: 1.8n, Capacitor_SMD:C_0603_1608Metric, F.Cu at (-75.7, 1.00)
- added C317: 1.8n, Capacitor_SMD:C_0603_1608Metric, F.Cu at (-75.7, 3.52)
- added C318: 1.8n, Capacitor_SMD:C_0603_1608Metric, F.Cu at (-75.7, 6.03)
- added C401: 1.8n, Capacitor_SMD:C_0603_1608Metric, F.Cu at (-101.8, -14.1)
- added C402: 1.8n, Capacitor_SMD:C_0603_1608Metric, F.Cu at (-101.8, -11.5)
- added C403: 1.8n, Capacitor_SMD:C_0603_1608Metric, F.Cu at (-101.8, -9.04)
- added C404: 1.8n, Capacitor_SMD:C_0603_1608Metric, F.Cu at (-101.8, -6.53)
- added C405: 100n, Capacitor_SMD:C_0603_1608Metric, F.Cu at (-101.8, -4.01)
- added C406: 1.8n, Capacitor_SMD:C_0603_1608Metric, F.Cu at (-101.8, -1.50)
- added C407: 1.8n, Capacitor_SMD:C_0603_1608Metric, F.Cu at (-101.8, 1.00)
- added C408: 100n, Capacitor_SMD:C_0603_1608Metric, F.Cu at (-101.8, 3.52)
- added C409: 1.8n, Capacitor_SMD:C_0603_1608Metric, F.Cu at (-101.8, 6.03)
- added C410: 1.8n, Capacitor_SMD:C_0603_1608Metric, F.Cu at (-97.8, -14.1)
- added C411: 1.8n, Capacitor_SMD:C_0603_1608Metric, F.Cu at (-97.8, -11.5)
- added C412: 1.8n, Capacitor_SMD:C_0603_1608Metric, F.Cu at (-97.8, -9.04)
- added C413: 1.8n, Capacitor_SMD:C_0603_1608Metric, F.Cu at (-97.8, -6.53)
- added C414: 1.8n, Capacitor_SMD:C_0603_1608Metric, F.Cu at (-97.8, -4.01)
- added C415: 1.8n, Capacitor_SMD:C_0603_1608Metric, F.Cu at (-97.8, -1.50)
- added C416: 1.8n, Capacitor_SMD:C_0603_1608Metric, F.Cu at (-97.8, 1.00)
- added C417: 1.8n, Capacitor_SMD:C_0603_1608Metric, F.Cu at (-97.8, 3.52)
- added C418: 1.8n, Capacitor_SMD:C_0603_1608Metric, F.Cu at (-97.8, 6.03)
- added C501: 1.8n, Capacitor_SMD:C_0603_1608Metric, F.Cu at (-123.8, -14.1)
- added C502: 1.8n, Capacitor_SMD:C_0603_1608Metric, F.Cu at (-123.8, -11.5)
- added C503: 1.8n, Capacitor_SMD:C_0603_1608Metric, F.Cu at (-123.8, -9.04)
- added C504: 1.8n, Capacitor_SMD:C_0603_1608Metric, F.Cu at (-123.8, -6.53)
- added C505: 100n, Capacitor_SMD:C_0603_1608Metric, F.Cu at (-123.8, -4.01)
- added C506: 1.8n, Capacitor_SMD:C_0603_1608Metric, F.Cu at (-123.8, -1.50)
- added C507: 1.8n, Capacitor_SMD:C_0603_1608Metric, F.Cu at (-123.8, 1.00)
- added C508: 100n, Capacitor_SMD:C_0603_1608Metric, F.Cu at (-123.8, 3.52)
- added C509: 1.8n, Capacitor_SMD:C_0603_1608Metric, F.Cu at (-123.8, 6.03)
- added C510: 1.8n, Capacitor_SMD:C_0603_1608Metric, F.Cu at (-119.8, -14.1)
- added C511: 1.8n, Capacitor_SMD:C_0603_1608Metric, F.Cu at (-119.8, -11.5)
- added C512: 1.8n, Capacitor_SMD:C_0603_1608Metric, F.Cu at (-119.8, -9.04)
- added C513: 1.8n, Capacitor_SMD:C_0603_1608Metric, F.Cu at (-119.8, -6.53)
- added C514: 1.8n, Capacitor_SMD:C_0603_1608Metric, F.Cu at (-119.8, -4.01)
- added C515: 1.8n, Capacitor_SMD:C_0603_1608Metric, F.Cu at (-119.8, -1.50)
- added C516: 1.8n, Capacitor_SMD:C_0603_1608Metric, F.Cu at (-119.8, 1.00)
- added C517: 1.8n, Capacitor_SMD:C_0603_1608Metric, F.Cu at (-119.8, 3.52)
- added C518: 1.8n, Capacitor_SMD:C_0603_1608Metric, F.Cu at (-119.8, 6.03)
- added C601: 1.8n, Capacitor_SMD:C_0603_1608Metric, F.Cu at (-145.9, -14.1)
- added C602: 1.8n, Capacitor_SMD:C_0603_1608Metric, F.Cu at (-145.9, -11.5)
- added C603: 1.8n, Capacitor_SMD:C_0603_1608Metric, F.Cu at (-145.9, -9.04)
- added C604: 1.8n, Capacitor_SMD:C_0603_1608Metric, F.Cu at (-145.9, -6.53)
- added C605: 100n, Capacitor_SMD:C_0603_1608Metric, F.Cu at (-145.9, -4.01)
- added C606: 1.8n, Capacitor_SMD:C_0603_1608Metric, F.Cu at (-145.9, -1.50)
- added C607: 1.8n, Capacitor_SMD:C_0603_1608Metric, F.Cu at (-145.9, 1.00)
- added C608: 100n, Capacitor_SMD:C_0603_1608Metric, F.Cu at (-145.9, 3.52)
- added C609: 1.8n, Capacitor_SMD:C_0603_1608Metric, F.Cu at (-145.9, 6.03)
- added C610: 1.8n, Capacitor_SMD:C_0603_1608Metric, F.Cu at (-141.9, -14.1)
- added C611: 1.8n, Capacitor_SMD:C_0603_1608Metric, F.Cu at (-141.9, -11.5)
- added C612: 1.8n, Capacitor_SMD:C_0603_1608Metric, F.Cu at (-141.9, -9.04)
- added C613: 1.8n, Capacitor_SMD:C_0603_1608Metric, F.Cu at (-141.9, -6.53)
- added C614: 1.8n, Capacitor_SMD:C_0603_1608Metric, F.Cu at (-141.9, -4.01)
- added C615: 1.8n, Capacitor_SMD:C_0603_1608Metric, F.Cu at (-141.9, -1.50)
- added C616: 1.8n, Capacitor_SMD:C_0603_1608Metric, F.Cu at (-141.9, 1.00)
- added C617: 1.8n, Capacitor_SMD:C_0603_1608Metric, F.Cu at (-141.9, 3.52)
- added C618: 1.8n, Capacitor_SMD:C_0603_1608Metric, F.Cu at (-141.9, 6.03)
- added C701: 100n, Capacitor_SMD:C_0603_1608Metric, F.Cu at (-222.0, -2.44)
- added C702: 100n, Capacitor_SMD:C_0603_1608Metric, F.Cu at (-222.0, 0.07)
- added C703: 100n, Capacitor_SMD:C_0603_1608Metric, F.Cu at (-222.0, 2.58)
- added C704: 39p, Capacitor_SMD:C_0603_1608Metric, F.Cu at (-222.0, 5.09)
- added C705: 39p, Capacitor_SMD:C_0603_1608Metric, F.Cu at (-222.0, 7.61)
- added C706: 39p, Capacitor_SMD:C_0603_1608Metric, F.Cu at (-222.0, 10.1)
- added C707: 39p, Capacitor_SMD:C_0603_1608Metric, F.Cu at (-222.0, 12.6)
- added C708: 56p, Capacitor_SMD:C_0603_1608Metric, F.Cu at (-222.0, 15.1)
- added C709: 56p, Capacitor_SMD:C_0603_1608Metric, F.Cu at (-218.0, -2.44)
- added C710: 56p, Capacitor_SMD:C_0603_1608Metric, F.Cu at (-218.0, 0.07)
- added C711: 56p, Capacitor_SMD:C_0603_1608Metric, F.Cu at (-218.0, 2.58)
- added C712: 56p, Capacitor_SMD:C_0603_1608Metric, F.Cu at (-218.0, 5.09)
- added C713: 56p, Capacitor_SMD:C_0603_1608Metric, F.Cu at (-218.0, 7.61)
- added C801: 100n, Capacitor_SMD:C_0603_1608Metric, F.Cu at (65.2, -16.9)
- added C802: 100n, Capacitor_SMD:C_0603_1608Metric, F.Cu at (65.2, -14.4)
- added C803: 100n, Capacitor_SMD:C_0603_1608Metric, F.Cu at (65.2, -11.9)
- added C804: 39p, Capacitor_SMD:C_0603_1608Metric, F.Cu at (65.2, -9.38)
- added C805: 39p, Capacitor_SMD:C_0603_1608Metric, F.Cu at (65.2, -6.88)
- added C806: 39p, Capacitor_SMD:C_0603_1608Metric, F.Cu at (65.2, -4.37)
- added C807: 39p, Capacitor_SMD:C_0603_1608Metric, F.Cu at (65.2, -1.85)
- added C808: 56p, Capacitor_SMD:C_0603_1608Metric, F.Cu at (65.2, 0.66)
- added C809: 56p, Capacitor_SMD:C_0603_1608Metric, F.Cu at (69.2, -16.9)
- added C810: 56p, Capacitor_SMD:C_0603_1608Metric, F.Cu at (69.2, -14.4)
- added C811: 56p, Capacitor_SMD:C_0603_1608Metric, F.Cu at (69.2, -11.9)
- added C812: 56p, Capacitor_SMD:C_0603_1608Metric, F.Cu at (69.2, -9.38)
- added C813: 56p, Capacitor_SMD:C_0603_1608Metric, F.Cu at (69.2, -6.88)
- added C901: 100n, Capacitor_SMD:C_0603_1608Metric, F.Cu at (33.0, -28.5)
- added C902: 10u, Capacitor_SMD:C_0603_1608Metric, F.Cu at (33.0, -26.0)
- added C903: 100n, Capacitor_SMD:C_0603_1608Metric, F.Cu at (33.0, -23.5)
- added C904: 100n, Capacitor_SMD:C_0603_1608Metric, F.Cu at (33.0, -21.0)
- added C905: 47n, Capacitor_SMD:C_0603_1608Metric, F.Cu at (33.0, -18.5)
- added C906: 100n, Capacitor_SMD:C_0603_1608Metric, F.Cu at (33.0, -16.0)
- added C907: 100n, Capacitor_SMD:C_0603_1608Metric, F.Cu at (33.0, -13.5)
- added C908: 100n, Capacitor_SMD:C_0603_1608Metric, F.Cu at (37.0, -28.5)
- added C909: 100n, Capacitor_SMD:C_0603_1608Metric, F.Cu at (37.0, -26.0)
- added C910: 100n, Capacitor_SMD:C_0603_1608Metric, F.Cu at (37.0, -23.5)
- added C911: 100n, Capacitor_SMD:C_0603_1608Metric, F.Cu at (37.0, -21.0)
- added C912: 100n, Capacitor_SMD:C_0603_1608Metric, F.Cu at (37.0, -18.5)
- added D1101: E, LED_SMD:LED_0603_1608Metric, F.Cu at (22.9, -15.9)
- added D1102: C, LED_SMD:LED_0603_1608Metric, F.Cu at (22.9, -13.3)
- added D1103: X, LED_SMD:LED_0603_1608Metric, F.Cu at (22.9, -10.7)
- added D1104: X, LED_SMD:LED_0603_1608Metric, F.Cu at (22.9, -8.12)
- added D1105: Z, LED_SMD:LED_0603_1608Metric, F.Cu at (22.9, -5.54)
- added D1106: Y, LED_SMD:LED_0603_1608Metric, F.Cu at (27.0, -15.9)
- added D1107: Y, LED_SMD:LED_0603_1608Metric, F.Cu at (27.0, -13.3)
- added D1108: L, LED_SMD:LED_0603_1608Metric, F.Cu at (27.0, -10.7)
- added D1109: X, LED_SMD:LED_0603_1608Metric, F.Cu at (27.0, -8.12)
- added D1110: X, LED_SMD:LED_0603_1608Metric, F.Cu at (27.0, -5.54)
- added FB1201: 120, Inductor_SMD:L_1206_3216Metric, F.Cu at (-159.1, -3.54)
- added FB1202: 120, Inductor_SMD:L_1206_3216Metric, F.Cu at (-159.1, -0.10)
- added H105: MountingHole, MountingHole:MountingHole_3.2mm_M3, F.Cu at (-177.6, -11.3)
- added H106: MountingHole, MountingHole:MountingHole_3.2mm_M3, F.Cu at (-177.6, -3.38)
- added J1301: 1.71" SSD1312 OLED, Display:1.71 OLED SSD1312, F.Cu at (267.5, 68.0)
- added J901: USB_C_Receptacle_USB2.0_16P, Connector_USB:USB_C_Receptacle_GCT_USB4110, F.Cu at (38.2, -6.93)
- added JP901: 3.3V STLINK, Jumper:SolderJumper-2_P1.3mm_Open_RoundedPad1.0x1.5mm, F.Cu at (38.3, -0.46)
- added L1001: L, Coil:5x160, B.Cu at (-17.7, 79.9)
- added L1002: L, Coil:5x160, B.Cu at (-23.6, 79.9)
- added L1003: L, Coil:5x160, B.Cu at (-29.5, 79.9)
- added L1004: L, Coil:5x160, B.Cu at (-35.4, 79.9)
- added L1005: L, Coil:5x160, B.Cu at (-41.3, 79.9)
- added L1006: L, Coil:5x160, B.Cu at (-47.2, 79.9)
- added L1007: L, Coil:5x160, B.Cu at (-53.1, 79.9)
- added L1008: L, Coil:5x160, B.Cu at (-59.0, 79.9)
- added L1009: L, Coil:5x160, B.Cu at (-64.9, 79.9)
- added L1010: L, Coil:5x160, B.Cu at (-70.8, 79.9)
- added L1011: L, Coil:5x160, B.Cu at (-76.7, 79.9)
- added L1012: L, Coil:5x160, B.Cu at (-82.6, 79.9)
- added L1013: L, Coil:5x160, B.Cu at (-88.5, 79.9)
- added L1014: L, Coil:5x160, B.Cu at (-94.4, 79.9)
- added L1015: L, Coil:5x160, B.Cu at (-100.3, 79.9)
- added L1016: L, Coil:5x160, B.Cu at (-106.2, 79.9)
- added L1017: L, Coil:5x160, B.Cu at (-112.1, 79.9)
- added L1018: L, Coil:5x160, B.Cu at (-118.0, 79.9)
- added L1019: L, Coil:5x160, B.Cu at (-123.9, 79.9)
- added L1020: L, Coil:5x160, B.Cu at (-129.8, 79.9)
- added L1021: L, Coil:5x160, B.Cu at (-135.7, 79.9)
- added L1022: L, Coil:5x160, B.Cu at (-141.6, 79.9)
- added L1023: L, Coil:5x160, B.Cu at (-147.5, 79.9)
- added L1024: L, Coil:5x160, B.Cu at (-153.4, 79.9)
- added L1025: L, Coil:5x160, B.Cu at (-159.3, 79.9)
- added L1026: L, Coil:5x160, B.Cu at (-165.2, 79.9)
- added L1027: L, Coil:5x160, B.Cu at (-171.1, 79.9)
- added L1028: L, Coil:5x160, B.Cu at (-177.0, 79.9)
- added L1029: L, Coil:5x160, B.Cu at (-182.9, 79.9)
- added L1030: L, Coil:5x160, B.Cu at (-188.8, 79.9)
- added L1031: L, Coil:5x160, B.Cu at (-194.7, 79.9)
- added L1032: L, Coil:5x160, B.Cu at (-200.6, 79.9)
- added R1101: TBD, Resistor_SMD:R_0603_1608Metric, F.Cu at (14.8, -13.4)
- added R1102: TBD, Resistor_SMD:R_0603_1608Metric, F.Cu at (14.8, -10.9)
- added R1103: TBD, Resistor_SMD:R_0603_1608Metric, F.Cu at (14.8, -8.40)
- added R1104: TBD, Resistor_SMD:R_0603_1608Metric, F.Cu at (14.8, -5.89)
- added R1105: TBD, Resistor_SMD:R_0603_1608Metric, F.Cu at (14.8, -3.38)
- added R1106: TBD, Resistor_SMD:R_0603_1608Metric, F.Cu at (18.9, -15.9)
- added R1107: TBD, Resistor_SMD:R_0603_1608Metric, F.Cu at (18.9, -13.4)
- added R1108: TBD, Resistor_SMD:R_0603_1608Metric, F.Cu at (18.9, -10.9)
- added R1109: TBD, Resistor_SMD:R_0603_1608Metric, F.Cu at (18.9, -8.40)
- added R1110: TBD, Resistor_SMD:R_0603_1608Metric, F.Cu at (18.9, -5.89)
- added R1201: 3.9k, Resistor_SMD:R_0603_1608Metric, F.Cu at (-151.9, -14.1)
- added R1202: 750, Resistor_SMD:R_0603_1608Metric, F.Cu at (-151.9, -11.5)
- added R1203: 2.4k, Resistor_SMD:R_0603_1608Metric, F.Cu at (-151.9, -9.04)
- added R1204: 2.4k, Resistor_SMD:R_0603_1608Metric, F.Cu at (-151.9, -6.53)
- added R1301: 10k, Resistor_SMD:R_0603_1608Metric, F.Cu at (-57.5, 3.62)
- added R1302: 550k, Resistor_SMD:R_0603_1608Metric, F.Cu at (-57.5, 6.13)
- added R1303: 10k, Resistor_SMD:R_0603_1608Metric, F.Cu at (-57.5, 8.64)
- added R301: 1k, Resistor_SMD:R_0603_1608Metric, F.Cu at (-71.7, -14.1)
- added R302: 1k, Resistor_SMD:R_0603_1608Metric, F.Cu at (-71.7, -11.5)
- added R303: 1k, Resistor_SMD:R_0603_1608Metric, F.Cu at (-71.7, -9.04)
- added R304: 1k, Resistor_SMD:R_0603_1608Metric, F.Cu at (-71.7, -6.53)
- added R305: 15k, Resistor_SMD:R_0603_1608Metric, F.Cu at (-71.7, -4.01)
- added R306: 15k, Resistor_SMD:R_0603_1608Metric, F.Cu at (-71.7, -1.50)
- added R307: 1k, Resistor_SMD:R_0603_1608Metric, F.Cu at (-71.7, 1.00)
- added R308: 1k, Resistor_SMD:R_0603_1608Metric, F.Cu at (-71.7, 3.52)
- added R309: 1k, Resistor_SMD:R_0603_1608Metric, F.Cu at (-71.7, 6.03)
- added R310: 1k, Resistor_SMD:R_0603_1608Metric, F.Cu at (-67.7, -14.1)
- added R311: 15k, Resistor_SMD:R_0603_1608Metric, F.Cu at (-67.7, -11.5)
- added R312: 15k, Resistor_SMD:R_0603_1608Metric, F.Cu at (-67.7, -9.04)
- added R313: 1k, Resistor_SMD:R_0603_1608Metric, F.Cu at (-67.7, -6.53)
- added R314: 1k, Resistor_SMD:R_0603_1608Metric, F.Cu at (-67.7, -4.01)
- added R315: 1k, Resistor_SMD:R_0603_1608Metric, F.Cu at (-67.7, -1.50)
- added R316: 1k, Resistor_SMD:R_0603_1608Metric, F.Cu at (-67.7, 1.00)
- added R317: 15k, Resistor_SMD:R_0603_1608Metric, F.Cu at (-67.7, 3.52)
- added R318: 15k, Resistor_SMD:R_0603_1608Metric, F.Cu at (-67.7, 6.03)
- added R319: 1k, Resistor_SMD:R_0603_1608Metric, F.Cu at (-63.7, -14.1)
- added R320: 1k, Resistor_SMD:R_0603_1608Metric, F.Cu at (-63.7, -11.5)
- added R321: 1k, Resistor_SMD:R_0603_1608Metric, F.Cu at (-63.7, -9.04)
- added R322: 1k, Resistor_SMD:R_0603_1608Metric, F.Cu at (-63.7, -6.53)
- added R323: 15k, Resistor_SMD:R_0603_1608Metric, F.Cu at (-63.7, -4.01)
- added R324: 15k, Resistor_SMD:R_0603_1608Metric, F.Cu at (-63.7, -1.50)
- added R401: 1k, Resistor_SMD:R_0603_1608Metric, F.Cu at (-93.8, -14.1)
- added R402: 1k, Resistor_SMD:R_0603_1608Metric, F.Cu at (-93.8, -11.5)
- added R403: 1k, Resistor_SMD:R_0603_1608Metric, F.Cu at (-93.8, -9.04)
- added R404: 1k, Resistor_SMD:R_0603_1608Metric, F.Cu at (-93.8, -6.53)
- added R405: 15k, Resistor_SMD:R_0603_1608Metric, F.Cu at (-93.8, -4.01)
- added R406: 15k, Resistor_SMD:R_0603_1608Metric, F.Cu at (-93.8, -1.50)
- added R407: 1k, Resistor_SMD:R_0603_1608Metric, F.Cu at (-93.8, 1.00)
- added R408: 1k, Resistor_SMD:R_0603_1608Metric, F.Cu at (-93.8, 3.52)
- added R409: 1k, Resistor_SMD:R_0603_1608Metric, F.Cu at (-93.8, 6.03)
- added R410: 1k, Resistor_SMD:R_0603_1608Metric, F.Cu at (-89.8, -14.1)
- added R411: 15k, Resistor_SMD:R_0603_1608Metric, F.Cu at (-89.8, -11.5)
- added R412: 15k, Resistor_SMD:R_0603_1608Metric, F.Cu at (-89.8, -9.04)
- added R413: 1k, Resistor_SMD:R_0603_1608Metric, F.Cu at (-89.8, -6.53)
- added R414: 1k, Resistor_SMD:R_0603_1608Metric, F.Cu at (-89.8, -4.01)
- added R415: 1k, Resistor_SMD:R_0603_1608Metric, F.Cu at (-89.8, -1.50)
- added R416: 1k, Resistor_SMD:R_0603_1608Metric, F.Cu at (-89.8, 1.00)
- added R417: 15k, Resistor_SMD:R_0603_1608Metric, F.Cu at (-89.8, 3.52)
- added R418: 15k, Resistor_SMD:R_0603_1608Metric, F.Cu at (-89.8, 6.03)
- added R419: 1k, Resistor_SMD:R_0603_1608Metric, F.Cu at (-85.8, -14.1)
- added R420: 1k, Resistor_SMD:R_0603_1608Metric, F.Cu at (-85.8, -11.5)
- added R421: 1k, Resistor_SMD:R_0603_1608Metric, F.Cu at (-85.8, -9.04)
- added R422: 1k, Resistor_SMD:R_0603_1608Metric, F.Cu at (-85.8, -6.53)
- added R423: 15k, Resistor_SMD:R_0603_1608Metric, F.Cu at (-85.8, -4.01)
- added R424: 15k, Resistor_SMD:R_0603_1608Metric, F.Cu at (-85.8, -1.50)
- added R501: 1k, Resistor_SMD:R_0603_1608Metric, F.Cu at (-115.8, -14.1)
- added R502: 1k, Resistor_SMD:R_0603_1608Metric, F.Cu at (-115.8, -11.5)
- added R503: 1k, Resistor_SMD:R_0603_1608Metric, F.Cu at (-115.8, -9.04)
- added R504: 1k, Resistor_SMD:R_0603_1608Metric, F.Cu at (-115.8, -6.53)
- added R505: 15k, Resistor_SMD:R_0603_1608Metric, F.Cu at (-115.8, -4.01)
- added R506: 15k, Resistor_SMD:R_0603_1608Metric, F.Cu at (-115.8, -1.50)
- added R507: 1k, Resistor_SMD:R_0603_1608Metric, F.Cu at (-115.8, 1.00)
- added R508: 1k, Resistor_SMD:R_0603_1608Metric, F.Cu at (-115.8, 3.52)
- added R509: 1k, Resistor_SMD:R_0603_1608Metric, F.Cu at (-115.8, 6.03)
- added R510: 1k, Resistor_SMD:R_0603_1608Metric, F.Cu at (-111.8, -14.1)
- added R511: 15k, Resistor_SMD:R_0603_1608Metric, F.Cu at (-111.8, -11.5)
- added R512: 15k, Resistor_SMD:R_0603_1608Metric, F.Cu at (-111.8, -9.04)
- added R513: 1k, Resistor_SMD:R_0603_1608Metric, F.Cu at (-111.8, -6.53)
- added R514: 1k, Resistor_SMD:R_0603_1608Metric, F.Cu at (-111.8, -4.01)
- added R515: 1k, Resistor_SMD:R_0603_1608Metric, F.Cu at (-111.8, -1.50)
- added R516: 1k, Resistor_SMD:R_0603_1608Metric, F.Cu at (-111.8, 1.00)
- added R517: 15k, Resistor_SMD:R_0603_1608Metric, F.Cu at (-111.8, 3.52)
- added R518: 15k, Resistor_SMD:R_0603_1608Metric, F.Cu at (-111.8, 6.03)
- added R519: 1k, Resistor_SMD:R_0603_1608Metric, F.Cu at (-107.8, -14.1)
- added R520: 1k, Resistor_SMD:R_0603_1608Metric, F.Cu at (-107.8, -11.5)
- added R521: 1k, Resistor_SMD:R_0603_1608Metric, F.Cu at (-107.8, -9.04)
- added R522: 1k, Resistor_SMD:R_0603_1608Metric, F.Cu at (-107.8, -6.53)
- added R523: 15k, Resistor_SMD:R_0603_1608Metric, F.Cu at (-107.8, -4.01)
- added R524: 15k, Resistor_SMD:R_0603_1608Metric, F.Cu at (-107.8, -1.50)
- added R601: 1k, Resistor_SMD:R_0603_1608Metric, F.Cu at (-137.9, -14.1)
- added R602: 1k, Resistor_SMD:R_0603_1608Metric, F.Cu at (-137.9, -11.5)
- added R603: 1k, Resistor_SMD:R_0603_1608Metric, F.Cu at (-137.9, -9.04)
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Connections:
- L201 pad 2: unconnected-(L201-Pad2) -> /Receiver Stage/Rx Row Amplifier 1/RXIN1
- L202 pad 2: unconnected-(L202-Pad2) -> /Receiver Stage/Rx Row Amplifier 1/RXIN2
- L203 pad 2: unconnected-(L203-Pad2) -> /Receiver Stage/Rx Row Amplifier 1/RXIN3
- L204 pad 2: unconnected-(L204-Pad2) -> /Receiver Stage/Rx Row Amplifier 1/RXIN4
- L205 pad 2: unconnected-(L205-Pad2) -> /Receiver Stage/RXIN5_1
- L206 pad 2: unconnected-(L206-Pad2) -> /Receiver Stage/RXIN6_1
- L207 pad 2: unconnected-(L207-Pad2) -> /Receiver Stage/RXIN7_1
- L208 pad 2: unconnected-(L208-Pad2) -> /Receiver Stage/RXIN8_1
- L209 pad 2: unconnected-(L209-Pad2) -> /Receiver Stage/Rx Row Amplifier 2/RXIN1
- L210 pad 2: unconnected-(L210-Pad2) -> /Receiver Stage/Rx Row Amplifier 2/RXIN2
- L211 pad 2: unconnected-(L211-Pad2) -> /Receiver Stage/Rx Row Amplifier 2/RXIN3
- L212 pad 2: unconnected-(L212-Pad2) -> /Receiver Stage/Rx Row Amplifier 2/RXIN4
- L213 pad 2: unconnected-(L213-Pad2) -> /Receiver Stage/RXIN5_3
- L214 pad 2: unconnected-(L214-Pad2) -> /Receiver Stage/RXIN6_3
- L215 pad 2: unconnected-(L215-Pad2) -> /Receiver Stage/RXIN7_3
- L216 pad 2: unconnected-(L216-Pad2) -> /Receiver Stage/RXIN8_3
- L217 pad 2: unconnected-(L217-Pad2) -> /Receiver Stage/Rx Row Amplifier 3/RXIN1
- L218 pad 2: unconnected-(L218-Pad2) -> /Receiver Stage/Rx Row Amplifier 3/RXIN2
- L219 pad 2: unconnected-(L219-Pad2) -> /Receiver Stage/Rx Row Amplifier 3/RXIN3
- L220 pad 2: unconnected-(L220-Pad2) -> /Receiver Stage/Rx Row Amplifier 3/RXIN4
- L221 pad 2: unconnected-(L221-Pad2) -> /Receiver Stage/RXIN5
- L222 pad 2: unconnected-(L222-Pad2) -> /Receiver Stage/RXIN6
- L223 pad 2: unconnected-(L223-Pad2) -> /Receiver Stage/RXIN7
- L224 pad 2: unconnected-(L224-Pad2) -> /Receiver Stage/RXIN8
- L225 pad 2: unconnected-(L225-Pad2) -> /Receiver Stage/Rx Row Amplifier 4/RXIN1
- L226 pad 2: unconnected-(L226-Pad2) -> /Receiver Stage/Rx Row Amplifier 4/RXIN2
- L227 pad 2: unconnected-(L227-Pad2) -> /Receiver Stage/Rx Row Amplifier 4/RXIN3
- L228 pad 2: unconnected-(L228-Pad2) -> /Receiver Stage/Rx Row Amplifier 4/RXIN4
- L229 pad 2: unconnected-(L229-Pad2) -> /Receiver Stage/RXIN5_2
- L230 pad 2: unconnected-(L230-Pad2) -> /Receiver Stage/RXIN6_2
- L231 pad 2: unconnected-(L231-Pad2) -> /Receiver Stage/RXIN7_2
- L232 pad 2: unconnected-(L232-Pad2) -> /Receiver Stage/RXIN8_2

Commit message: Layout
Parts:
- C301, C302, C303, C304, C305, C306, C307, C308, C309, C310, C311, C312, C313, C314, C315, C316, C317, C318, C401, C402, C403, C404, C405, C406, C407, C408, C409, C410, C411, C412, C413, C414, C415, C416, C417, C418, C501, C502, C503, C504, C505, C506, C507, C508, C509, C510, C511, C512, C513, C514, C515, C516, C517, C518, C601, C602, C603, C604, C605, C606, C607, C608, C609, C610, C611, C612, C613, C614, C615, C616, C617, C618, R301, R302, R303, R304, R305, R306, R307, R308, R309, R310, R311, R312, R313, R314, R315, R316, R317, R318, R319, R320, R321, R322, R323, R324, R401, R402, R403, R404, R405, R406, R407, R408, R409, R410, R411, R412, R413, R414, R415, R416, R417, R418, R419, R420, R421, R422, R423, R424, R501, R502, R503, R504, R505, R506, R507, R508, R509, R510, R511, R512, R513, R514, R515, R516, R517, R518, R519, R520, R521, R522, R523, R524, R601, R602, R603, R604, R605, R606, R607, R608, R609, R610, R611, R612, R613, R614, R615, R616, R617, R618, R619, R620, R621, R622, R623, R624, U1001, U301, U302, U401, U402, U501, U502, U601, U602: moved to B.Cu
- SW1101, SW1102: footprint Connector_PinHeader_2.54mm:PinHeader_1x05_P2.54mm_Vertical_SMD_Pin1Right -> Encoder:Untitled
- moved R712 578.5 mm to (366.9, 41.4)
- moved R713 578.5 mm to (366.9, 43.9)
- moved R714 578.5 mm to (366.9, 46.4)
- moved R715 578.5 mm to (366.9, 48.9)
- moved R716 578.5 mm to (366.9, 51.4)
- moved R717 578.5 mm to (366.9, 53.9)
- moved R718 578.5 mm to (366.9, 56.5)
- moved C701 578.5 mm to (354.8, 41.4)
- moved C702 578.5 mm to (354.8, 43.9)
- moved C703 578.5 mm to (354.8, 46.4)
- moved C704 578.5 mm to (354.8, 48.9)
- moved C705 578.5 mm to (354.8, 51.4)
- moved C706 578.5 mm to (354.8, 53.9)
- moved C707 578.5 mm to (354.8, 56.5)
- moved C708 578.5 mm to (354.8, 59.0)
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Connections:
- C311 pad 2: /Receiver Stage/Rx Row Amplifier 1/RXIN1 -> /Receiver Stage/Rx Row Amplifier 1/RXIN5
- C312 pad 2: /Receiver Stage/Rx Row Amplifier 1/RXIN2 -> /Receiver Stage/Rx Row Amplifier 1/RXIN6
- C315 pad 2: /Receiver Stage/Rx Row Amplifier 1/RXIN3 -> /Receiver Stage/Rx Row Amplifier 1/RXIN7
- C316 pad 2: /Receiver Stage/Rx Row Amplifier 1/RXIN4 -> /Receiver Stage/Rx Row Amplifier 1/RXIN8
- C411 pad 2: /Receiver Stage/Rx Row Amplifier 2/RXIN1 -> /Receiver Stage/Rx Row Amplifier 2/RXIN5
- C412 pad 2: /Receiver Stage/Rx Row Amplifier 2/RXIN2 -> /Receiver Stage/Rx Row Amplifier 2/RXIN6
- C415 pad 2: /Receiver Stage/Rx Row Amplifier 2/RXIN3 -> /Receiver Stage/Rx Row Amplifier 2/RXIN7
- C416 pad 2: /Receiver Stage/Rx Row Amplifier 2/RXIN4 -> /Receiver Stage/Rx Row Amplifier 2/RXIN8
- C511 pad 2: /Receiver Stage/Rx Row Amplifier 3/RXIN1 -> /Receiver Stage/Rx Row Amplifier 3/RXIN5
- C512 pad 2: /Receiver Stage/Rx Row Amplifier 3/RXIN2 -> /Receiver Stage/Rx Row Amplifier 3/RXIN6
- C515 pad 2: /Receiver Stage/Rx Row Amplifier 3/RXIN3 -> /Receiver Stage/Rx Row Amplifier 3/RXIN7
- C516 pad 2: /Receiver Stage/Rx Row Amplifier 3/RXIN4 -> /Receiver Stage/Rx Row Amplifier 3/RXIN8
- C611 pad 2: /Receiver Stage/Rx Row Amplifier 4/RXIN1 -> /Receiver Stage/Rx Row Amplifier 4/RXIN5
- C612 pad 2: /Receiver Stage/Rx Row Amplifier 4/RXIN2 -> /Receiver Stage/Rx Row Amplifier 4/RXIN6
- C615 pad 2: /Receiver Stage/Rx Row Amplifier 4/RXIN3 -> /Receiver Stage/Rx Row Amplifier 4/RXIN7
- C616 pad 2: /Receiver Stage/Rx Row Amplifier 4/RXIN4 -> /Receiver Stage/Rx Row Amplifier 4/RXIN8
- L201 pad 1: GNDPWR -> GND
- L202 pad 1: GNDPWR -> GND
- L203 pad 1: GNDPWR -> GND
- L204 pad 1: GNDPWR -> GND
- L205 pad 1: GNDPWR -> GND
- L205 pad 2: /Receiver Stage/RXIN5_1 -> /Receiver Stage/Rx Row Amplifier 1/RXIN5
- L206 pad 1: GNDPWR -> GND
- L206 pad 2: /Receiver Stage/RXIN6_1 -> /Receiver Stage/Rx Row Amplifier 1/RXIN6
- L207 pad 1: GNDPWR -> GND
- L207 pad 2: /Receiver Stage/RXIN7_1 -> /Receiver Stage/Rx Row Amplifier 1/RXIN7
- L208 pad 1: GNDPWR -> GND
- L208 pad 2: /Receiver Stage/RXIN8_1 -> /Receiver Stage/Rx Row Amplifier 1/RXIN8
- L209 pad 1: GNDPWR -> GND
- L210 pad 1: GNDPWR -> GND
- L211 pad 1: GNDPWR -> GND
- L212 pad 1: GNDPWR -> GND
- L213 pad 1: GNDPWR -> GND
- L213 pad 2: /Receiver Stage/RXIN5_3 -> /Receiver Stage/Rx Row Amplifier 2/RXIN5
- L214 pad 1: GNDPWR -> GND
- L214 pad 2: /Receiver Stage/RXIN6_3 -> /Receiver Stage/Rx Row Amplifier 2/RXIN6
- L215 pad 1: GNDPWR -> GND
- L215 pad 2: /Receiver Stage/RXIN7_3 -> /Receiver Stage/Rx Row Amplifier 2/RXIN7
- L216 pad 1: GNDPWR -> GND
- L216 pad 2: /Receiver Stage/RXIN8_3 -> /Receiver Stage/Rx Row Amplifier 2/RXIN8
- L217 pad 1: GNDPWR -> GND
- L218 pad 1: GNDPWR -> GND
- L219 pad 1: GNDPWR -> GND
- L220 pad 1: GNDPWR -> GND
- L221 pad 1: GNDPWR -> GND
- L221 pad 2: /Receiver Stage/RXIN5 -> /Receiver Stage/Rx Row Amplifier 3/RXIN5
- L222 pad 1: GNDPWR -> GND
- L222 pad 2: /Receiver Stage/RXIN6 -> /Receiver Stage/Rx Row Amplifier 3/RXIN6
- L223 pad 1: GNDPWR -> GND
- L223 pad 2: /Receiver Stage/RXIN7 -> /Receiver Stage/Rx Row Amplifier 3/RXIN7
- L224 pad 1: GNDPWR -> GND
- L224 pad 2: /Receiver Stage/RXIN8 -> /Receiver Stage/Rx Row Amplifier 3/RXIN8
- L225 pad 1: GNDPWR -> GND
- L226 pad 1: GNDPWR -> GND
- L227 pad 1: GNDPWR -> GND
- L228 pad 1: GNDPWR -> GND
- L229 pad 1: GNDPWR -> GND
- L229 pad 2: /Receiver Stage/RXIN5_2 -> /Receiver Stage/Rx Row Amplifier 4/RXIN5
- L230 pad 1: GNDPWR -> GND
- L230 pad 2: /Receiver Stage/RXIN6_2 -> /Receiver Stage/Rx Row Amplifier 4/RXIN6
- L231 pad 1: GNDPWR -> GND
- L231 pad 2: /Receiver Stage/RXIN7_2 -> /Receiver Stage/Rx Row Amplifier 4/RXIN7
- L232 pad 1: GNDPWR -> GND
- L232 pad 2: /Receiver Stage/RXIN8_2 -> /Receiver Stage/Rx Row Amplifier 4/RXIN8
- R317 pad 2: /Mux & Amplifier 1/In1 -> /Mux & Amplifier 1/In5
- R318 pad 2: /Mux & Amplifier 1/In2 -> /Mux & Amplifier 1/In6
- R323 pad 2: /Mux & Amplifier 1/In3 -> /Mux & Amplifier 1/In7
- R324 pad 2: /Mux & Amplifier 1/In4 -> /Mux & Amplifier 1/In8
- R417 pad 2: /Mux & Amplifier 1/In9 -> /Mux & Amplifier 1/In13
- R418 pad 2: /Mux & Amplifier 1/In10 -> /Mux & Amplifier 1/In14
- R423 pad 2: /Mux & Amplifier 1/In11 -> /Mux & Amplifier 1/In15
- R424 pad 2: /Mux & Amplifier 1/In12 -> /Mux & Amplifier 1/In16
- R517 pad 2: /Mux & Amplifier 2/In1 -> /Mux & Amplifier 2/In5
- R518 pad 2: /Mux & Amplifier 2/In2 -> /Mux & Amplifier 2/In6
- R523 pad 2: /Mux & Amplifier 2/In3 -> /Mux & Amplifier 2/In7
- R524 pad 2: /Mux & Amplifier 2/In4 -> /Mux & Amplifier 2/In8
- R617 pad 2: /Mux & Amplifier 2/In9 -> /Mux & Amplifier 2/In13
- R618 pad 2: /Mux & Amplifier 2/In10 -> /Mux & Amplifier 2/In14
- R623 pad 2: /Mux & Amplifier 2/In11 -> /Mux & Amplifier 2/In15
- R624 pad 2: /Mux & Amplifier 2/In12 -> /Mux & Amplifier 2/In16
- U302 pad 1: /Mux & Amplifier 1/In1 -> /Mux & Amplifier 1/In5
- U302 pad 14: /Mux & Amplifier 1/In4 -> /Mux & Amplifier 1/In8
- U302 pad 7: /Mux & Amplifier 1/In2 -> /Mux & Amplifier 1/In6
- U302 pad 8: /Mux & Amplifier 1/In3 -> /Mux & Amplifier 1/In7
- U402 pad 1: /Mux & Amplifier 1/In9 -> /Mux & Amplifier 1/In13
- U402 pad 14: /Mux & Amplifier 1/In12 -> /Mux & Amplifier 1/In16
- U402 pad 7: /Mux & Amplifier 1/In10 -> /Mux & Amplifier 1/In14
- U402 pad 8: /Mux & Amplifier 1/In11 -> /Mux & Amplifier 1/In15
- U502 pad 1: /Mux & Amplifier 2/In1 -> /Mux & Amplifier 2/In5
- U502 pad 14: /Mux & Amplifier 2/In4 -> /Mux & Amplifier 2/In8
- U502 pad 7: /Mux & Amplifier 2/In2 -> /Mux & Amplifier 2/In6
- U502 pad 8: /Mux & Amplifier 2/In3 -> /Mux & Amplifier 2/In7
- U602 pad 1: /Mux & Amplifier 2/In9 -> /Mux & Amplifier 2/In13
- U602 pad 14: /Mux & Amplifier 2/In12 -> /Mux & Amplifier 2/In16
- U602 pad 7: /Mux & Amplifier 2/In10 -> /Mux & Amplifier 2/In14
- U602 pad 8: /Mux & Amplifier 2/In11 -> /Mux & Amplifier 2/In15
Routing:
- net 1.65V: track 0.00 -> 49.4 mm
- net +3.3VA: track 0.00 -> 35.2 mm
- net /Receiver Stage/Rx Row Amplifier 1/RXIN8: track 0.00 -> 20.5 mm, vias 0 -> 1
- net /Receiver Stage/Rx Row Amplifier 1/RXIN4: track 0.00 -> 20.5 mm, vias 0 -> 1
- net /Receiver Stage/Rx Row Amplifier 1/RXIN1: track 0.00 -> 19.4 mm, vias 0 -> 1
- net /Receiver Stage/Rx Row Amplifier 1/RXIN5: track 0.00 -> 19.2 mm, vias 0 -> 1
- net /Receiver Stage/Rx Row Amplifier 1/RXIN7: track 0.00 -> 19.0 mm, vias 0 -> 1
- net /Receiver Stage/Rx Row Amplifier 1/RXIN3: track 0.00 -> 17.8 mm, vias 0 -> 1
- net /Receiver Stage/Rx Row Amplifier 1/RXIN2: track 0.00 -> 17.4 mm, vias 0 -> 1
- net /Receiver Stage/Rx Row Amplifier 1/RXIN6: track 0.00 -> 17.0 mm, vias 0 -> 1
- net /Receiver Stage/Rx Row Amplifier 2/RXIN2: track 0.00 -> 13.6 mm
- net /Receiver Stage/Rx Row Amplifier 4/RXIN2: track 0.00 -> 13.6 mm
- net /Receiver Stage/Rx Row Amplifier 3/RXIN2: track 0.00 -> 13.6 mm
- net /Receiver Stage/Rx Row Amplifier 3/RXIN6: track 0.00 -> 13.4 mm
- net /Receiver Stage/Rx Row Amplifier 2/RXIN6: track 0.00 -> 13.4 mm
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
Commit message: Filter Amplifier Layout
Parts:
- C703, C704, C705, C706, C707, C708, C709, C710, C711, C712, C713, C803, C804, C805, C806, C807, C808, C809, C810, C811, C812, C813, R701, R702, R703, R704, R705, R706, R707, R708, R709, R710, R711, R712, R713, R714, R715, R716, R717, R718, R801, R802, R803, R804, R805, R806, R807, R808, R809, R810, R811, R812, R813, R814, R815, R816, R817, R818, TP701, TP801, U701, U702, U703, U801, U802, U803: moved to B.Cu
- U1101: value 74HCS95 -> 74HC595
- moved R804 318.8 mm to (291.3, 215.6), turned to 180 degrees
- moved C805 318.3 mm to (291.3, 217.1)
- moved C809 318.3 mm to (291.3, 211.0)
- moved R807 317.7 mm to (291.3, 221.7), turned to 180 degrees
- moved C807 316.9 mm to (291.3, 220.2), turned to 180 degrees
- moved R808 313.7 mm to (291.3, 218.7), turned to 180 degrees
- moved C811 313.6 mm to (291.3, 209.5), turned to 180 degrees
- moved R805 311.3 mm to (276.1, 221.7)
- moved R802 309.8 mm to (291.3, 214.1), turned to 180 degrees
- moved C804 309.5 mm to (276.1, 217.1), turned to 180 degrees
- moved R812 308.3 mm to (291.3, 204.9)
- moved C806 308.0 mm to (276.1, 220.2)
- moved C803 308.0 mm to (276.1, 212.6), turned to 180 degrees
- moved R806 307.1 mm to (276.1, 218.7)
- moved C802 306.2 mm to (255.2, 225.7)
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Connections:
- C705 pad 1: Net-(U701C-+) -> Net-(U701D-+)
- C711 pad 2: Net-(U701D-+) -> Net-(U701C-+)
- C805 pad 1: Net-(U801C-+) -> Net-(U801D-+)
- C811 pad 2: Net-(U801D-+) -> Net-(U801C-+)
- R704 pad 2: Net-(U701C-+) -> Net-(U701D-+)
- R707 pad 1: Net-(U701C--) -> Net-(U701D--)
- R708 pad 2: Net-(U701C--) -> Net-(U701D--)
- R710 pad 2: Net-(U701D-+) -> Net-(U701C-+)
- R715 pad 1: Net-(U701D--) -> Net-(U701C--)
- R716 pad 2: Net-(U701D--) -> Net-(U701C--)
- R804 pad 2: Net-(U801C-+) -> Net-(U801D-+)
- R807 pad 1: Net-(U801C--) -> Net-(U801D--)
- R808 pad 2: Net-(U801C--) -> Net-(U801D--)
- R810 pad 2: Net-(U801D-+) -> Net-(U801C-+)
- R815 pad 1: Net-(U801D--) -> Net-(U801C--)
- R816 pad 2: Net-(U801D--) -> Net-(U801C--)
- U701 pad 14: Net-(R712-Pad1) -> Net-(C707-Pad2)
- U701 pad 8: Net-(C707-Pad2) -> Net-(R712-Pad1)
- U702 pad 1: /Mux & Amplifier 1/In5 -> /Mux & Amplifier 1/In8
- U702 pad 12: /Mux & Amplifier 1/In4 -> /Mux & Amplifier 1/In2
- U702 pad 14: /Mux & Amplifier 1/In2 -> /Mux & Amplifier 1/In4
- U702 pad 4: /Mux & Amplifier 1/In8 -> /Mux & Amplifier 1/In5
- U703 pad 1: /Mux & Amplifier 1/In13 -> /Mux & Amplifier 1/In16
- U703 pad 12: /Mux & Amplifier 1/In12 -> /Mux & Amplifier 1/In10
- U703 pad 14: /Mux & Amplifier 1/In10 -> /Mux & Amplifier 1/In12
- U703 pad 4: /Mux & Amplifier 1/In16 -> /Mux & Amplifier 1/In13
- U801 pad 14: Net-(R812-Pad1) -> Net-(C807-Pad2)
- U801 pad 8: Net-(C807-Pad2) -> Net-(R812-Pad1)
- U802 pad 1: /Mux & Amplifier 2/In5 -> /Mux & Amplifier 2/In8
- U802 pad 12: /Mux & Amplifier 2/In4 -> /Mux & Amplifier 2/In2
- U802 pad 14: /Mux & Amplifier 2/In2 -> /Mux & Amplifier 2/In4
- U802 pad 4: /Mux & Amplifier 2/In8 -> /Mux & Amplifier 2/In5
- U803 pad 1: /Mux & Amplifier 2/In13 -> /Mux & Amplifier 2/In16
- U803 pad 12: /Mux & Amplifier 2/In12 -> /Mux & Amplifier 2/In10
- U803 pad 14: /Mux & Amplifier 2/In10 -> /Mux & Amplifier 2/In12
- U803 pad 4: /Mux & Amplifier 2/In16 -> /Mux & Amplifier 2/In13
Routing:
- net /Measurement & Control/Mux B: track 0.00 -> 124.3 mm, vias 0 -> 4
- net /Measurement & Control/Mux A: track 0.00 -> 123.8 mm, vias 0 -> 4
- net /Measurement & Control/Mux C: track 0.00 -> 121.9 mm, vias 0 -> 4
- net /Mux & Amplifier 2/In4: track 3.83 -> 52.4 mm
- net /Mux & Amplifier 2/In12: track 3.83 -> 52.3 mm
- net /Mux & Amplifier 1/In12: track 3.83 -> 51.7 mm
- net /Mux & Amplifier 1/In9: track 3.89 -> 51.5 mm
- net /Mux & Amplifier 2/In1: track 3.89 -> 51.5 mm
- net /Mux & Amplifier 2/In9: track 3.89 -> 51.4 mm
- net /Mux & Amplifier 1/In4: track 3.83 -> 51.1 mm
- net /Mux & Amplifier 1/In1: track 3.89 -> 49.5 mm
- net /Mux & Amplifier 2/In2: track 3.89 -> 42.8 mm
- net /Mux & Amplifier 2/In10: track 3.89 -> 42.5 mm
- net /Mux & Amplifier 1/In10: track 3.89 -> 42.5 mm
- net /Mux & Amplifier 1/In2: track 3.89 -> 40.9 mm
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
Commit message: Analogue layout
Parts:
- removed H105, H106: MountingHole, MountingHole:MountingHole_3.2mm_M3
- removed TP901, TP904: TestPoint, TestPoint:TestPoint_Pad_1.5x1.5mm
- C1201, C1202, C1203, C1204, C1205, C1206, C1207, C1208, C1301, C1302, C1303, C1304, C1305, C1306, C702, C801, C802, FB1201, FB1202, J901, JP901, R1103, R1104, R1106, R1107, R1201, R1202, R1203, R1204, R1301, R1302, R1303, R901, R903, R905, TP1201, TP1202, TP1203, TP1204, TP1205, TP702, TP802, TP902, TP903, TP905, TP906, TP907, TP908, TP909, TP910, TP911, TP912, TP913, TP914, TP915, TP916, U1101, U1201, U1202, U901, U902, Y901: moved to B.Cu
- moved C1301 380.1 mm to (312.1, 77.2)
- moved C1302 378.9 mm to (312.1, 74.7)
- moved C1303 377.9 mm to (312.1, 72.2)
- moved C1304 376.8 mm to (312.1, 69.7)
- moved C1305 375.9 mm to (312.1, 67.2)
- moved C1306 375.0 mm to (312.1, 64.6)
- moved R1301 374.2 mm to (312.1, 62.1)
- moved R1302 373.4 mm to (312.1, 59.6)
- moved R1303 372.8 mm to (312.1, 57.1)
- moved H103 358.9 mm to (300.0, 225.0)
- moved C901 339.8 mm to (320.5, 152.6)
- moved C902 339.8 mm to (320.5, 155.1)
- moved C903 339.8 mm to (320.5, 157.6)
- moved C904 339.8 mm to (320.5, 160.2)
- moved C905 339.8 mm to (320.5, 162.7)
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Connections:
- U902 pad 18: /Measurement & Control/Rx1 -> /Measurement & Control/Rx4
- U902 pad 20: /Measurement & Control/Rx1 -> /Measurement & Control/Rx4
- U902 pad 30: /Measurement & Control/Rx4 -> /Measurement & Control/Rx1
- U902 pad 33: /Measurement & Control/Rx4 -> /Measurement & Control/Rx1
- Y901 pad 1: Net-(Y901-Tri-State) -> unconnected-(Y901-Tri-State-Pad1)
Routing:
- net Net-(U702-X): track 0.00 -> 122.0 mm
- net Net-(U703-X): track 0.00 -> 119.1 mm
- net Net-(U802-X): track 0.00 -> 81.1 mm
- net Net-(U803-X): track 0.00 -> 67.9 mm
- net /Measurement & Control/Rx4: track 0.00 -> 23.9 mm
- net /Measurement & Control/Rx2: track 0.00 -> 21.9 mm
- net /Measurement & Control/Rx3: track 0.00 -> 21.4 mm
- net /Measurement & Control/Rx1: track 0.00 -> 21.2 mm
- net 1.65V: track 61.7 -> 68.8 mm
- net Net-(R711-Pad1): track 9.06 -> 11.2 mm
- net Net-(R712-Pad1): track 9.06 -> 11.2 mm
- net Net-(R811-Pad1): track 9.06 -> 11.2 mm
- net Net-(R812-Pad1): track 9.06 -> 11.2 mm
- net GND: track 1.02 -> 0.00 mm, vias 1 -> 0
- net /Measurement & Control/Mux Inhibit: track 1.02 -> 2.04 mm, vias 1 -> 2
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- added copper zone on B.Cu, net GND
Other:
- board text added: "X"
- board text added: "Y"

Commit message: Layout Progress
Parts:
- removed JP901: 3.3V STLINK, Jumper:SolderJumper-2_P1.3mm_Open_RoundedPad1.0x1.5mm
- C901, R902, R904, R906: moved to B.Cu
- moved C1205 192.2 mm to (352.0, 211.9)
- moved C1207 192.2 mm to (352.0, 206.9)
- moved TP1204 192.2 mm to (338.1, 200.7)
- moved FB1201 192.2 mm to (348.9, 201.4)
- moved U1202 173.6 mm to (332.0, 188.8)
- moved C1202 171.3 mm to (318.8, 200.4)
- moved C1204 171.3 mm to (318.8, 195.4)
- moved C1206 171.3 mm to (322.8, 200.4)
- moved C1208 171.3 mm to (322.8, 195.4)
- moved FB1202 171.3 mm to (319.7, 188.9)
- moved R1202 171.3 mm to (326.8, 200.4)
- moved R1204 171.3 mm to (326.8, 195.4)
- moved TP1203 171.3 mm to (308.9, 195.3)
- moved TP1205 171.3 mm to (308.9, 188.2)
- moved C901 60.6 mm to (264.0, 174.7)
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Routing:
- net 1.65V: track 68.8 -> 398.4 mm
- net +3.3VA: track 44.0 -> 265.3 mm, vias 0 -> 7
- net +3.3V: track 0.00 -> 47.2 mm
- net +5V: track 0.00 -> 20.5 mm
- net /Measurement & Control/OLED_SCL: track 0.00 -> 14.8 mm
- net /Measurement & Control/OLED_SDA: track 0.00 -> 14.3 mm
- net Net-(J1301-Pin_3): track 0.00 -> 12.3 mm
- net Net-(J1301-Pin_2): track 0.00 -> 11.9 mm
- net Net-(J1301-Pin_8): track 0.00 -> 10.2 mm
- net Net-(J1301-Pin_1): track 0.00 -> 10.2 mm
- net Net-(J1301-Pin_4): track 0.00 -> 10.1 mm
- net Net-(J1301-Pin_7): track 0.00 -> 9.94 mm
- net Net-(J1301-Pin_6): track 0.00 -> 9.59 mm
- net Net-(J901-D--PadA7): track 0.00 -> 7.02 mm
- net Net-(J901-D+-PadA6): track 0.00 -> 6.23 mm
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
Commit message: Layout
Parts:
- removed C1001, C1002, C1003, C1004: 100n, Capacitor_SMD:C_0603_1608Metric
- removed TP902, TP903: TestPoint, TestPoint:TestPoint_Pad_1.5x1.5mm
- removed U1001, U1002, U1003, U1004: TPIC6595, Package_SO:SOIC-20W_7.5x12.8mm_P1.27mm
- C701, C902, C903, C905, C907, C908, C909, C910, C911: moved to B.Cu
- moved C909 71.9 mm to (263.4, 193.0), turned to 180 degrees
- moved C910 66.2 mm to (263.4, 183.1), turned to 180 degrees
- moved C908 56.3 mm to (283.7, 191.5)
- moved C1205 55.3 mm to (297.1, 204.9)
- moved C1207 55.0 mm to (297.1, 203.4)
- moved FB1201 50.1 mm to (299.2, 195.3)
- moved C905 47.7 mm to (283.7, 193.0)
- moved C902 47.6 mm to (283.7, 185.4)
- moved C903 47.0 mm to (283.7, 186.9)
- moved TP1204 46.1 mm to (292.1, 199.6)
- moved C911 44.2 mm to (287.5, 184.4)
- moved TP906 35.6 mm to (291.0, 186.7)
- moved C907 35.1 mm to (287.5, 179.8)
- moved R902 26.3 mm to (287.5, 181.3)
- moved C901 24.9 mm to (287.5, 182.8)
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Routing:
- net /Measurement & Control/Mux Inhibit: track 2.04 -> 181.7 mm, vias 2 -> 5
- net +3.3VA: track 265.3 -> 373.4 mm, vias 7 -> 13
- net 1.65V: track 398.4 -> 461.5 mm
- net /Measurement & Control/Mux B: track 124.3 -> 179.4 mm, vias 4 -> 5
- net /Measurement & Control/Mux C: track 121.9 -> 176.8 mm, vias 4 -> 5
- net /Measurement & Control/Mux A: track 123.8 -> 173.0 mm, vias 4 -> 5
- net +3.3V: track 47.2 -> 82.4 mm
- net Net-(U702-X): track 122.0 -> 153.9 mm
- net /Measurement & Control/USB_DN: track 0.00 -> 23.9 mm
- net /Measurement & Control/OLED_SCL: track 14.8 -> 38.4 mm, vias 0 -> 2
- net /Measurement & Control/USB_DP: track 0.00 -> 22.9 mm
- net /Measurement & Control/OLED_SDA: track 14.3 -> 36.8 mm, vias 0 -> 2
- net /Measurement & Control/~{RST}: track 0.00 -> 18.0 mm
- net Net-(U802-X): track 81.1 -> 97.0 mm
- net /Measurement & Control/SWCLK: track 0.00 -> 15.3 mm
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Other:
- board text added: "3.3V"
- board text added: "GND"
- board text added: "RST"
- board text added: "SWCLK"
- board text added: "SWDIO"
