File: Input Hardware/PCB/Input Board/Input Board.kicad_pcb (KiCad board)
At the start: 2 copper layers, 255 x 180 mm, 415 parts, among them J1301 1.71" SSD1312 OLED, J901 USB_C_Receptacle_USB2.0_16P, SW1101 Rotary encoder, SW1102 Rotary encoder, U1101 74HC595, U1201 LM317_TO-252, U1202 LM317_TO-252, U301 ADA4891, U302 ADA4891, U401 ADA4891, U402 ADA4891, U501 ADA4891, U502 ADA4891, U601 ADA4891, U602 ADA4891, U701 ADA4891, U702 CD4051B, U703 CD4051B, U801 ADA4891, U802 CD4051B, U803 CD4051B, U901 USBLC6-2SC6, U902 STM32F303RBTx, Y901 ECS-2520MV-xxx-xx

Commit message: Layout Progress
Parts:
- removed R914: 10k, Resistor_SMD:R_0603_1608Metric
- added C1101: 100n, Capacitor_SMD:C_0603_1608Metric, B.Cu at (187.0, 56.0)
- added C1102: 100n, Capacitor_SMD:C_0603_1608Metric, B.Cu at (197.0, 56.0)
- added C1103: 100n, Capacitor_SMD:C_0603_1608Metric, B.Cu at (207.0, 56.0)
- added C1104: 100n, Capacitor_SMD:C_0603_1608Metric, B.Cu at (217.0, 56.0)
- added C1105: 100n, Capacitor_SMD:C_0603_1608Metric, B.Cu at (211.5, 56.7)
- added C1201: 100n, Capacitor_SMD:C_0603_1608Metric, B.Cu at (147.0, 56.0)
- added C1202: 100n, Capacitor_SMD:C_0603_1608Metric, B.Cu at (157.0, 56.0)
- added C1203: 100n, Capacitor_SMD:C_0603_1608Metric, B.Cu at (167.0, 56.0)
- added C1204: 100n, Capacitor_SMD:C_0603_1608Metric, B.Cu at (177.0, 56.0)
- added C1205: 100n, Capacitor_SMD:C_0603_1608Metric, B.Cu at (171.5, 56.7)
- added C1301: 100n, Capacitor_SMD:C_0603_1608Metric, B.Cu at (107.0, 56.0)
- added C1302: 100n, Capacitor_SMD:C_0603_1608Metric, B.Cu at (117.0, 56.0)
- added C1303: 100n, Capacitor_SMD:C_0603_1608Metric, B.Cu at (127.0, 56.0)
- added C1304: 100n, Capacitor_SMD:C_0603_1608Metric, B.Cu at (137.0, 56.0)
- added C1305: 100n, Capacitor_SMD:C_0603_1608Metric, B.Cu at (131.5, 56.7)
- added C1401: 100n, Capacitor_SMD:C_0603_1608Metric, B.Cu at (67.0, 56.0)
- added C1402: 100n, Capacitor_SMD:C_0603_1608Metric, B.Cu at (77.0, 56.0)
- added C1403: 100n, Capacitor_SMD:C_0603_1608Metric, B.Cu at (87.0, 56.0)
- added C1404: 100n, Capacitor_SMD:C_0603_1608Metric, B.Cu at (97.0, 56.0)
- added C1405: 100n, Capacitor_SMD:C_0603_1608Metric, B.Cu at (91.5, 56.7)
- added C1701: 100u, Capacitor_SMD:C_Elec_4x5.8, B.Cu at (252.0, 67.8)
- added JP901: SolderJumper_2_Bridged, Jumper:SolderJumper-2_P1.3mm_Bridged_RoundedPad1.0x1.5mm, B.Cu at (277.9, 169.8)
- added R1503: 10k, Resistor_SMD:R_0603_1608Metric, F.Cu at (258.0, 104.6)
- added R1504: 10k, Resistor_SMD:R_0603_1608Metric, F.Cu at (258.0, 107.1)
- added U1101: 74HCS95, Package_DFN_QFN:DHVQFN-16-1EP_2.5x3.5mm_P0.5mm_EP1x2mm, B.Cu at (210.0, 53.2)
- added U1102: DRV8837, Package_SON:WSON-8-1EP_2x2mm_P0.5mm_EP0.9x1.6mm, B.Cu at (215.0, 56.0)
- added U1103: DRV8837, Package_SON:WSON-8-1EP_2x2mm_P0.5mm_EP0.9x1.6mm, B.Cu at (205.0, 56.0)
- added U1104: DRV8837, Package_SON:WSON-8-1EP_2x2mm_P0.5mm_EP0.9x1.6mm, B.Cu at (195.0, 56.0)
- added U1105: DRV8837, Package_SON:WSON-8-1EP_2x2mm_P0.5mm_EP0.9x1.6mm, B.Cu at (185.0, 56.0)
- added U1201: 74HCS95, Package_DFN_QFN:DHVQFN-16-1EP_2.5x3.5mm_P0.5mm_EP1x2mm, B.Cu at (170.0, 53.2)
- added U1202: DRV8837, Package_SON:WSON-8-1EP_2x2mm_P0.5mm_EP0.9x1.6mm, B.Cu at (175.0, 56.0)
- added U1203: DRV8837, Package_SON:WSON-8-1EP_2x2mm_P0.5mm_EP0.9x1.6mm, B.Cu at (165.0, 56.0)
- added U1204: DRV8837, Package_SON:WSON-8-1EP_2x2mm_P0.5mm_EP0.9x1.6mm, B.Cu at (155.0, 56.0)
- added U1205: DRV8837, Package_SON:WSON-8-1EP_2x2mm_P0.5mm_EP0.9x1.6mm, B.Cu at (145.0, 56.0)
- added U1301: 74HCS95, Package_DFN_QFN:DHVQFN-16-1EP_2.5x3.5mm_P0.5mm_EP1x2mm, B.Cu at (130.0, 53.2)
- added U1302: DRV8837, Package_SON:WSON-8-1EP_2x2mm_P0.5mm_EP0.9x1.6mm, B.Cu at (135.0, 56.0)
- added U1303: DRV8837, Package_SON:WSON-8-1EP_2x2mm_P0.5mm_EP0.9x1.6mm, B.Cu at (125.0, 56.0)
- added U1304: DRV8837, Package_SON:WSON-8-1EP_2x2mm_P0.5mm_EP0.9x1.6mm, B.Cu at (115.0, 56.0)
- added U1305: DRV8837, Package_SON:WSON-8-1EP_2x2mm_P0.5mm_EP0.9x1.6mm, B.Cu at (105.0, 56.0)
- added U1401: 74HCS95, Package_DFN_QFN:DHVQFN-16-1EP_2.5x3.5mm_P0.5mm_EP1x2mm, B.Cu at (90.0, 53.2)
- added U1402: DRV8837, Package_SON:WSON-8-1EP_2x2mm_P0.5mm_EP0.9x1.6mm, B.Cu at (95.0, 56.0)
- added U1403: DRV8837, Package_SON:WSON-8-1EP_2x2mm_P0.5mm_EP0.9x1.6mm, B.Cu at (85.0, 56.0)
- added U1404: DRV8837, Package_SON:WSON-8-1EP_2x2mm_P0.5mm_EP0.9x1.6mm, B.Cu at (75.0, 56.0)
- added U1405: DRV8837, Package_SON:WSON-8-1EP_2x2mm_P0.5mm_EP0.9x1.6mm, B.Cu at (65.0, 56.0)
- C706, C707, C806, C807: value 39p -> 33p
- C708, C709, C710, C711, C808, C809, C810, C811: value 56p -> 39p
- C904, C906: moved to B.Cu
- R911: value 10k -> 1M
- U1501: renamed from U1101; footprint Package_SO:SOIC-16_3.9x9.9mm_P1.27mm -> Package_DFN_QFN:DHVQFN-16-1EP_2.5x3.5mm_P0.5mm_EP1x2mm
- moved TP1702 49.2 mm to (290.8, 54.6)
- moved C904 36.9 mm to (277.5, 177.0), turned to 90 degrees
- moved U1501 32.2 mm to (263.9, 117.5)
- moved C906 30.7 mm to (283.8, 180.2)
- moved C1702 27.6 mm to (278.4, 56.6)
- moved C1704 27.6 mm to (278.4, 51.6)
- moved R1701 27.6 mm to (286.4, 56.6)
- moved R1703 27.6 mm to (286.4, 51.6)
- moved TP1704 8.98 mm to (296.4, 207.5)
- moved R1508 6.31 mm to (273.5, 120.1), turned to 180 degrees
- moved R909 3.72 mm to (325.2, 169.5)
- moved R913 3.72 mm to (329.3, 162.0)
- moved C912 3.72 mm to (321.2, 164.5)
- moved R907 3.72 mm to (325.2, 164.5)
- moved R908 3.72 mm to (325.2, 167.0)
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- renumbered C1101 to C1501, C1301 to C1601, C1302 to C1602, C1303 to C1603, C1304 to C1604, C1305 to C1605, C1306 to C1606, C1201 to C1702, C1202 to C1703, C1203 to C1704, C1204 to C1705, C1205 to C1706, C1206 to C1707, C1207 to C1708, C1208 to C1709, D1101 to D1501, D1102 to D1502, D1104 to D1503, D1103 to D1504, D1105 to D1505, D1107 to D1506, D1106 to D1507, D1108 to D1508, D1109 to D1509, D1110 to D1510, FB1201 to FB1701, FB1202 to FB1702, J1301 to J1601, R1101 to R1501, R1102 to R1502, R1104 to R1505, R1103 to R1506, R1105 to R1507, R1107 to R1508, R1108 to R1509, R1106 to R1510, R1109 to R1511, R1110 to R1512, R1301 to R1601, R1302 to R1602, R1303 to R1603, R1201 to R1701, R1202 to R1702, R1203 to R1703, R1204 to R1704, S1101 to S1501, S1102 to S1502, SW1101 to SW1501, SW1102 to SW1502, TP1201 to TP1701, TP1202 to TP1702, TP1203 to TP1703, TP1204 to TP1704, TP1205 to TP1705, TP905 to TP901, TP906 to TP902, TP907 to TP903, TP908 to TP904, TP909 to TP905, TP910 to TP906, TP911 to TP907, TP912 to TP908, TP913 to TP909, TP914 to TP910, TP915 to TP911, TP916 to TP912, U1201 to U1701, U1202 to U1702
Connections:
- net /Measurement & Control/TX_DSO renamed /Measurement & Control/TX_SDO
- C703 pad 2: GNDA -> GND
- C803 pad 2: GNDA -> GND
- L1001 pad 1: Net-(U1001-DRAIN0) -> /Transmit Coils/Dual H-Bridge 1/OUT1
- L1001 pad 2: +5V -> GND
- L1002 pad 1: Net-(U1001-DRAIN1) -> /Transmit Coils/Dual H-Bridge 1/OUT2
- L1002 pad 2: +5V -> GND
- L1003 pad 1: Net-(U1001-DRAIN2) -> /Transmit Coils/Dual H-Bridge 1/OUT3
- L1003 pad 2: +5V -> GND
- L1004 pad 1: Net-(U1001-DRAIN3) -> /Transmit Coils/Dual H-Bridge 1/OUT4
- L1004 pad 2: +5V -> GND
- L1005 pad 1: Net-(U1001-DRAIN4) -> /Transmit Coils/Dual H-Bridge 1/OUT5
- L1005 pad 2: +5V -> GND
- L1006 pad 1: Net-(U1001-DRAIN5) -> /Transmit Coils/Dual H-Bridge 1/OUT6
- L1006 pad 2: +5V -> GND
- L1007 pad 1: Net-(U1001-DRAIN6) -> /Transmit Coils/Dual H-Bridge 1/OUT7
- L1007 pad 2: +5V -> GND
- L1008 pad 1: Net-(U1001-DRAIN7) -> /Transmit Coils/Dual H-Bridge 1/OUT8
- L1008 pad 2: +5V -> GND
- L1009 pad 1: Net-(U1002-DRAIN0) -> /Transmit Coils/Dual H-Bridge 2/OUT1
- L1009 pad 2: +5V -> GND
- L1010 pad 1: Net-(U1002-DRAIN1) -> /Transmit Coils/Dual H-Bridge 2/OUT2
- L1010 pad 2: +5V -> GND
- L1011 pad 1: Net-(U1002-DRAIN2) -> /Transmit Coils/Dual H-Bridge 2/OUT3
- L1011 pad 2: +5V -> GND
- L1012 pad 1: Net-(U1002-DRAIN3) -> /Transmit Coils/Dual H-Bridge 2/OUT4
- L1012 pad 2: +5V -> GND
- L1013 pad 1: Net-(U1002-DRAIN4) -> /Transmit Coils/Dual H-Bridge 2/OUT5
- L1013 pad 2: +5V -> GND
- L1014 pad 1: Net-(U1002-DRAIN5) -> /Transmit Coils/Dual H-Bridge 2/OUT6
- L1014 pad 2: +5V -> GND
- L1015 pad 1: Net-(U1002-DRAIN6) -> /Transmit Coils/Dual H-Bridge 2/OUT7
- L1015 pad 2: +5V -> GND
- L1016 pad 1: Net-(U1002-DRAIN7) -> /Transmit Coils/Dual H-Bridge 2/OUT8
- L1016 pad 2: +5V -> GND
- L1017 pad 1: Net-(U1003-DRAIN0) -> /Transmit Coils/Dual H-Bridge 3/OUT1
- L1017 pad 2: +5V -> GND
- L1018 pad 1: Net-(U1003-DRAIN1) -> /Transmit Coils/Dual H-Bridge 3/OUT2
- L1018 pad 2: +5V -> GND
- L1019 pad 1: Net-(U1003-DRAIN2) -> /Transmit Coils/Dual H-Bridge 3/OUT3
- L1019 pad 2: +5V -> GND
- L1020 pad 1: Net-(U1003-DRAIN3) -> /Transmit Coils/Dual H-Bridge 3/OUT4
- L1020 pad 2: +5V -> GND
- L1021 pad 1: Net-(U1003-DRAIN4) -> /Transmit Coils/Dual H-Bridge 3/OUT5
- L1021 pad 2: +5V -> GND
- L1022 pad 1: Net-(U1003-DRAIN5) -> /Transmit Coils/Dual H-Bridge 3/OUT6
- L1022 pad 2: +5V -> GND
- L1023 pad 1: Net-(U1003-DRAIN6) -> /Transmit Coils/Dual H-Bridge 3/OUT7
- L1023 pad 2: +5V -> GND
- L1024 pad 1: Net-(U1003-DRAIN7) -> /Transmit Coils/Dual H-Bridge 3/OUT8
- L1024 pad 2: +5V -> GND
- L1025 pad 1: Net-(U1004-DRAIN0) -> /Transmit Coils/Dual H-Bridge 4/OUT1
- L1025 pad 2: +5V -> GND
- L1026 pad 1: Net-(U1004-DRAIN1) -> /Transmit Coils/Dual H-Bridge 4/OUT2
- L1026 pad 2: +5V -> GND
- L1027 pad 1: Net-(U1004-DRAIN2) -> /Transmit Coils/Dual H-Bridge 4/OUT3
- L1027 pad 2: +5V -> GND
- L1028 pad 1: Net-(U1004-DRAIN3) -> /Transmit Coils/Dual H-Bridge 4/OUT4
- L1028 pad 2: +5V -> GND
- L1029 pad 1: Net-(U1004-DRAIN4) -> /Transmit Coils/Dual H-Bridge 4/OUT5
- L1029 pad 2: +5V -> GND
- L1030 pad 1: Net-(U1004-DRAIN5) -> /Transmit Coils/Dual H-Bridge 4/OUT6
- L1030 pad 2: +5V -> GND
- L1031 pad 1: Net-(U1004-DRAIN6) -> /Transmit Coils/Dual H-Bridge 4/OUT7
- L1031 pad 2: +5V -> GND
- L1032 pad 1: Net-(U1004-DRAIN7) -> /Transmit Coils/Dual H-Bridge 4/OUT8
- L1032 pad 2: +5V -> GND
- R910 pad 2: /Measurement & Control/TX_~{OE} -> /Measurement & Control/UI_SRCLK
- R912 pad 2: /Measurement & Control/UI_SRCLK -> /Measurement & Control/UI_RCLK
- R913 pad 2: /Measurement & Control/UI_RCLK -> /Measurement & Control/UI_SER
- TP901 pad 1: Net-(JP901-A) -> +3.3V
- U701 pad 11: GNDA -> GND
- U801 pad 11: GNDA -> GND
- U902 pad 56: /Measurement & Control/TX_~{OE} -> unconnected-(U902-PB4-Pad56)
Routing:
- net (no net): track 0.00 -> 7539.2 mm
- net /Measurement & Control/TX_SRCLK: track 1.55 -> 282.3 mm, vias 1 -> 6
- net +5V: track 22.6 -> 300.6 mm, vias 0 -> 37
- net /Measurement & Control/TX_RCLK: track 3.82 -> 279.1 mm, vias 1 -> 6
- net GND: track 0.00 -> 191.9 mm, vias 205 -> 372
- net /Measurement & Control/TX_SDO: track 3.06 -> 152.5 mm, vias 1 -> 3
- net /Measurement & Control/USB_DP: track 22.9 -> 128.7 mm
- net /Measurement & Control/OLED_SCL: track 38.4 -> 144.0 mm
- net /Measurement & Control/OLED_SDA: track 36.8 -> 142.2 mm
- net /Measurement & Control/USB_DN: track 23.9 -> 129.2 mm
- net /Transmit Coils/Dual H-Bridge 1/QH': track 0.00 -> 42.9 mm, vias 0 -> 2
- net /Transmit Coils/QH': track 0.00 -> 42.9 mm, vias 0 -> 2
- net /Transmit Coils/Dual H-Bridge 3/QH': track 0.00 -> 42.9 mm, vias 0 -> 2
- net Net-(U1401-QH): track 0.00 -> 27.4 mm
- net Net-(U1301-QH): track 0.00 -> 27.4 mm
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- added copper zone on B.Cu, net (none)
- added copper zone on F.Cu, net (none)
- added copper zone on F.Cu, net GND
Other:
- board text added: "Complex Plotter Input Board"
- board text added: "HAYES - Second Year Group Project"
