File: Input Hardware/PCB/Input Board/Input Board.kicad_pcb (KiCad board)
At the start: 2 copper layers, 255 x 180 mm, 458 parts, among them J1601 1.71" SSD1312 OLED, J901 USB_C_Receptacle_USB2.0_16P, SW1501 Rotary encoder, SW1502 Rotary encoder, U1101 74HCS95, U1102 DRV8837, U1103 DRV8837, U1104 DRV8837, U1105 DRV8837, U1201 74HCS95, U1202 DRV8837, U1203 DRV8837, U1204 DRV8837, U1205 DRV8837, U1301 74HCS95, U1302 DRV8837, U1303 DRV8837, U1304 DRV8837, U1305 DRV8837, U1401 74HCS95, U1402 DRV8837, U1403 DRV8837, U1404 DRV8837, U1405 DRV8837, U1501 74HC595, U1701 LM317_TO-252, U1702 LM317_TO-252, U301 ADA4891, U302 ADA4891, U401 ADA4891, U402 ADA4891, U501 ADA4891, U502 ADA4891, U601 ADA4891, U602 ADA4891, U701 ADA4891, U702 CD4051B, U703 CD4051B, U801 ADA4891, U802 CD4051B, U803 CD4051B, U901 USBLC6-2SC6, U902 STM32F303RBTx, Y901 ECS-2520MV-xxx-xx

Commit message: changes
Parts:
- added C1: 100n, Capacitor_SMD:C_0603_1608Metric, F.Cu at (352.1, 123.7)
- added C2: 100n, Capacitor_SMD:C_0603_1608Metric, F.Cu at (352.1, 126.2)
- added C3: 100n, Capacitor_SMD:C_0603_1608Metric, F.Cu at (352.1, 128.7)
- added C4: 1u, Capacitor_SMD:C_Elec_4x5.8, F.Cu at (359.9, 125.3)
- added D1: ~, LED_SMD:LED_0603_1608Metric, F.Cu at (358.2, 129.5)
- added R1: 1k, Resistor_SMD:R_0603_1608Metric, F.Cu at (352.1, 131.2)
- added R2: 1k, Resistor_SMD:R_0603_1608Metric, F.Cu at (352.1, 133.7)
- added R3: 1k, Resistor_SMD:R_0603_1608Metric, F.Cu at (352.1, 136.2)
- added R4: 180, Resistor_SMD:R_0603_1608Metric, F.Cu at (362.2, 129.5)
- added SW1: SW_Push, Button_Switch_SMD:SW_Push_1P1T_XKB_TS-1187A, F.Cu at (343.5, 120.3)
- added SW2: SW_Push, Button_Switch_SMD:SW_Push_1P1T_XKB_TS-1187A, F.Cu at (343.5, 128.8)
- added SW3: SW_Push, Button_Switch_SMD:SW_Push_1P1T_XKB_TS-1187A, F.Cu at (343.5, 137.2)
- R1501, R1502, R1505, R1506, R1507, R1508, R1509, R1510, R1511, R1512: value TBD -> 180
Connections:
- U902 pad 14: /Measurement &amp; Control/TSC_1 -> /Measurement & Control/TSC_1
- U902 pad 15: /Measurement &amp; Control/TSC_2 -> /Measurement & Control/TSC_2
- U902 pad 16: /Measurement &amp; Control/TSC_3 -> /Measurement & Control/TSC_3
Routing:
- net /Measurement &amp; Control/TSC_3: track 13.5 -> 0.00 mm
- net /Measurement & Control/TSC_3: track 0.00 -> 13.5 mm
- net /Measurement &amp; Control/TSC_2: track 13.4 -> 0.00 mm
- net /Measurement & Control/TSC_2: track 0.00 -> 13.4 mm
- net /Measurement &amp; Control/TSC_1: track 13.3 -> 0.00 mm
- net /Measurement & Control/TSC_1: track 0.00 -> 13.3 mm

Commit message: minor layout changes
Parts:
- removed C1, C2, C3: 100n, Capacitor_SMD:C_0603_1608Metric
- C4, R1, R2, R3, SW1, SW2, SW3: moved to B.Cu
- moved C4 128.6 mm to (245.5, 66.5), turned to -90 degrees
- moved SW1 103.8 mm to (247.5, 159.9)
- moved SW2 81.7 mm to (268.0, 159.9)
- moved R1 79.9 mm to (287.5, 178.2), turned to 180 degrees
- moved R2 77.6 mm to (287.5, 176.8), turned to 180 degrees
- moved R3 75.5 mm to (287.5, 175.2), turned to 180 degrees
- moved SW3 60.5 mm to (287.5, 160.0)
- moved FB1701 5.85 mm to (297.9, 201.0)
- moved C1701 1.21 mm to (245.5, 59.9)
- moved J901 0.25 mm to (255.0, 53.6)
Routing:
- net /Measurement & Control/TSC_3: track 13.5 -> 46.1 mm
- net /Measurement & Control/TSC_2: track 13.4 -> 44.1 mm
- net /Measurement & Control/TSC_1: track 13.3 -> 43.2 mm
- net /Measurement & Control/TX_SRCLK: track 282.3 -> 274.4 mm
- net /Measurement & Control/TX_SDO: track 152.5 -> 144.9 mm
- net /Measurement & Control/TX_RCLK: track 279.1 -> 271.7 mm
- net +5V: track 306.0 -> 309.7 mm
- net /Measurement & Control/TSC_CS: track 5.70 -> 6.41 mm
