File: Input Hardware/PCB/Input Board/Input Board.kicad_pcb (KiCad board)
At the start: 2 copper layers, 255 x 180 mm, 458 parts, among them J1601 1.71" SSD1312 OLED, J901 USB_C_Receptacle_USB2.0_16P, SW1501 Rotary encoder, SW1502 Rotary encoder, U1101 74HCS95, U1102 DRV8837, U1103 DRV8837, U1104 DRV8837, U1105 DRV8837, U1201 74HCS95, U1202 DRV8837, U1203 DRV8837, U1204 DRV8837, U1205 DRV8837, U1301 74HCS95, U1302 DRV8837, U1303 DRV8837, U1304 DRV8837, U1305 DRV8837, U1401 74HCS95, U1402 DRV8837, U1403 DRV8837, U1404 DRV8837, U1405 DRV8837, U1501 74HC595, U1701 LM317_TO-252, U1702 LM317_TO-252, U301 ADA4891, U302 ADA4891, U401 ADA4891, U402 ADA4891, U501 ADA4891, U502 ADA4891, U601 ADA4891, U602 ADA4891, U701 ADA4891, U702 CD4051B, U703 CD4051B, U801 ADA4891, U802 CD4051B, U803 CD4051B, U901 USBLC6-2SC6, U902 STM32F303RBTx, Y901 ECS-2520MV-xxx-xx

Commit message: USB & OLED wiring
Parts:
- moved C1701 10.8 mm to (244.3, 60.2), turned to 90 degrees
Routing:
- net /Measurement & Control/OLED_SDA: track 142.5 -> 169.5 mm
- net /Measurement & Control/OLED_SCL: track 144.3 -> 167.6 mm
- net /Measurement & Control/USB_DP: track 129.0 -> 144.9 mm
- net /Measurement & Control/USB_DN: track 129.5 -> 145.1 mm
- net +5V: track 300.6 -> 306.0 mm

Commit message: minor schematic changes and value assignment
Parts:
- moved J901 0.31 mm to (255.0, 53.4)
Changed lines of the file:
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@@
 	(footprint "Connector_USB:USB_C_Receptacle_GCT_USB4110"
 		(layer "B.Cu")
-		(at 255 53.71)
+		(at 255 53.395)
 		(descr "USB 2.0 Type C Receptacle, GCT, 16P, top mounted, horizontal, 5A, https://gct.co/files/drawings/usb4110.pdf")
 		(tags "USB 2.0 C Type-C Receptacle SMD 16P 16C USB4110-GF-A")

Commit message: Layout Progress
Parts:
- removed the C1707 at (322.8, 200.4)
- removed the C1709 at (322.8, 195.4)
- removed the C905 at (283.7, 193.0)
- removed the C907 at (287.5, 179.8)
- removed FB1702: 120, Inductor_SMD:L_1206_3216Metric
- removed TP1705, TP911: TestPoint, TestPoint:TestPoint_Pad_1.5x1.5mm
- removed the TP910 at (269.7, 177.0)
- added C1502: 100n, Capacitor_SMD:C_0603_1608Metric, B.Cu at (257.5, 162.2)
- added C1503: 100n, Capacitor_SMD:C_0603_1608Metric, B.Cu at (277.5, 162.2)
- added C1504: 100n, Capacitor_SMD:C_0603_1608Metric, B.Cu at (277.5, 157.8)
- added C1701: 1u, Capacitor_SMD:C_0603_1608Metric, B.Cu at (265.2, 57.9)
- added D1701: ~, LED_SMD:LED_0603_1608Metric, B.Cu at (283.9, 57.9)
- added R1502: 10k, Resistor_SMD:R_0603_1608Metric, B.Cu at (257.5, 160.8)
- added R1510: 10k, Resistor_SMD:R_0603_1608Metric, B.Cu at (277.5, 160.8)
- added R1514: 10k, Resistor_SMD:R_0603_1608Metric, B.Cu at (277.5, 159.2)
- added R1701: 180, Resistor_SMD:R_0603_1608Metric, B.Cu at (282.4, 57.9)
- added SW1501: SW_Push, Button_Switch_SMD:SW_SPST_B3S-1000, F.Cu at (247.5, 160.0)
- added SW1504: SW_Push, Button_Switch_SMD:SW_SPST_B3S-1000, F.Cu at (267.5, 160.0)
- added SW1505: SW_Push, Button_Switch_SMD:SW_SPST_B3S-1000, F.Cu at (287.5, 160.0)
- C1501, R907, R908, R909, R910, R911, R912, R913: moved to B.Cu
- C911: renamed from C912; moved to B.Cu
- R1501, R1505: value TBD -> 180
- R1503: renamed from R1504; moved to B.Cu
- R1504: renamed from R1502; value TBD -> 180
- R1506: renamed from R1503; moved to B.Cu
- R1507: renamed from R1508; value TBD -> 180
- R1508: renamed from R1506; value TBD -> 180
- R1509: renamed from R1507; value TBD -> 180
- R1511: renamed from R1509; value TBD -> 180
- R1512: renamed from R1510; value TBD -> 180
- R1513: renamed from R1511; value TBD -> 180
- R1515: renamed from R1512; value TBD -> 180
- moved R909 150.0 mm to (226.8, 56.4), turned to -90 degrees
- moved R908 149.5 mm to (224.8, 56.4), turned to -90 degrees
- moved R907 149.0 mm to (222.7, 56.4), turned to -90 degrees
- moved R913 77.6 mm to (258.5, 130.3)
- moved R912 75.7 mm to (258.5, 132.8)
- moved R910 72.7 mm to (258.5, 137.8)
- moved R1501 63.0 mm to (250.2, 144.9)
- moved R1504 63.0 mm to (250.2, 147.4)
- moved D1501 63.0 mm to (258.3, 142.4)
- moved D1503 63.0 mm to (258.3, 145.0)
- moved R911 53.3 mm to (279.9, 177.0), turned to -90 degrees
- moved D1508 53.3 mm to (271.6, 144.3)
- moved D1506 53.3 mm to (267.5, 149.5)
- moved R1509 53.3 mm to (259.5, 151.7)
- moved R1511 53.3 mm to (263.5, 144.1)
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- renumbered C1701 to C1702, C1702 to C1703, C1703 to C1704, C1704 to C1705, C1705 to C1706, C1706 to C1707, C1708 to C1709, C906 to C905, C908 to C907, C909 to C908, C910 to C909, C911 to C910, D1503 to D1502, D1502 to D1503, D1506 to D1504, D1504 to D1505, D1505 to D1506, R1701 to R1702, R1702 to R1703, R1703 to R1704, R1704 to R1705, SW1501 to SW1503, TP912 to TP910
Connections:
- C1705 pad 1: 3.3V -> +3.3V
- C1706 pad 1: Net-(U1702-VO) -> 1.65V
- FB1701 pad 2: 3.3V -> +3.3V
- JP901 pad 1: /Measurement & Control/S_PUSH -> /Measurement & Control/Push_3
- R1704 pad 1: 3.3V -> +3.3V
- R1705 pad 1: Net-(U1702-VO) -> 1.65V
- TP1702 pad 1: 3.3V -> +3.3V
- TP1703 pad 1: Net-(U1702-VO) -> 1.65V
- U1701 pad 2: 3.3V -> +3.3V
- U1702 pad 2: Net-(U1702-VO) -> 1.65V
- U902 pad 14: /Measurement &amp; Control/TSC_1 -> unconnected-(U902-PA0-Pad14)
- U902 pad 15: /Measurement &amp; Control/TSC_2 -> unconnected-(U902-PA1-Pad15)
- U902 pad 16: /Measurement &amp; Control/TSC_3 -> unconnected-(U902-PA2-Pad16)
- U902 pad 17: /Measurement & Control/TSC_CS -> unconnected-(U902-PA3-Pad17)
- U902 pad 50: Net-(U902-PA15) -> /Measurement & Control/Push_1
- U902 pad 56: unconnected-(U902-PB4-Pad56) -> /Measurement & Control/Push_2
- U902 pad 59: Net-(U902-PB7) -> /Measurement & Control/Push_3
Routing:
- net +5V: track 306.0 -> 567.1 mm, vias 37 -> 44
- net +3.3V: track 82.8 -> 264.7 mm, vias 0 -> 2
- net /Measurement & Control/UI_SER: track 12.6 -> 79.4 mm, vias 1 -> 2
- net /Measurement & Control/UI_RCLK: track 12.7 -> 77.9 mm, vias 1 -> 0
- net /Measurement & Control/UI_SRCLK: track 12.7 -> 75.6 mm, vias 1 -> 2
- net /Measurement & Control/Push_1: track 0.00 -> 49.8 mm, vias 0 -> 2
- net /User Input/LED_IX: track 0.00 -> 47.9 mm
- net /User Input/LED_IY: track 0.00 -> 46.2 mm
- net /Measurement & Control/Push_3: track 0.00 -> 37.9 mm, vias 0 -> 1
- net /Measurement & Control/TX_RCLK: track 279.1 -> 313.3 mm
- net /Measurement & Control/Push_2: track 0.00 -> 34.1 mm, vias 0 -> 1
- net /Measurement & Control/TX_SDO: track 152.5 -> 185.5 mm, vias 3 -> 2
- net /Measurement & Control/TX_SRCLK: track 282.3 -> 313.5 mm, vias 6 -> 7
- net /Measurement & Control/I_COM: track 0.00 -> 16.9 mm
- net /Measurement & Control/O_COM: track 0.00 -> 16.5 mm, vias 0 -> 2
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
Commit message: Layout Progress
Parts:
- R1501, R1504, R1505, R1507, R1508, R1509, R1511, R1512, R1513, R1515, R1701: value 180 -> 220
- moved R1703 30.1 mm to (297.6, 193.2), turned to 180 degrees
- moved R1705 29.5 mm to (297.6, 191.8), turned to 180 degrees
- moved C1706 21.2 mm to (297.6, 194.8), turned to 180 degrees
- moved U1702 16.8 mm to (298.7, 188.4)
- moved R901 15.0 mm to (257.0, 66.3), turned to 180 degrees
- moved R1509 10.2 mm to (268.9, 147.8)
- moved R1511 9.32 mm to (272.2, 140.9)
- moved TP1703 7.71 mm to (301.5, 197.3)
- moved D1506 6.77 mm to (274.3, 150.3)
- moved R913 6.66 mm to (256.0, 136.4), turned to 180 degrees
- moved R912 6.22 mm to (256.0, 138.5), turned to 180 degrees
- moved C1704 4.20 mm to (297.3, 185.1), turned to 180 degrees
- moved R910 3.68 mm to (256.0, 140.5), turned to 180 degrees
- moved D1501 3.35 mm to (257.0, 145.5)
- moved D1503 3.35 mm to (257.0, 148.1)
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Connections:
- U902 pad 2: /Measurement & Control/O_LEFT -> /Measurement & Control/O_CENTER
- U902 pad 4: /Measurement & Control/O_CENTER -> /Measurement & Control/O_UP
- U902 pad 61: /Measurement & Control/O_UP -> /Measurement & Control/O_LEFT
Routing:
- net /Measurement & Control/O_UP: track 0.00 -> 126.0 mm, vias 0 -> 4
- net /Measurement & Control/O_LEFT: track 0.00 -> 119.4 mm, vias 0 -> 4
- net /Measurement & Control/I_COM: track 16.9 -> 129.5 mm, vias 0 -> 1
- net /Measurement & Control/O_RIGHT: track 0.00 -> 109.0 mm, vias 0 -> 4
- net /Measurement & Control/O_CENTER: track 0.00 -> 107.1 mm, vias 0 -> 4
- net /Measurement & Control/O_DOWN: track 0.00 -> 105.9 mm, vias 0 -> 4
- net +5V: track 567.1 -> 635.2 mm, vias 44 -> 50
- net /Measurement & Control/S_PUSH: track 0.00 -> 44.2 mm
- net /Measurement & Control/S_B: track 0.00 -> 40.4 mm
- net /Measurement & Control/O_COM: track 16.5 -> 56.3 mm
- net /Measurement & Control/S_A: track 0.00 -> 36.3 mm
- net +3.3VA: track 401.7 -> 421.0 mm
- net +3.3V: track 264.7 -> 280.0 mm, vias 2 -> 3
- net 1.65V: track 463.2 -> 476.1 mm
- net /Measurement & Control/~{RST}: track 10.8 -> 18.2 mm
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