File: Input Hardware/PCB/Input Board/Input.kicad_sch (KiCad schematic)
At the start: 26 parts, among them SW1101 Rotary encoder, SW1102 Rotary encoder, U1101 74HC595

Commit message: package type change
Parts:
- U1101: footprint Package_SO:SOIC-16_3.9x9.9mm_P1.27mm -> Package_DFN_QFN:DHVQFN-16-1EP_2.5x3.5mm_P0.5mm_EP1x2mm
Changed lines of the file:
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@@
 			)
 		)
-		(property "Footprint" "Package_SO:SOIC-16_3.9x9.9mm_P1.27mm"
+		(property "Footprint" "Package_DFN_QFN:DHVQFN-16-1EP_2.5x3.5mm_P0.5mm_EP1x2mm"
 			(at 44.45 63.5 0)
 			(effects

Commit message: Schematic Cleanup
Parts:
- added R? (x2): 10k, Resistor_SMD:R_0603_1608Metric, symbol Device:R
Connections:
- net GND: now also R?.2
- net I_COM: now also R?.2
- net O_COM: now also R?.1
- new net +3.3V: R?.1

Commit message: Layout Progress
Parts:
- gave numbers to parts that had none: 2
- renumbered C1101 to C1501, D1101 to D1501, D1102 to D1502, D1104 to D1503, D1103 to D1504, D1105 to D1505, D1107 to D1506, D1106 to D1507, D1108 to D1508, D1109 to D1509, D1110 to D1510, R1101 to R1501, R1102 to R1502, R1104 to R1505, R1103 to R1506, R1105 to R1507, R1107 to R1508, R1108 to R1509, R1106 to R1510, R1109 to R1511, R1110 to R1512, S1101 to S1501, S1102 to S1502, SW1101 to SW1501, SW1102 to SW1502, U1101 to U1501

Commit message: minor schematic changes and value assignment
Parts:
- added C? (x3): 100n, Capacitor_SMD:C_0603_1608Metric, symbol Device:C
- added R? (x3): 1k, Resistor_SMD:R_0603_1608Metric, symbol Device:R
- added SW? (x3): SW_Push, Button_Switch_SMD:SW_SPST_B3S-1000, symbol Switch:SW_Push
- R1501, R1502, R1505, R1506, R1507, R1508, R1509, R1510, R1511, R1512: value TBD -> 220
Connections:
- net +5V: now also C?.1, C?.1, C?.1, R?.2, R?.2, R?.2
- net GND: now also SW?.2, SW?.2, SW?.2
- net TSC_1: now also C?.2, R?.1, SW?.1
- net TSC_2: now also C?.2, R?.1, SW?.1
- net TSC_3: now also C?.2, R?.1, SW?.1
- no-connect marks 7 -> 4
Other:
- note removed: "Do you just wanna make all the TBD LED resistors 220/330ohm?"
- note removed: "what is this?"
- moved on the sheet: C1501, D1501, D1502, D1503, D1504, D1505, D1506, D1507, D1508, D1509, D1510, R1501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

Commit message: updates
Parts:
- R1501, R1502, R1505, R1506, R1507, R1508, R1509, R1510, R1511, R1512: value 220 -> 180
Changed lines of the file:
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@@
 			)
 		)
-		(property "Value" "220"
+		(property "Value" "180"
 			(at 97.79 128.27 90)
 			(effects
@@
 			)
 		)
-		(property "Value" "220"
+		(property "Value" "180"
 			(at 147.32 128.27 90)
 			(effects
@@
 			)
 		)
-		(property "Value" "220"
+		(property "Value" "180"
 			(at 115.57 71.1199 0)
 			(effects
@@
 			)
 		)
-		(property "Value" "220"
+		(property "Value" "180"
 			(at 157.48 128.27 90)
 			(effects
@@
 			)
 		)
-		(property "Value" "220"
+		(property "Value" "180"
 			(at 93.98 71.1199 0)
 			(effects
@@
 			)
 		)
-		(property "Value" "220"
+		(property "Value" "180"
 			(at 68.58 115.5699 0)
 			(effects
@@
 			)
 		)
-		(property "Value" "220"
+		(property "Value" "180"
 			(at 107.95 128.27 90)
 			(effects
@@
 			)
 		)
-		(property "Value" "220"
+		(property "Value" "180"
 			(at 90.17 115.5699 0)
 			(effects
@@
 			)
 		)
-		(property "Value" "220"
+		(property "Value" "180"
 			(at 57.15 128.27 90)
 			(effects
@@
 			)
 		)
-		(property "Value" "220"
+		(property "Value" "180"
 			(at 46.99 128.27 90)
 			(effects

Commit message: changes
Parts:
- gave numbers to parts that had none: 9
Changed lines of the file:
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@@
 		(dnp no)
 		(fields_autoplaced yes)
-		(property "Reference" "SW?"
+		(property "Reference" "SW1"
 			(at 55.88 171.4499 90)
 			(effects
@@
 			(project ""
 				(path "/198ad8d1-66e3-4deb-889c-1af2b81e67c3/6ff1d53f-9520-4015-acff-de10540e78ee"
-					(reference "SW?")
+					(reference "SW1")
 					(unit 1)
 				)
@@
 		(dnp no)
 		(fields_autoplaced yes)
-		(property "Reference" "R?"
+		(property "Reference" "R2"
 			(at 100.33 160.0199 0)
 			(effects
@@
 			(project "Input Board"
 				(path "/198ad8d1-66e3-4deb-889c-1af2b81e67c3/6ff1d53f-9520-4015-acff-de10540e78ee"
-					(reference "R?")
+					(reference "R2")
 					(unit 1)
 				)
@@
 		(dnp no)
 		(fields_autoplaced yes)
-		(property "Reference" "C?"
+		(property "Reference" "C3"
 			(at 161.29 160.0199 0)
 			(effects
@@
 			(project "Input Board"
 				(path "/198ad8d1-66e3-4deb-889c-1af2b81e67c3/6ff1d53f-9520-4015-acff-de10540e78ee"
-					(reference "C?")
+					(reference "C3")
 					(unit 1)
 				)
@@
 		(dnp no)
 		(fields_autoplaced yes)
-		(property "Reference" "SW?"
+		(property "Reference" "SW3"
 			(at 156.21 171.4499 90)
 			(effects
@@
 			(project "Input Board"
 				(path "/198ad8d1-66e3-4deb-889c-1af2b81e67c3/6ff1d53f-9520-4015-acff-de10540e78ee"
-					(reference "SW?")
+					(reference "SW3")
 					(unit 1)
 				)
@@
 		(dnp no)
 		(fields_autoplaced yes)
-		(property "Reference" "C?"
+		(property "Reference" "C2"
 			(at 111.76 160.0199 0)
 			(effects
@@
 			(project "Input Board"
 				(path "/198ad8d1-66e3-4deb-889c-1af2b81e67c3/6ff1d53f-9520-4015-acff-de10540e78ee"
-					(reference "C?")
+					(reference "C2")
 					(unit 1)
 				)
@@
 		(dnp no)
 		(fields_autoplaced yes)
-		(property "Reference" "SW?"
+		(property "Reference" "SW2"
 			(at 106.68 171.4499 90)
 			(effects
@@
 			(project "Input Board"
 				(path "/198ad8d1-66e3-4deb-889c-1af2b81e67c3/6ff1d53f-9520-4015-acff-de10540e78ee"
-					(reference "SW?")
+					(reference "SW2")
 					(unit 1)
 				)
@@
 		(dnp no)
 		(fields_autoplaced yes)
-		(property "Reference" "C?"
+		(property "Reference" "C1"
 			(at 60.96 160.0199 0)
 			(effects
@@
 			(project "Input Board"
 				(path "/198ad8d1-66e3-4deb-889c-1af2b81e67c3/6ff1d53f-9520-4015-acff-de10540e78ee"
-					(reference "C?")
+					(reference "C1")
 					(unit 1)
 				)
@@
 		(dnp no)
 		(fields_autoplaced yes)
-		(property "Reference" "R?"
+		(property "Reference" "R3"
 			(at 149.86 160.0199 0)
 			(effects
@@
 			(project "Input Board"
 				(path "/198ad8d1-66e3-4deb-889c-1af2b81e67c3/6ff1d53f-9520-4015-acff-de10540e78ee"
-					(reference "R?")
+					(reference "R3")
 					(unit 1)
 				)
@@
 		(dnp no)
 		(fields_autoplaced yes)
-		(property "Reference" "R?"
+		(property "Reference" "R1"
 			(at 49.53 160.0199 0)
 			(effects
@@
 			(project "Input Board"
 				(path "/198ad8d1-66e3-4deb-889c-1af2b81e67c3/6ff1d53f-9520-4015-acff-de10540e78ee"
-					(reference "R?")
+					(reference "R1")
 					(unit 1)
 				)

Commit message: minor layout changes
Parts:
- removed C1, C2, C3: 100n, Capacitor_SMD:C_0603_1608Metric, symbol Device:C
