File: Input Hardware/PCB/Input Board/ctrl.kicad_sch (KiCad schematic)
At the start: 38 parts

Commit message: stmcube model and fixes
Parts:
- added TP? (x9): TestPoint, TestPoint:TestPoint_Pad_1.5x1.5mm, symbol Connector:TestPoint
Connections:
- net at J?.A6 (D+), J?.B6 (D+), U?.3 (I/O2): now also TP?.1
- net at J?.A7 (D-), J?.B7 (D-), U?.1 (I/O1): now also TP?.1
- net at U?.23 (PA7): now also TP?.1
- net at U?.24 (PC4): now also TP?.1
- net at U?.25 (PC5): now also TP?.1
- net at U?.29 (PB10): now also TP?.1
- net at U?.41 (PA8): now also TP?.1
- net at U?.50 (PA15): now also TP?.1
- net at U?.59 (PB7): now also TP?.1
- no-connect marks 5 -> 3
Other:
- note added: "Mux"
- note added: "OLED"
- note added: "OSC OUT?"
- note added: "RX"
- note added: "USB/STLINK/TX"

Commit message: Fix files idc
Parts:
- gave numbers to parts that had none: 41
- renumbered TP6 to TP904, TP1 to TP905, TP2 to TP906, TP3 to TP907, TP4 to TP908, TP5 to TP909

Commit message: Analogue layout
Parts:
- removed TP901, TP904: TestPoint, TestPoint:TestPoint_Pad_1.5x1.5mm, symbol Connector:TestPoint
Connections:
- net Rx1: now also U902.30 (PB11), U902.33 (PB12); no longer U902.18 (PF4), U902.20 (PA4)
- net Rx4: now also U902.18 (PF4), U902.20 (PA4); no longer U902.30 (PB11), U902.33 (PB12)
- no-connect marks 3 -> 4
Changed lines of the file:
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@@
 	)
 	(no_connect
+		(at 27.94 152.4)
+	)
+	(no_connect
 		(at 50.8 58.42)
 	)
@@
 	(wire
 		(pts
-			(xy 25.4 152.4) (xy 27.94 152.4)
-		)
-		(stroke
-			(width 0)
-			(type default)
-		)
-	)
-	(wire
-		(pts
 			(xy 63.5 187.96) (xy 63.5 190.5)
 		)
@@
 		)
 	)
-	(wire
-		(pts
-			(xy 76.2 101.6) (xy 71.12 101.6)
-		)
-		(stroke
-			(width 0)
-			(type default)
-		)
-	)
 	(polyline
 		(pts
@@
 		)
 	)
-	(label "TX_SRCLK"
-		(at 71.12 101.6 180)
-		(effects
-			(font
-				(size 1.27 1.27)
-			)
-			(justify right)
-		)
-	)
 	(label "BOOT0"
 		(at 210.82 48.26 180)
@@
 	(hierarchical_label "Rx4"
 		(shape input)
-		(at 246.38 114.3 0)
+		(at 246.38 53.34 0)
 		(effects
 			(font
@@
 	(hierarchical_label "Rx1"
 		(shape input)
-		(at 210.82 58.42 180)
+		(at 246.38 116.84 0)
 		(effects
 			(font
@@
 				(color 255 30 0 1)
 			)
-			(justify right)
+			(justify left)
 		)
 	)
@@
 	(hierarchical_label "Rx1"
 		(shape input)
-		(at 246.38 53.34 0)
+		(at 246.38 114.3 0)
 		(effects
 			(font
@@
 	(hierarchical_label "Rx4"
 		(shape input)
-		(at 246.38 116.84 0)
+		(at 210.82 58.42 180)
 		(effects
 			(font
@@
 				(color 255 30 0 1)
 			)
-			(justify left)
+			(justify right)
 		)
 	)
@@
 	)
 	(symbol
-		(lib_id "Connector:TestPoint")
-		(at 76.2 101.6 270)
-		(unit 1)
-		(exclude_from_sim no)
-		(in_bom yes)
-		(on_board yes)
-		(dnp no)
-		(property "Reference" "TP904"
-			(at 81.28 101.6 90)
-			(effects
-				(font
-					(size 1.27 1.27)
-				)
-				(justify left)
-			)
-		)
-		(property "Value" "TestPoint"
-			(at 81.28 92.71 90)
-			(effects
-				(font
-					(size 1.27 1.27)
-				)
-				(justify left)
-				(hide yes)
-			)
-		)
-		(property "Footprint" "TestPoint:TestPoint_Pad_1.5x1.5mm"
-			(at 76.2 106.68 0)
-			(effects
-				(font
-					(size 1.27 1.27)
-				)
-				(hide yes)
-			)
-		)
-		(property "Datasheet" "~"
-			(at 76.2 106.68 0)
-			(effects
-				(font
-					(size 1.27 1.27)
-				)
-				(hide yes)
-			)
-		)
-		(property "Description" "test point"
-			(at 76.2 101.6 0)
-			(effects
-				(font
-					(size 1.27 1.27)
-				)
-				(hide yes)
-			)
-		)
-		(pin "1"
-		)
-		(instances
-			(project "Input Board"
-				(path "/198ad8d1-66e3-4deb-889c-1af2b81e67c3/5c16bd2e-d56c-40b8-b84c-f5532d41d46a"
-					(reference "TP904")
-					(unit 1)
-				)
-			)
-		)
-	)
-	(symbol
 		(lib_name "GND_1")
 		(lib_id "power:GND")
@@
 					(unit 1)
 				)
-			)
-		)
-	)
-	(symbol
-		(lib_id "Connector:TestPoint")
-		(at 25.4 152.4 90)
-		(unit 1)
-		(exclude_from_sim no)
-		(in_bom yes)
-		(on_board yes)
-		(dnp no)
-		(property "Reference" "TP901"
-			(at 20.32 152.4 90)
-			(effects
-				(font
-					(size 1.27 1.27)
-				)
-				(justify left)
-			)
-		)
-		(property "Value" "TestPoint"
-			(at 20.32 161.29 90)
-			(effects
-				(font
-					(size 1.27 1.27)
-				)
-				(justify left)
-				(hide yes)
-			)
-		)
-		(property "Footprint" "TestPoint:TestPoint_Pad_1.5x1.5mm"
-			(at 25.4 147.32 0)
-			(effects
-				(font
-					(size 1.27 1.27)
-				)
-				(hide yes)
-			)
-		)
-		(property "Datasheet" "~"
-			(at 25.4 147.32 0)
-			(effects
-				(font
-					(size 1.27 1.27)
-				)
-				(hide yes)
-			)
-		)
-		(property "Description" "test point"
-			(at 25.4 152.4 0)
-			(effects
-				(font
-					(size 1.27 1.27)
-				)
-				(hide yes)
-			)
-		)
-		(pin "1"
-		)
-		(instances
-			(project "Input Board"
-				(path "/198ad8d1-66e3-4deb-889c-1af2b81e67c3/5c16bd2e-d56c-40b8-b84c-f5532d41d46a"
-					(reference "TP901")
-					(unit 1)
-				)

Commit message: Layout Progress
Parts:
- removed JP901: 3.3V STLINK, Jumper:SolderJumper-2_P1.3mm_Open_RoundedPad1.0x1.5mm, symbol Jumper:SolderJumper_2_Open
- removed TP902, TP903: TestPoint, TestPoint:TestPoint_Pad_1.5x1.5mm, symbol Connector:TestPoint
Connections:
- net +3.3V: now also TP905.1
Changed lines of the file:
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@@
 	)
 	(junction
-		(at 55.88 45.72)
-		(diameter 0)
-		(color 0 0 0 0)
-	)
-	(junction
 		(at 158.75 156.21)
 		(diameter 0)
@@
 		(color 0 0 0 0)
 	)
-	(junction
-		(at 55.88 43.18)
-		(diameter 0)
-		(color 0 0 0 0)
-	)
 	(no_connect
 		(at 210.82 63.5)
@@
 	(wire
 		(pts
-			(xy 55.88 43.18) (xy 58.42 43.18)
+			(xy 50.8 43.18) (xy 58.42 43.18)
 		)
 		(stroke
@@
 	(wire
 		(pts
-			(xy 50.8 43.18) (xy 55.88 43.18)
-		)
-		(stroke
-			(width 0)
-			(type default)
-		)
-	)
-	(wire
-		(pts
 			(xy 38.1 187.96) (xy 38.1 190.5)
 		)
@@
 	(wire
 		(pts
-			(xy 55.88 45.72) (xy 58.42 45.72)
-		)
-		(stroke
-			(width 0)
-			(type default)
-		)
-	)
-	(wire
-		(pts
-			(xy 50.8 45.72) (xy 55.88 45.72)
+			(xy 50.8 45.72) (xy 58.42 45.72)
 		)
 		(stroke
@@
 	(wire
 		(pts
-			(xy 69.85 120.65) (xy 69.85 118.11)
-		)
-		(stroke
-			(width 0)
-			(type default)
-		)
-	)
-	(wire
-		(pts
 			(xy 107.95 133.35) (xy 120.65 133.35)
 		)
@@
 	(wire
 		(pts
-			(xy 69.85 107.95) (xy 69.85 110.49)
+			(xy 69.85 107.95) (xy 69.85 120.65)
 		)
 		(stroke
@@
 	)
 	(symbol
-		(lib_id "Connector:TestPoint")
-		(at 55.88 45.72 180)
-		(unit 1)
-		(exclude_from_sim no)
-		(in_bom yes)
-		(on_board yes)
-		(dnp no)
-		(property "Reference" "TP903"
-			(at 55.88 50.8 90)
-			(effects
-				(font
-					(size 1.27 1.27)
-				)
-				(justify left)
-			)
-		)
-		(property "Value" "TestPoint"
-			(at 64.77 50.8 90)
-			(effects
-				(font
-					(size 1.27 1.27)
-				)
-				(justify left)
-				(hide yes)
-			)
-		)
-		(property "Footprint" "TestPoint:TestPoint_Pad_1.5x1.5mm"
-			(at 50.8 45.72 0)
-			(effects
-				(font
-					(size 1.27 1.27)
-				)
-				(hide yes)
-			)
-		)
-		(property "Datasheet" "~"
-			(at 50.8 45.72 0)
-			(effects
-				(font
-					(size 1.27 1.27)
-				)
-				(hide yes)
-			)
-		)
-		(property "Description" "test point"
-			(at 55.88 45.72 0)
-			(effects
-				(font
-					(size 1.27 1.27)
-				)
-				(hide yes)
-			)
-		)
-		(pin "1"
-		)
-		(instances
-			(project "Input Board"
-				(path "/198ad8d1-66e3-4deb-889c-1af2b81e67c3/5c16bd2e-d56c-40b8-b84c-f5532d41d46a"
-					(reference "TP903")
-					(unit 1)
-				)
-			)
-		)
-	)
-	(symbol
 		(lib_id "power:+3.3V")
 		(at 226.06 35.56 0)
@@
 	)
 	(symbol
-		(lib_id "Connector:TestPoint")
-		(at 55.88 43.18 0)
-		(unit 1)
-		(exclude_from_sim no)
-		(in_bom yes)
-		(on_board yes)
-		(dnp no)
-		(property "Reference" "TP902"
-			(at 55.88 38.1 90)
-			(effects
-				(font
-					(size 1.27 1.27)
-				)
-				(justify left)
-			)
-		)
-		(property "Value" "TestPoint"
-			(at 46.99 38.1 90)
-			(effects
-				(font
-					(size 1.27 1.27)
-				)
-				(justify left)
-				(hide yes)
-			)
-		)
-		(property "Footprint" "TestPoint:TestPoint_Pad_1.5x1.5mm"
-			(at 60.96 43.18 0)
-			(effects
-				(font
-					(size 1.27 1.27)
-				)
-				(hide yes)
-			)
-		)
-		(property "Datasheet" "~"
-			(at 60.96 43.18 0)
-			(effects
-				(font
-					(size 1.27 1.27)
-				)
-				(hide yes)
-			)
-		)
-		(property "Description" "test point"
-			(at 55.88 43.18 0)
-			(effects
-				(font
-					(size 1.27 1.27)
-				)
-				(hide yes)
-			)
-		)
-		(pin "1"
-		)
-		(instances
-			(project "Input Board"
-				(path "/198ad8d1-66e3-4deb-889c-1af2b81e67c3/5c16bd2e-d56c-40b8-b84c-f5532d41d46a"
-					(reference "TP902")
-					(unit 1)
-				)
-			)
-		)
-	)
-	(symbol
 		(lib_id "Device:C")
 		(at 50.8 184.15 0)
@@
 					(unit 1)
 				)
-			)
-		)
-	)
-	(symbol
-		(lib_id "Jumper:SolderJumper_2_Open")
-		(at 69.85 114.3 90)
-		(unit 1)
-		(exclude_from_sim no)
-		(in_bom no)
-		(on_board yes)
-		(dnp no)
-		(fields_autoplaced yes)
-		(property "Reference" "JP901"
-			(at 72.39 113.0299 90)
-			(effects
-				(font
-					(size 1.27 1.27)
-				)
-				(justify right)
-			)
-		)
-		(property "Value" "3.3V STLINK"
-			(at 72.39 115.5699 90)
-			(effects
-				(font
-					(size 1.27 1.27)
-				)
-				(justify right)
-			)
-		)
-		(property "Footprint" "Jumper:SolderJumper-2_P1.3mm_Open_RoundedPad1.0x1.5mm"
-			(at 69.85 114.3 0)
-			(effects
-				(font
-					(size 1.27 1.27)
-				)
-				(hide yes)
-			)
-		)
-		(property "Datasheet" "~"
-			(at 69.85 114.3 0)
-			(effects
-				(font
-					(size 1.27 1.27)
-				)
-				(hide yes)
-			)
-		)
-		(property "Description" "Solder Jumper, 2-pole, open"
-			(at 69.85 114.3 0)
-			(effects
-				(font
-					(size 1.27 1.27)
-				)
-				(hide yes)
-			)
-		)
-		(pin "1"
-		)
-		(pin "2"
-		)
-		(instances
-			(project ""
-				(path "/198ad8d1-66e3-4deb-889c-1af2b81e67c3/5c16bd2e-d56c-40b8-b84c-f5532d41d46a"
-					(reference "JP901")
-					(unit 1)
-				)

Commit message: Schematic Cleanup
Parts:
- removed R914: 10k, Resistor_SMD:R_0603_1608Metric, symbol Device:R
- added JP?: SolderJumper_2_Bridged, Jumper:SolderJumper-2_P1.3mm_Bridged_RoundedPad1.0x1.5mm, symbol Jumper:SolderJumper_2_Bridged
- R911: value 10k -> 1M
Connections:
- net BOOT0: now also JP?.2 (B)
- net S_PUSH: now also JP?.1 (A)
- net UI_RCLK: now also R912.2; no longer R913.2
- net UI_SER: now also R913.2
- net UI_SRCLK: now also R910.2; no longer R912.2
- net ~{OE} renamed TX_~{OE}
- net TX_~{OE}: no longer R910.2
Other:
- note removed: "connect boot0"

Commit message: Layout Progress
Parts:
- gave numbers to parts that had none: 1
- renumbered TP905 to TP901, TP906 to TP902, TP907 to TP903, TP908 to TP904, TP909 to TP905, TP910 to TP906, TP911 to TP907, TP912 to TP908, TP913 to TP909, TP914 to TP910, TP915 to TP911, TP916 to TP912
Connections:
- net TX_~{OE}: no longer names the net of U902.56 (PB4)
- no-connect marks 4 -> 5
Changed lines of the file:
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@@
 	)
 	(no_connect
+		(at 246.38 96.52)
+	)
+	(no_connect
 		(at 210.82 63.5)
 	)
@@
 		)
 	)
-	(label "TX_DSO"
+	(label "TX_SDO"
 		(at 101.6 148.59 180)
 		(effects
@@
 		)
 	)
-	(label "TX_~{OE}"
-		(at 246.38 96.52 0)
-		(effects
-			(font
-				(size 1.27 1.27)
-			)
-			(justify left)
-		)
-	)
 	(label "UI_SER"
 		(at 101.6 158.75 180)
@@
 		)
 	)
-	(label "TX_DSO"
+	(label "TX_SDO"
 		(at 246.38 99.06 0)
 		(effects
@@
 		(on_board yes)
 		(dnp no)
-		(property "Reference" "TP905"
+		(property "Reference" "TP901"
 			(at 81.28 120.65 90)
 			(effects
@@
 			(project "Input Board"
 				(path "/198ad8d1-66e3-4deb-889c-1af2b81e67c3/5c16bd2e-d56c-40b8-b84c-f5532d41d46a"
-					(reference "TP905")
+					(reference "TP901")
 					(unit 1)
 				)
@@
 		(on_board yes)
 		(dnp no)
-		(property "Reference" "TP910"
+		(property "Reference" "TP906"
 			(at 205.74 78.74 90)
 			(effects
@@
 			(project "Input Board"
 				(path "/198ad8d1-66e3-4deb-889c-1af2b81e67c3/5c16bd2e-d56c-40b8-b84c-f5532d41d46a"
-					(reference "TP910")
+					(reference "TP906")
 					(unit 1)
 				)
@@
 		(on_board yes)
 		(dnp no)
-		(property "Reference" "JP?"
+		(property "Reference" "JP901"
 			(at 196.85 44.45 0)
 			(effects
@@
 			(project ""
 				(path "/198ad8d1-66e3-4deb-889c-1af2b81e67c3/5c16bd2e-d56c-40b8-b84c-f5532d41d46a"
-					(reference "JP?")
+					(reference "JP901")
 					(unit 1)
 				)
@@
 		(on_board yes)
 		(dnp no)
-		(property "Reference" "TP908"
+		(property "Reference" "TP904"
 			(at 81.28 128.27 90)
 			(effects
@@
 			(project "Input Board"
 				(path "/198ad8d1-66e3-4deb-889c-1af2b81e67c3/5c16bd2e-d56c-40b8-b84c-f5532d41d46a"
-					(reference "TP908")
+					(reference "TP904")
 					(unit 1)
 				)
@@
 		(on_board yes)
 		(dnp no)
-		(property "Reference" "TP912"
+		(property "Reference" "TP908"
 			(at 251.46 60.96 90)
 			(effects
@@
 			(project "Input Board"
 				(path "/198ad8d1-66e3-4deb-889c-1af2b81e67c3/5c16bd2e-d56c-40b8-b84c-f5532d41d46a"
-					(reference "TP912")
+					(reference "TP908")
 					(unit 1)
 				)
@@
 		(on_board yes)
 		(dnp no)
-		(property "Reference" "TP914"
+		(property "Reference" "TP910"
 			(at 251.46 81.28 90)
 			(effects
@@
 			(project "Input Board"
 				(path "/198ad8d1-66e3-4deb-889c-1af2b81e67c3/5c16bd2e-d56c-40b8-b84c-f5532d41d46a"
-					(reference "TP914")
+					(reference "TP910")
 					(unit 1)
 				)
@@
 		(on_board yes)
 		(dnp no)
-		(property "Reference" "TP907"
+		(property "Reference" "TP903"
 			(at 81.28 125.73 90)
 			(effects
@@
 			(project "Input Board"
 				(path "/198ad8d1-66e3-4deb-889c-1af2b81e67c3/5c16bd2e-d56c-40b8-b84c-f5532d41d46a"
-					(reference "TP907")
+					(reference "TP903")
 					(unit 1)
 				)
@@
 		(on_board yes)
 		(dnp no)
-		(property "Reference" "TP906"
+		(property "Reference" "TP902"
 			(at 81.28 123.19 90)
 			(effects
@@
 			(project "Input Board"
 				(path "/198ad8d1-66e3-4deb-889c-1af2b81e67c3/5c16bd2e-d56c-40b8-b84c-f5532d41d46a"
-					(reference "TP906")
+					(reference "TP902")
 					(unit 1)
 				)
@@
 		(on_board yes)
 		(dnp no)
-		(property "Reference" "TP916"
+		(property "Reference" "TP912"
 			(at 251.46 111.76 90)
 			(effects
@@
 			(project "Input Board"
 				(path "/198ad8d1-66e3-4deb-889c-1af2b81e67c3/5c16bd2e-d56c-40b8-b84c-f5532d41d46a"
-					(reference "TP916")
+					(reference "TP912")
 					(unit 1)
 				)
@@
 		(on_board yes)
 		(dnp no)
-		(property "Reference" "TP909"
+		(property "Reference" "TP905"
 			(at 81.28 130.81 90)
 			(effects
@@
 			(project "Input Board"
 				(path "/198ad8d1-66e3-4deb-889c-1af2b81e67c3/5c16bd2e-d56c-40b8-b84c-f5532d41d46a"
-					(reference "TP909")
+					(reference "TP905")
 					(unit 1)
 				)
@@
 		(on_board yes)
 		(dnp no)
-		(property "Reference" "TP911"
+		(property "Reference" "TP907"
 			(at 205.74 81.28 90)
 			(effects
@@
 			(project "Input Board"
 				(path "/198ad8d1-66e3-4deb-889c-1af2b81e67c3/5c16bd2e-d56c-40b8-b84c-f5532d41d46a"
-					(reference "TP911")
+					(reference "TP907")
 					(unit 1)
 				)
@@
 		(on_board yes)
 		(dnp no)
-		(property "Reference" "TP915"
+		(property "Reference" "TP911"
 			(at 251.46 104.14 90)
 			(effects
@@
 			(project "Input Board"
 				(path "/198ad8d1-66e3-4deb-889c-1af2b81e67c3/5c16bd2e-d56c-40b8-b84c-f5532d41d46a"
-					(reference "TP915")
+					(reference "TP911")
 					(unit 1)
 				)
@@
 		(on_board yes)
 		(dnp no)
-		(property "Reference" "TP913"
+		(property "Reference" "TP909"
 			(at 251.46 63.5 90)
 			(effects
@@
 			(project "Input Board"
 				(path "/198ad8d1-66e3-4deb-889c-1af2b81e67c3/5c16bd2e-d56c-40b8-b84c-f5532d41d46a"
-					(reference "TP913")
+					(reference "TP909")
 					(unit 1)
 				)

Commit message: Layout Progress
Parts:
- removed C905: 47n, Capacitor_SMD:C_0603_1608Metric, symbol Device:C
- removed C907: 100n, Capacitor_SMD:C_0603_1608Metric, symbol Device:C
- removed TP910, TP911: TestPoint, TestPoint:TestPoint_Pad_1.5x1.5mm, symbol Connector:TestPoint
- renumbered C906 to C905, C908 to C907, C909 to C908, C910 to C909, C911 to C910, C912 to C911, TP912 to TP910
Connections:
- net S_PUSH: no longer JP901.1 (A)
- net Push_1: now reaches U902.50 (PA15)
- net Push_2: now reaches U902.56 (PB4)
- net Push_3: now reaches U902.59 (PB7)
- net Push_3: now also JP901.1 (A)
- net TSC_1: no longer names the net of U902.14 (PA0)
- net TSC_2: no longer names the net of U902.15 (PA1)
- net TSC_3: no longer names the net of U902.16 (PA2)
- net TSC_CS: no longer names the net of U902.17 (PA3)
- no-connect marks 5 -> 4
Other:
- note removed: "TSC_G1_IO1"
- note removed: "TSC_G1_IO2"
- note removed: "TSC_G1_IO3"
- note removed: "TSC_G1_IO4"
- moved on the sheet: C902, C903, C904, C905

Commit message: Layout Progress
Connections:
- net O_CENTER: now also U902.2 (PC13); no longer U902.4 (PC15)
- net O_LEFT: now also U902.61 (PB8); no longer U902.2 (PC13)
- net O_UP: now also U902.4 (PC15); no longer U902.61 (PB8)
