File: Input Hardware/PCB/Input Board/ctrl.kicad_sch (KiCad schematic)
At the start: 38 parts, among them J901 USB_C_Receptacle_USB2.0_16P, U901 USBLC6-2SC6, U902 STM32F303RBTx, Y901 ECS-2520MV-xxx-xx

Commit message: Layout Progress
Connections:
- net S_A: now also U902.10 (PC2); no longer U902.9 (PC1)
- net S_B: now also U902.9 (PC1); no longer U902.10 (PC2)
Changed lines of the file:
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@@
 	(hierarchical_label "S_A"
 		(shape input)
-		(at 210.82 71.12 180)
+		(at 210.82 73.66 180)
 		(effects
 			(font
@@
 	(hierarchical_label "S_B"
 		(shape input)
-		(at 210.82 73.66 180)
+		(at 210.82 71.12 180)
 		(effects
 			(font

Commit message: Fixed Switches
Parts:
- R911: value 1M -> 10k
Changed lines of the file:
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@@
 			)
 		)
-		(property "Value" "1M"
+		(property "Value" "10k"
 			(at 154.94 185.4199 0)
 			(effects

Commit message: add bias resistor, fix LED polarity
Parts:
- renumbered C907 to C906, C908 to C907, C909 to C908, C910 to C909, C911 to C910
Connections:
- no-connect marks 4 -> 8
Other:
- note removed: "OSC OUT?"

Commit message: sleep pin rewire
Parts:
- removed TP909: TestPoint, TestPoint:TestPoint_Pad_1.5x1.5mm, symbol Connector:TestPoint
Connections:
- net SLEEP: now reaches U902.41 (PA8)
Changed lines of the file:
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@@
 		)
 	)
+	(hierarchical_label "SLEEP"
+		(shape input)
+		(at 246.38 63.5 0)
+		(effects
+			(font
+				(size 1.27 1.27)
+			)
+			(justify left)
+		)
+	)
 	(hierarchical_label "O_UP"
 		(shape input)
@@
 					(unit 1)
 				)
-			)
-		)
-	)
-	(symbol
-		(lib_id "Connector:TestPoint")
-		(at 246.38 63.5 270)
-		(unit 1)
-		(exclude_from_sim no)
-		(in_bom yes)
-		(on_board yes)
-		(dnp no)
-		(property "Reference" "TP909"
-			(at 251.46 63.5 90)
-			(effects
-				(font
-					(size 1.27 1.27)
-				)
-				(justify left)
-			)
-		)
-		(property "Value" "TestPoint"
-			(at 251.46 54.61 90)
-			(effects
-				(font
-					(size 1.27 1.27)
-				)
-				(justify left)
-				(hide yes)
-			)
-		)
-		(property "Footprint" "TestPoint:TestPoint_Pad_1.5x1.5mm"
-			(at 246.38 68.58 0)
-			(effects
-				(font
-					(size 1.27 1.27)
-				)
-				(hide yes)
-			)
-		)
-		(property "Datasheet" "~"
-			(at 246.38 68.58 0)
-			(effects
-				(font
-					(size 1.27 1.27)
-				)
-				(hide yes)
-			)
-		)
-		(property "Description" "test point"
-			(at 246.38 63.5 0)
-			(effects
-				(font
-					(size 1.27 1.27)
-				)
-				(hide yes)
-			)
-		)
-		(pin "1"
-		)
-		(instances
-			(project "Input Board"
-				(path "/198ad8d1-66e3-4deb-889c-1af2b81e67c3/5c16bd2e-d56c-40b8-b84c-f5532d41d46a"
-					(reference "TP909")
-					(unit 1)
-				)

Commit message: add TX sleep
Parts:
- added R?: 10k, Resistor_SMD:R_0603_1608Metric, symbol Device:R
Connections:
- net +5V: now also R?.1
- net SLEEP: now also R?.2
Other:
- moved on the sheet: R907, R908, R909, R910, R912, R913

Commit message: Final Layout
Parts:
- removed C901: 100n, Capacitor_SMD:C_0603_1608Metric, symbol Device:C
- gave numbers to parts that had none: 1
- renumbered C902 to C901, C903 to C902, C904 to C903, C905 to C904, C906 to C905, C907 to C906, C908 to C907, C909 to C908, C910 to C909, R910 to R912, R912 to R913, R913 to R914, TP910 to TP909

Commit message: minor cosmetic
Other:
- note removed: "Set IO as open-drain"
Changed lines of the file:
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@@
-		)
-	)
-	(text "Set IO as open-drain"
-		(exclude_from_sim no)
-		(at 120.65 129.54 0)
-		(effects
-			(font
-				(size 1.27 1.27)
-			)
 		)
 	)
